Commit message: the segbot description package has been fixed - at least to a good enough point

File: segbot_description/urdf/segbot_base.xacro (robot description, xacro)
@@ -3,5 +3,4 @@
   <!-- Included URDF Files -->
   <include filename="$(find segbot_description)/urdf/segbot_wheel.xacro" />
-  <include filename="$(find segbot_description)/urdf/kinect.urdf.xacro" />
   <macro name="segbot">
     <link name="base_footprint">

File: segbot_description/urdf/sensors/hokuyo_04lx_laser.urdf.xacro (robot description, xacro)
@@ -18,4 +18,10 @@
         <inertia ixx="0.0001" ixy="0" ixz="0" iyy="0.000001" iyz="0" izz="0.0001" />
       </inertial>
+      <visual>
+        <origin xyz="0 0 0" rpy="0 0 0" />
+        <geometry>
+          <box size="0.05 0.05 0.07" />
+        </geometry>
+      </visual>
     </link>
     <!-- gazebo extensions -->
