Commit message: fixed a minor mistake in the Kinect mount, added a mount description for the hokuyo as well - still missing a mesh model for the hokuyo

File: segbot_description/urdf/common.urdf.xacro (robot description, xacro)
@@ -1,5 +1,13 @@
 <?xml version="1.0"?>
 <root xmlns:xacro="http://ros.org/wiki/xacro">
+  <!-- constants -->
   <xacro:property name="M_PI" value="3.14159"/>
   <xacro:property name="INCH_TO_M" value="0.0254"/>
+  <!-- colors -->
+  <material name="beam_grey">
+    <color rgba="0.7 0.7 0.7 1" />
+  </material>
+  <material name="sheet_grey">
+    <color rgba="0.5 0.5 0.5 1" />
+  </material>
 </root>

File: segbot_description/urdf/components/aluminium_sheet.urdf.xacro (robot description, xacro)
@@ -20,7 +20,5 @@
           <box size="${length} ${width} ${thickness}" />
         </geometry>
-        <material name="sheet_grey">
-          <color rgba="0.5 0.5 0.5 1" />
-        </material>
+        <material name="sheet_grey" />
       </visual>
     </link>

File: segbot_description/urdf/components/beam_8020.urdf.xacro (robot description, xacro)
@@ -23,7 +23,5 @@
           <box size="${1*INCH_TO_M} ${1*INCH_TO_M} ${length}" />
         </geometry>
-        <material name="beam_grey">
-          <color rgba="0.8 0.8 0.8 1" />
-        </material>
+        <material name="beam_grey" />
       </visual>
     </link>

File: segbot_description/urdf/components/standoff_632.urdf.xacro (robot description, xacro)
@@ -20,7 +20,5 @@
           <cylinder length="${length}" radius="0.003175" />
         </geometry>
-        <material name="beam_grey">
-          <color rgba="0.8 0.8 0.8 1" />
-        </material>
+        <material name="beam_grey" />
       </visual>
     </link>

File: segbot_description/urdf/mounts/kinect_mount.urdf.xacro (robot description, xacro)
@@ -4,5 +4,4 @@
       xmlns:interface="http://playerstage.sourceforge.net/gazebo/xmlschema/#interface"
       xmlns:xacro="http://ros.org/wiki/xacro">
-  <include filename="$(find segbot_description)/urdf/common.urdf.xacro" />
   <include filename="$(find segbot_description)/urdf/components/beam_8020.urdf.xacro" />
   <include filename="$(find segbot_description)/urdf/components/standoff_632.urdf.xacro" />
@@ -14,25 +13,25 @@
     </xacro:beam_8020>
     <xacro:aluminium_sheet name="${name}_base_plate" parent="${name}_sensor_beam"
-                           thickness="${0.125*INCH_TO_M}" length="${4*INCH_TO_M}" width="${9*INCH_TO_M}">
+                           thickness="${0.0625*INCH_TO_M}" length="${4*INCH_TO_M}" width="${9*INCH_TO_M}">
                            <origin xyz="${0.5*INCH_TO_M} 0 ${length/2}" rpy="${M_PI/2} 0 ${M_PI/2}" />
     </xacro:aluminium_sheet>
     <xacro:standoff_632 name="${name}_standoff_1" parent="${name}_base_plate" length="${2.0*INCH_TO_M}">
-      <origin xyz="${1.5*INCH_TO_M} ${-4*INCH_TO_M} ${0.125*INCH_TO_M}"
+      <origin xyz="${1.5*INCH_TO_M} ${-4*INCH_TO_M} ${0.0625*INCH_TO_M}"
               rpy="0 0 0" />
     </xacro:standoff_632>
     <xacro:standoff_632 name="${name}_standoff_2" parent="${name}_base_plate" length="${2.0*INCH_TO_M}">
-      <origin xyz="${1.5*INCH_TO_M} ${4*INCH_TO_M} ${0.125*INCH_TO_M}"
+      <origin xyz="${1.5*INCH_TO_M} ${4*INCH_TO_M} ${0.0625*INCH_TO_M}"
               rpy="0 0 0" />
     </xacro:standoff_632>
     <xacro:standoff_632 name="${name}_standoff_3" parent="${name}_base_plate" length="${2.0*INCH_TO_M}">
-      <origin xyz="${-1.5*INCH_TO_M} ${4*INCH_TO_M} ${0.125*INCH_TO_M}"
+      <origin xyz="${-1.5*INCH_TO_M} ${4*INCH_TO_M} ${0.0625*INCH_TO_M}"
               rpy="0 0 0" />
     </xacro:standoff_632>
     <xacro:standoff_632 name="${name}_standoff_4" parent="${name}_base_plate" length="${2.0*INCH_TO_M}">
-      <origin xyz="${-1.5*INCH_TO_M} ${-4*INCH_TO_M} ${0.125*INCH_TO_M}"
+      <origin xyz="${-1.5*INCH_TO_M} ${-4*INCH_TO_M} ${0.0625*INCH_TO_M}"
               rpy="0 0 0" />
     </xacro:standoff_632>
     <xacro:aluminium_sheet name="${name}_top_plate" parent="${name}_standoff_1"
-                           thickness="${0.125*INCH_TO_M}" length="${4*INCH_TO_M}" width="${9*INCH_TO_M}">
+                           thickness="${0.0625*INCH_TO_M}" length="${4*INCH_TO_M}" width="${9*INCH_TO_M}">
       <origin xyz="${-1.5*INCH_TO_M} ${4*INCH_TO_M} ${2*INCH_TO_M}"
               rpy="0 0 0" />

Commit message: finished the entire segbot chassis

File: segbot_description/urdf/common.urdf.xacro (robot description, xacro)
@@ -11,3 +11,6 @@
     <color rgba="0.5 0.5 0.5 1" />
   </material>
+  <material name="black">
+    <color rgba="0 0 0 1" />
+  </material>
 </root>

File: segbot_description/urdf/components/aluminium_sheet.urdf.xacro (robot description, xacro)
@@ -3,5 +3,5 @@
   <xacro:macro name="aluminium_sheet" params="name parent thickness length width *origin">
     <joint name="${name}_joint" type="fixed">
-      <insert_block name="origin" />
+      <xacro:insert_block name="origin" />
       <parent link="${parent}_link"/>
       <child link="${name}_link"/>

Commit message: minor change in color to get some depth in rviz

File: segbot_description/urdf/common.urdf.xacro (robot description, xacro)
@@ -22,3 +22,6 @@
     <color rgba="0 0 0 1" />
   </material>
+  <material name="almost_black">
+    <color rgba="0.02 0.02 0.02 1" />
+  </material>
 </root>

File: segbot_description/urdf/segbot_chassis.urdf.xacro (robot description, xacro)
@@ -39,5 +39,5 @@
           <box size="${7*INCH_TO_M} ${14*INCH_TO_M} ${11*INCH_TO_M}" />
         </geometry>
-        <material name="black" />
+        <material name="almost_black" />
       </visual>
     </link>
