Commit message: Add arm robot
Prefix some unprefixed xacro tags

File: segbot_description/urdf/segway_110_base.urdf.xacro (robot description, xacro)
@@ -33,5 +33,5 @@
   <xacro:include filename="$(find segway_description)/urdf/segway_components/ui_box_spacer_mount.urdf.xacro" />
   <xacro:include filename="$(find segway_description)/urdf/accessories.urdf.xacro" />
-  <property name="M_PI" value="3.14159"/>
+  <xacro:property name="M_PI" value="3.14159"/>
   <!-- Wheel Mounting Positions -->
   <xacro:property name="track" value="0.479111" />

File: segbot_description/urdf/sensors/hokuyo_laser.urdf.xacro (robot description, xacro)
@@ -8,5 +8,5 @@
     <joint name="${name}_joint" type="fixed">
       <axis xyz="0 1 0" />
-      <insert_block name="origin" />
+      <xacro:insert_block name="origin" />
       <parent link="${parent}_link"/>
       <child link="${name}_link"/>

File: segbot_description/urdf/sensors/kinect_camera.urdf.xacro (robot description, xacro)
@@ -7,5 +7,5 @@
   <xacro:macro name="kinect_camera" params="name parent *origin">
     <joint name="${name}_joint" type="fixed">
-      <insert_block name="origin" />
+      <xacro:insert_block name="origin" />
       <parent link="${parent}_link"/>
       <child link="${name}_link"/>
