Commit message: in combination with updates in bwi_launch, allows simulated planning through MoveIt

File: segbot_description/urdf/segbot_base.arm.urdf.xacro (robot description, xacro)
@@ -41,7 +41,10 @@
       <joint_properties damping="0.0" friction="0.0"/>
     </joint>
-    <transmission type="pr2_mechanism_model/SimpleTransmission" name="base_caster_support_trans">
+    <transmission name="base_caster_support_trans">
+      <type>transmission_interface/SimpleTransmission</type>
       <actuator name="base_caster_support_motor"/>
-      <joint name="base_caster_support_joint"/>
+      <joint name="base_caster_support_joint">
+          <hardwareInterface>hardware_interface/EffortJointInterface</hardwareInterface>
+      </joint>
       <mechanicalReduction>1.0</mechanicalReduction>
     </transmission>
@@ -76,7 +79,10 @@
       <joint_properties damping="0.0" friction="0.0"/>
     </joint>
-    <transmission type="pr2_mechanism_model/SimpleTransmission" name="caster_wheel_trans">
+    <transmission name="caster_wheel_trans">
+      <type>transmission_interface/SimpleTransmission</type>
       <actuator name="caster_wheel_motor"/>
-      <joint name="caster_wheel_joint"/>
+      <joint name="caster_wheel_joint">
+          <hardwareInterface>hardware_interface/EffortJointInterface</hardwareInterface>
+      </joint>
       <mechanicalReduction>1.0</mechanicalReduction>
     </transmission>
@@ -106,7 +112,10 @@
       <joint_properties damping="0.0" friction="0.0"/>
     </joint>
-    <transmission type="pr2_mechanism_model/SimpleTransmission" name="base_caster_support_trans">
+    <transmission name="base_caster_support_trans">
+      <type>transmission_interface/SimpleTransmission</type>
       <actuator name="base_caster_support_motor"/>
-      <joint name="base_caster_support_joint_front"/>
+      <joint name="base_caster_support_joint_front">
+          <hardwareInterface>hardware_interface/EffortJointInterface</hardwareInterface>
+      </joint>
       <mechanicalReduction>1.0</mechanicalReduction>
     </transmission>
@@ -142,7 +151,10 @@
       <joint_properties damping="0.0" friction="0.0"/>
     </joint>
-    <transmission type="pr2_mechanism_model/SimpleTransmission" name="caster_wheel_trans">
+    <transmission name="caster_wheel_trans">
+      <type>transmission_interface/SimpleTransmission</type>
       <actuator name="caster_wheel_motor"/>
-      <joint name="caster_wheel_joint_front"/>
+      <joint name="caster_wheel_joint_front">
+          <hardwareInterface>hardware_interface/EffortJointInterface</hardwareInterface>
+      </joint>
       <mechanicalReduction>1.0</mechanicalReduction>
     </transmission>
