Commit message: a bit more cleaning up of the urdf file description

File: segbot_description/urdf/segbot_base.urdf.xacro (robot description, xacro)
@@ -1,7 +1,9 @@
 <?xml version="1.0"?>
-<robot>
+<root
+      xmlns:xacro="http://ros.org/wiki/xacro">
   <!-- Included URDF Files -->
   <include filename="$(find segbot_description)/urdf/segbot_wheel.urdf.xacro" />
-  <macro name="segbot">
+  <xacro:macro name="segbot">
+    <!-- root link, on the ground just below the robot origin -->
     <link name="base_footprint">
       <visual>
@@ -17,5 +19,5 @@
       <child link="base_link" />
     </joint>
-    <!-- Links and Joints (i.e., the robot) -->
+    <!-- This is the robot origin, middle of the wheel axis -->
     <link name="base_link">
       <inertial>
@@ -27,11 +29,12 @@
       </inertial>
       <visual>
-        <segbot_base_link_visual />
+        <xacro:segbot_base_link_visual />
       </visual>
       <collision>
-        <segbot_base_link_collision />
+        <xacro:segbot_base_link_collision />
       </collision>
     </link>
-    <gazebo_segbot_base_link_surface />
+    <xacro:gazebo_segbot_base_link_surface />
+    <!-- pushing the center of mass of the body to a more appropriate pos -->
     <joint name="base_center_of_mass_joint" type="fixed">
       <origin xyz="-0.1 0 -0.075" rpy="0 0 0" />
@@ -48,4 +51,5 @@
       </inertial>
     </link>
+    <!-- castor joint and wheel -->
     <joint name="base_caster_support_joint" type="continuous">
       <origin xyz="-0.3292 0 -0.0485" rpy="0 0 0" />
@@ -100,21 +104,21 @@
       </inertial>
       <visual>
-        <segbot_castor_wheel_link_visual />
+        <xacro:segbot_castor_wheel_link_visual />
       </visual>
       <collision>
-        <segbot_castor_wheel_link_collision />
+        <xacro:segbot_castor_wheel_link_collision />
       </collision>
     </link>
-    <gazebo_castor_wheel_link_surface />
+    <xacro:gazebo_segbot_castor_wheel_link_surface />
     <!-- left wheel -->
-    <segbot_wheel suffix="left" parent="base_link">
+    <xacro:segbot_wheel suffix="left" parent="base_link">
       <origin xyz="0 0.2689 0.0239" rpy="0 0 0" />
-    </segbot_wheel>
+    </xacro:segbot_wheel>
     <!-- right wheel -->
-    <segbot_wheel suffix="right" parent="base_link">
+    <xacro:segbot_wheel suffix="right" parent="base_link">
       <origin xyz="0 -0.2689 0.0239" rpy="0 0 0" />
-    </segbot_wheel>
+    </xacro:segbot_wheel>
     <!-- ros controllers -->
-    <gazebo_segbot_ros_controllers/>
-  </macro>
-</robot>
+    <xacro:gazebo_segbot_ros_controllers/>
+  </xacro:macro>
+</root>

File: segbot_description/urdf/segbot_wheel.urdf.xacro (robot description, xacro)
@@ -1,10 +1,8 @@
 <?xml version="1.0"?>
-<robot
-  xmlns:sensor="http://playerstage.sourceforge.net/gazebo/xmlschema/#sensor"
-  xmlns:controller="http://playerstage.sourceforge.net/gazebo/xmlschema/#controller"
-  xmlns:interface="http://playerstage.sourceforge.net/gazebo/xmlschema/#interface">
-  <macro name="segbot_wheel" params="suffix parent *origin">
+<root
+      xmlns:xacro="http://ros.org/wiki/xacro">
+  <xacro:macro name="segbot_wheel" params="suffix parent *origin">
     <joint name="${parent}_${suffix}_wheel_joint" type="continuous">
-      <insert_block name="origin" />
+      <xacro:insert_block name="origin" />
       <axis xyz="0 1 0" />
       <anchor xyz="0 0 0" />
@@ -23,11 +21,11 @@
       </inertial>
       <visual>
-        <segbot_wheel_visual suffix="${suffix}" />
+        <xacro:segbot_wheel_visual suffix="${suffix}" />
       </visual>
       <collision>
-        <segbot_wheel_collision suffix="${suffix}" />
+        <xacro:segbot_wheel_collision suffix="${suffix}" />
       </collision>
     </link>
-    <gazebo_segbot_wheel_surface />
+    <xacro:gazebo_segbot_wheel_surface />
     <transmission type="pr2_mechanism_model/SimpleTransmission" name="${parent}_${suffix}_wheel_trans">
       <actuator name="${parent}_${suffix}_wheel_motor" />
@@ -35,4 +33,4 @@
       <mechanicalReduction>1.0</mechanicalReduction>
     </transmission>
-  </macro>
-</robot>
+  </xacro:macro>
+</root>

Commit message: reenabled transmission - now gazebo produces the correct joint states - useful in rviz visualization

File: segbot_description/urdf/segbot_base.urdf.xacro (robot description, xacro)
@@ -96,9 +96,9 @@
       <joint_properties damping="0.0" friction="0.0" />
     </joint>
-    <!-- <transmission type="pr2_mechanism_model/SimpleTransmission" name="caster_wheel_trans"> -->
-    <!--   <actuator name="caster_wheel_motor" /> -->
-    <!--   <joint name="caster_wheel_joint" /> -->
-    <!--   <mechanicalReduction>1.0</mechanicalReduction> -->
-    <!-- </transmission> -->
+    <transmission type="pr2_mechanism_model/SimpleTransmission" name="caster_wheel_trans">
+      <actuator name="caster_wheel_motor" />
+      <joint name="caster_wheel_joint" />
+      <mechanicalReduction>1.0</mechanicalReduction>
+    </transmission>
     <link name="caster_wheel_link">
       <inertial>

File: segbot_description/urdf/segbot_wheel.urdf.xacro (robot description, xacro)
@@ -28,9 +28,9 @@
     </link>
     <xacro:gazebo_segbot_wheel_surface parent="${parent}" suffix="${suffix}" />
-    <!-- <transmission type="pr2_mechanism_model/SimpleTransmission" name="${parent}_${suffix}_wheel_trans"> -->
-    <!--   <actuator name="${parent}_${suffix}_wheel_motor" /> -->
-    <!--   <joint name="${parent}_${suffix}_wheel_joint" /> -->
-    <!--   <mechanicalReduction>1.0</mechanicalReduction> -->
-    <!-- </transmission> -->
+    <transmission type="pr2_mechanism_model/SimpleTransmission" name="${parent}_${suffix}_wheel_trans">
+      <actuator name="${parent}_${suffix}_wheel_motor" />
+      <joint name="${parent}_${suffix}_wheel_joint" />
+      <mechanicalReduction>1.0</mechanicalReduction>
+    </transmission>
   </xacro:macro>
 </root>

Commit message: residual transmission syntax fixes

File: segbot_description/urdf/segbot_base.urdf.xacro (robot description, xacro)
@@ -42,7 +42,10 @@
       <joint_properties damping="0.0" friction="0.0" />
     </joint>
-    <transmission type="pr2_mechanism_model/SimpleTransmission" name="base_caster_support_trans">
+    <transmission name="base_caster_support_trans">
+      <type>transmission_interface/SimpleTransmission</type>
       <actuator name="base_caster_support_motor" />
-      <joint name="base_caster_support_joint" />
+      <joint name="base_caster_support_joint">
+          <hardwareInterface>hardware_interface/EffortJointInterface</hardwareInterface>
+      </joint>
       <mechanicalReduction>1.0</mechanicalReduction>
     </transmission>
@@ -79,7 +82,10 @@
       <joint_properties damping="0.0" friction="0.0" />
     </joint>
-    <transmission type="pr2_mechanism_model/SimpleTransmission" name="caster_wheel_trans">
+    <transmission name="caster_wheel_trans">
+      <type>transmission_interface/SimpleTransmission</type>
       <actuator name="caster_wheel_motor" />
-      <joint name="caster_wheel_joint" />
+      <joint name="caster_wheel_joint">
+          <hardwareInterface>hardware_interface/EffortJointInterface</hardwareInterface>
+      </joint>
       <mechanicalReduction>1.0</mechanicalReduction>
     </transmission>

File: segbot_description/urdf/segbot_wheel.urdf.xacro (robot description, xacro)
@@ -29,7 +29,10 @@
     </link>
     <xacro:gazebo_segbot_wheel_surface parent="${parent}" suffix="${suffix}" />
-    <transmission type="pr2_mechanism_model/SimpleTransmission" name="${parent}_${suffix}_wheel_trans">
+    <transmission name="${parent}_${suffix}_wheel_trans">
+      <type>transmission_interface/SimpleTransmission</type>
       <actuator name="${parent}_${suffix}_wheel_motor" />
-      <joint name="${parent}_${suffix}_wheel_joint" />
+      <joint name="${parent}_${suffix}_wheel_joint">
+          <hardwareInterface>hardware_interface/EffortJointInterface</hardwareInterface>
+      </joint>
       <mechanicalReduction>1.0</mechanicalReduction>
     </transmission>
