Commit message: a larger number of changes (added collision+material properties for gazebo, some bug fixes for hokuyo and kinect launches). Still trying to get gazebo to behave properly

File: segbot_description/urdf/components/aluminium_sheet.urdf.xacro (robot description, xacro)
@@ -22,5 +22,14 @@
         <material name="dark_grey" />
       </visual>
+      <collision>
+        <origin xyz="0 0 ${thickness/2}" rpy="0 0 0"/>
+        <geometry>
+          <box size="${length} ${width} ${thickness}" />
+        </geometry>
+      </collision>
     </link>
+    <gazebo reference="${name}_link">
+      <material>Gazebo/Grey</material>
+    </gazebo>
   </xacro:macro>
 </root>

File: segbot_description/urdf/components/beam_8020.urdf.xacro (robot description, xacro)
@@ -25,5 +25,14 @@
         <material name="light_grey" />
       </visual>
+      <collision>
+        <origin xyz="0 0 ${length/2}" rpy="0 0 0"/>
+        <geometry>
+          <box size="${1*INCH_TO_M} ${1*INCH_TO_M} ${length}" />
+        </geometry>
+      </collision>
     </link>
+    <gazebo reference="${name}_link">
+      <material>Gazebo/Grey</material>
+    </gazebo>
   </xacro:macro>
 </root>

File: segbot_description/urdf/components/standoff_632.urdf.xacro (robot description, xacro)
@@ -22,5 +22,14 @@
         <material name="light_grey" />
       </visual>
+      <collision>
+        <origin xyz="0 0 ${length/2}" rpy="0 0 0"/>
+        <geometry>
+          <cylinder length="${length}" radius="0.003175" />
+        </geometry>
+      </collision>
     </link>
+    <gazebo reference="${name}_link">
+      <material>Gazebo/Grey</material>
+    </gazebo>
   </xacro:macro>
 </root>

File: segbot_description/urdf/segbot_chassis.urdf.xacro (robot description, xacro)
@@ -41,4 +41,10 @@
         <material name="almost_black" />
       </visual>
+      <collision>
+        <origin xyz="0 0 ${5.5*INCH_TO_M}" rpy="0 0 0"/>
+        <geometry>
+          <box size="${7*INCH_TO_M} ${14*INCH_TO_M} ${11*INCH_TO_M}" />
+        </geometry>
+      </collision>
     </link>
     <!-- 80/20 base beams -->

File: segbot_description/urdf/sensors/hokuyo_04lx_laser.gazebo.xacro (robot description, xacro)
@@ -19,5 +19,5 @@
         <updateRate>${update_rate}</updateRate>
         <controller:gazebo_ros_laser name="gazebo_ros_${name}_controller" plugin="libgazebo_ros_laser.so">
-          <gaussianNoise>0.05</gaussianNoise>
+          <gaussianNoise>0.03</gaussianNoise>
           <alwaysOn>true</alwaysOn>
           <updateRate>${update_rate}</updateRate>

File: segbot_description/urdf/sensors/hokuyo_04lx_laser.urdf.xacro (robot description, xacro)
@@ -12,5 +12,5 @@
       <child link="${name}_link"/>
     </joint>
-    <link name="${name}_link" type="laser">
+    <link name="${name}_link">
       <inertial>
         <mass value="0.001" />
@@ -25,7 +25,27 @@
         </geometry>
       </visual>
+      <collision>
+        <origin xyz="0 0 0" rpy="0 0 0" />
+        <geometry>
+          <!-- <box size="0.05 0.05 0.07" /> -->
+          <mesh filename="package://segbot_description/meshes/hokuyo.dae" scale="0.0254 0.0254 0.0254" />
+        </geometry>
+      </collision>
+    </link>
+    <!-- go from the base of the laser to the actual sensor location -->
+    <joint name="${name}_laser_joint" type="fixed">
+      <origin xyz="0 0 0.058" />
+      <parent link="${name}_link"/>
+      <child link="${name}_laser_link"/>
+    </joint>
+    <link name="${name}_laser_link" type="laser">
+      <inertial>
+        <mass value="0.001" />
+        <origin xyz="0 0 0" rpy="0 0 0" />
+        <inertia ixx="0.0001" ixy="0" ixz="0" iyy="0.000001" iyz="0" izz="0.0001" />
+      </inertial>
     </link>
     <!-- gazebo extensions -->
-    <xacro:hokuyo_04lx_laser_gazebo name="${name}" ros_topic="${ros_topic}" update_rate="${update_rate}" min_angle="${min_angle}" max_angle="${max_angle}" />
+    <xacro:hokuyo_04lx_laser_gazebo name="${name}_laser" ros_topic="${ros_topic}" update_rate="${update_rate}" min_angle="${min_angle}" max_angle="${max_angle}" />
   </xacro:macro>
 </root>

File: segbot_description/urdf/sensors/kinect_camera.gazebo.xacro (robot description, xacro)
@@ -5,6 +5,6 @@
       xmlns:xacro="http://ros.org/wiki/xacro">
 <xacro:macro name="kinect_camera_gazebo" params="name">
-  <gazebo reference="${name}_frame">
-    <sensor:camera name="${name}_frame_sensor">
+  <gazebo reference="${name}_link">
+    <sensor:camera name="${name}_link_sensor">
       <imageFormat>R8G8B8</imageFormat>
       <imageSize>640 480</imageSize>
@@ -18,6 +18,6 @@
         <updateRate>20.0</updateRate>
         <cameraName>${name}</cameraName>
-        <imageTopicName>${name}/ir/image_raw</imageTopicName>
-        <cameraInfoTopicName>${name}/ir/camera_info</cameraInfoTopicName>
+        <imageTopicName>${name}/rgb/image_raw</imageTopicName>
+        <cameraInfoTopicName>${name}/rgb/camera_info</cameraInfoTopicName>
         <depthImageTopicName>${name}/depth/image_raw</depthImageTopicName>
         <depthImageInfoTopicName>${name}/depth/camera_info</depthImageInfoTopicName>

File: segbot_description/urdf/sensors/kinect_camera.urdf.xacro (robot description, xacro)
@@ -25,5 +25,4 @@
         </geometry>
       </visual>
-<!--
       <collision>
         <origin xyz="0.0 0.012 0" rpy="0 0 0"/>
@@ -32,5 +31,4 @@
         </geometry>
       </collision>
--->
     </link>
     <!-- extensions -->

Commit message: still trying to get simulator rendering to work

File: segbot_description/urdf/components/aluminium_sheet.urdf.xacro (robot description, xacro)
@@ -31,4 +31,8 @@
     <gazebo reference="${name}_link">
       <material>Gazebo/Grey</material>
+      <mu1 value="100.0" />
+      <mu2 value="100.0" />
+      <kp value="1000000.0" />
+      <kd value="1.0" />
     </gazebo>
   </xacro:macro>

File: segbot_description/urdf/components/beam_8020.urdf.xacro (robot description, xacro)
@@ -13,5 +13,4 @@
       <inertial>
         <mass value="0.1" />
-        <origin xyz="0 0 0" rpy="0 0 0"/>
         <inertia ixx="0.01"  ixy="0.0"  ixz="0.0"
                  iyy="0.01"  iyz="0.0"
@@ -34,4 +33,8 @@
     <gazebo reference="${name}_link">
       <material>Gazebo/Grey</material>
+      <mu1 value="100.0" />
+      <mu2 value="100.0" />
+      <kp value="1000000.0" />
+      <kd value="1.0" />
     </gazebo>
   </xacro:macro>

File: segbot_description/urdf/components/standoff_632.urdf.xacro (robot description, xacro)
@@ -31,4 +31,8 @@
     <gazebo reference="${name}_link">
       <material>Gazebo/Grey</material>
+      <mu1 value="100.0" />
+      <mu2 value="100.0" />
+      <kp value="1000000.0" />
+      <kd value="1.0" />
     </gazebo>
   </xacro:macro>
