Commit message: updating xml syntax based on current status of patch

File: segbot_description/urdf/components/laptop.urdf.xacro (robot description, xacro)
@@ -1,4 +1,7 @@
 <?xml version="1.0"?>
-<root xmlns:xacro="http://ros.org/wiki/xacro">
+<root xmlns:sensor="http://playerstage.sourceforge.net/gazebo/xmlschema/#sensor"
+      xmlns:controller="http://playerstage.sourceforge.net/gazebo/xmlschema/#controller"
+      xmlns:interface="http://playerstage.sourceforge.net/gazebo/xmlschema/#interface"
+      xmlns:xacro="http://ros.org/wiki/xacro">
   <xacro:macro name="laptop" params="name parent *origin">
     <!-- laptop base -->
@@ -19,5 +22,5 @@
         <origin xyz="0 0 ${0.375*INCH_TO_M}" rpy="0 0 0"/>
         <geometry>
-          <box size="${10*INCH_TO_M} ${13*INCH_TO_M} ${0.75*INCH_TO_M}" />
+          <box size="${9*INCH_TO_M} ${12*INCH_TO_M} ${0.75*INCH_TO_M}" />
         </geometry>
         <material name="almost_black" />
@@ -34,5 +37,5 @@
     <!-- laptop screen -->
     <joint name="${name}_screen_joint" type="fixed">
-      <origin xyz="${5*INCH_TO_M} 0 ${0.75*INCH_TO_M}" rpy="0 -${M_PI/3} 0"/>
+      <origin xyz="${4.5*INCH_TO_M} 0 ${0.75*INCH_TO_M}" rpy="0 -${M_PI/3} 0"/>
       <parent link="${name}_link" />
       <child link="${name}_screen_link" />
@@ -47,7 +50,7 @@
       </inertial>
       <visual>
-        <origin xyz="${5*INCH_TO_M} 0 -${0.375*INCH_TO_M}" rpy="0 0 0"/>
+        <origin xyz="${4.5*INCH_TO_M} 0 -${0.375*INCH_TO_M}" rpy="0 0 -${M_PI/2}"/>
         <geometry>
-          <box size="${10*INCH_TO_M} ${13*INCH_TO_M} ${0.75*INCH_TO_M}" />
+          <box size="${12*INCH_TO_M} ${9*INCH_TO_M} ${0.75*INCH_TO_M}" />
         </geometry>
         <material name="almost_black" />
@@ -56,9 +59,11 @@
     </link>
     <gazebo reference="${name}_screen_link">
-      <plugin name="${name}_video_controller" filename="libgazebo_ros_video.so">
-        <height>240</height>
-        <width>320</width>
-        <topicName>image_raw</topicName>
-      </plugin>
+      <visual>
+        <controller:laptop_visual_plugin name="${name}_video_controller" filename="libgazebo_ros_video.so">
+          <height>120</height>
+          <width>160</width>
+          <topicName>image</topicName>
+        </controller:laptop_visual_plugin>
+    </visual>
       <material>Gazebo/Grey</material>
       <mu1 value="100.0" />

Commit message: commenting out video controller while gazebo issues being sorted out

File: segbot_description/urdf/components/laptop.urdf.xacro (robot description, xacro)
@@ -59,11 +59,11 @@
     </link>
     <gazebo reference="${name}_screen_link">
-      <visual>
-        <plugin name="${name}_video_controller" filename="libgazebo_ros_video.so">
-          <height>120</height>
-          <width>160</width>
-          <topicName>image</topicName>
-        </plugin>
-      </visual>
+      <!-- <visual> -->
+      <!--   <plugin name="${name}_video_controller" filename="libgazebo_ros_video.so"> -->
+      <!--     <height>120</height> -->
+      <!--     <width>160</width> -->
+      <!--     <topicName>image</topicName> -->
+      <!--   </plugin> -->
+      <!-- </visual> -->
       <material>Gazebo/Grey</material>
       <mu1 value="100.0" />

Commit message: temporarily bypassing visual plugin hanndling as visual plugins are not handled in gazebo

File: segbot_description/urdf/components/laptop.urdf.xacro (robot description, xacro)
@@ -59,4 +59,18 @@
     </link>
     <gazebo reference="${name}_screen_link">
+      <!-- TODO fix this once visual plugins are parsed in urdf -->
+      <visual name="base_footprint_visuallaptop_screen_link_controller">
+        <pose>0.217799 -0.000000 1.082250 1.047200 0.000000 -1.570800</pose>
+        <geometry>
+          <box>
+            <size>0.304800 0.228600 0.019050</size>
+          </box>
+        </geometry>
+        <plugin name="${name}_video_controller" filename="libgazebo_ros_video.so">
+          <height>120</height>
+          <width>160</width>
+          <topicName>image</topicName>
+        </plugin>
+      </visual>
       <!-- <visual> -->
       <!--   <plugin name="${name}_video_controller" filename="libgazebo_ros_video.so"> -->

Commit message: video plugin works as expected with patched gazebo

File: segbot_description/urdf/components/laptop.urdf.xacro (robot description, xacro)
@@ -59,12 +59,5 @@
     </link>
     <gazebo reference="${name}_screen_link">
-      <!-- TODO fix this once visual plugins are parsed in urdf -->
-      <visual name="base_footprint_visuallaptop_screen_link_controller">
-        <pose>0.217799 -0.000000 1.082250 1.047200 0.000000 -1.570800</pose>
-        <geometry>
-          <box>
-            <size>0.304800 0.228600 0.019050</size>
-          </box>
-        </geometry>
+      <visual>
         <plugin name="${name}_video_controller" filename="libgazebo_ros_video.so">
           <height>120</height>
@@ -73,11 +66,4 @@
         </plugin>
       </visual>
-      <!-- <visual> -->
-      <!--   <plugin name="${name}_video_controller" filename="libgazebo_ros_video.so"> -->
-      <!--     <height>120</height> -->
-      <!--     <width>160</width> -->
-      <!--     <topicName>image</topicName> -->
-      <!--   </plugin> -->
-      <!-- </visual> -->
       <material>Gazebo/Grey</material>
       <mu1 value="100.0" />

Commit message: reverting laptop fix while patch propogates to system gazebo release

File: segbot_description/urdf/components/laptop.urdf.xacro (robot description, xacro)
@@ -59,5 +59,12 @@
     </link>
     <gazebo reference="${name}_screen_link">
-      <visual>
+      <!-- TODO fix this once visual plugins are parsed in urdf -->
+      <visual name="base_footprint_visuallaptop_screen_link_controller">
+        <pose>0.217799 -0.000000 1.082250 1.047200 0.000000 -1.570800</pose>
+        <geometry>
+          <box>
+            <size>0.304800 0.228600 0.019050</size>
+          </box>
+        </geometry>
         <plugin name="${name}_video_controller" filename="libgazebo_ros_video.so">
           <height>120</height>
@@ -66,4 +73,11 @@
         </plugin>
       </visual>
+      <!-- <visual> -->
+      <!--   <plugin name="${name}_video_controller" filename="libgazebo_ros_video.so"> -->
+      <!--     <height>120</height> -->
+      <!--     <width>160</width> -->
+      <!--     <topicName>image</topicName> -->
+      <!--   </plugin> -->
+      <!-- </visual> -->
       <material>Gazebo/Grey</material>
       <mu1 value="100.0" />

Commit message: added keyboard teleop script from teleop_twist_keyboard

File: segbot_description/urdf/components/laptop.urdf.xacro (robot description, xacro)
@@ -60,11 +60,18 @@
     <gazebo reference="${name}_screen_link">
       <!-- TODO fix this once visual plugins are parsed in urdf -->
-      <visual name="base_footprint_visuallaptop_screen_link_controller">
-        <pose>0.217799 -0.000000 1.082250 1.047200 0.000000 -1.570800</pose>
-        <geometry>
-          <box>
-            <size>0.304800 0.228600 0.019050</size>
-          </box>
-        </geometry>
+      <!-- <visual name="base_footprint_visuallaptop_screen_link_controller"> -->
+      <!--   <pose>0.217799 -0.000000 1.082250 1.047200 0.000000 -1.570800</pose> -->
+      <!--   <geometry> -->
+      <!--     <box> -->
+      <!--       <size>0.304800 0.228600 0.019050</size> -->
+      <!--     </box> -->
+      <!--   </geometry> -->
+      <!--   <plugin name="${name}_video_controller" filename="libgazebo_ros_video.so"> -->
+      <!--     <height>120</height> -->
+      <!--     <width>160</width> -->
+      <!--     <topicName>image</topicName> -->
+      <!--   </plugin> -->
+      <!-- </visual> -->
+      <visual>
         <plugin name="${name}_video_controller" filename="libgazebo_ros_video.so">
           <height>120</height>
@@ -73,11 +80,4 @@
         </plugin>
       </visual>
-      <!-- <visual> -->
-      <!--   <plugin name="${name}_video_controller" filename="libgazebo_ros_video.so"> -->
-      <!--     <height>120</height> -->
-      <!--     <width>160</width> -->
-      <!--     <topicName>image</topicName> -->
-      <!--   </plugin> -->
-      <!-- </visual> -->
       <material>Gazebo/Grey</material>
       <mu1 value="100.0" />

Commit message: reverting visual plugin change until pull request makes it to gazebo

File: segbot_description/urdf/components/laptop.urdf.xacro (robot description, xacro)
@@ -60,11 +60,18 @@
     <gazebo reference="${name}_screen_link">
       <!-- TODO fix this once visual plugins are parsed in urdf -->
-      <!-- <visual name="base_footprint_visuallaptop_screen_link_controller"> -->
-      <!--   <pose>0.217799 -0.000000 1.082250 1.047200 0.000000 -1.570800</pose> -->
-      <!--   <geometry> -->
-      <!--     <box> -->
-      <!--       <size>0.304800 0.228600 0.019050</size> -->
-      <!--     </box> -->
-      <!--   </geometry> -->
+      <visual name="base_footprint_visuallaptop_screen_link_controller">
+        <pose>0.217799 -0.000000 1.082250 1.047200 0.000000 -1.570800</pose>
+        <geometry>
+          <box>
+            <size>0.304800 0.228600 0.019050</size>
+          </box>
+        </geometry>
+        <plugin name="${name}_video_controller" filename="libgazebo_ros_video.so">
+          <height>120</height>
+          <width>160</width>
+          <topicName>image</topicName>
+        </plugin>
+      </visual>
+      <!-- <visual> -->
       <!--   <plugin name="${name}_video_controller" filename="libgazebo_ros_video.so"> -->
       <!--     <height>120</height> -->
@@ -73,11 +80,4 @@
       <!--   </plugin> -->
       <!-- </visual> -->
-      <visual>
-        <plugin name="${name}_video_controller" filename="libgazebo_ros_video.so">
-          <height>120</height>
-          <width>160</width>
-          <topicName>image</topicName>
-        </plugin>
-      </visual>
       <material>Gazebo/Grey</material>
       <mu1 value="100.0" />

Commit message: changed laptop lid angle such that it is now at a 45 degree angle

File: segbot_description/urdf/components/laptop.urdf.xacro (robot description, xacro)
@@ -37,5 +37,5 @@
     <!-- laptop screen -->
     <joint name="${name}_screen_joint" type="fixed">
-      <origin xyz="${4.5*INCH_TO_M} 0 ${0.75*INCH_TO_M}" rpy="0 -${21/48*M_PI} 0"/>
+      <origin xyz="${4.5*INCH_TO_M} 0 ${0.75*INCH_TO_M}" rpy="0 -${24/48*M_PI} 0"/>
       <parent link="${name}_link" />
       <child link="${name}_screen_link" />
