Commit message: fixed the kinect based robot description files

File: segbot_description/robots/segbot_full_kinect.urdf.xacro (robot description, xacro)
@@ -1,7 +1,4 @@
 <?xml version="1.0"?>
-<robot name="segbot"
-  xmlns:sensor="http://playerstage.sourceforge.net/gazebo/xmlschema/#sensor"
-  xmlns:controller="http://playerstage.sourceforge.net/gazebo/xmlschema/#controller"
-  xmlns:interface="http://playerstage.sourceforge.net/gazebo/xmlschema/#interface">
+<robot name="segbot">
   <!-- Included URDF Files -->
   <include filename="$(find segbot_description)/urdf/gazebo.xacro" />
@@ -9,4 +6,10 @@
   <property name="M_PI" value="3.14159"/>
   <property name="SCALE" value="0.0254"/>
+  <!-- Add the segbot base -->
   <segbot />
+  <!-- Add the forward facing kinect sensor for navigation -->
+  <include filename="$(find segbot_description)/urdf/sensors/kinect_camera.urdf.xacro" />
+  <kinect_camera name="nav_kinect" parent="base_link">
+    <origin xyz="0 0 0.3" rpy="0 0 0" />
+  </kinect_camera>
 </robot>

File: segbot_description/robots/segbot_simple_kinect.urdf.xacro (robot description, xacro)
@@ -1,7 +1,4 @@
 <?xml version="1.0"?>
-<robot name="segbot"
-  xmlns:sensor="http://playerstage.sourceforge.net/gazebo/xmlschema/#sensor"
-  xmlns:controller="http://playerstage.sourceforge.net/gazebo/xmlschema/#controller"
-  xmlns:interface="http://playerstage.sourceforge.net/gazebo/xmlschema/#interface">
+<robot name="segbot">
   <!-- Included URDF Files -->
   <include filename="$(find segbot_description)/urdf/gazebo_simple.xacro" />
@@ -9,4 +6,10 @@
   <property name="M_PI" value="3.14159"/>
   <property name="SCALE" value="0.0254"/>
+  <!-- Add the segbot base -->
   <segbot />
+  <!-- Add the forward facing kinect sensor for navigation -->
+  <include filename="$(find segbot_description)/urdf/sensors/kinect_camera.urdf.xacro" />
+  <kinect_camera name="nav_kinect" parent="base_link">
+    <origin xyz="0 0 0.3" rpy="0 0 0" />
+  </kinect_camera>
 </robot>

Commit message: fixed some inconsistencies in frame ids for the kinect based robot

File: segbot_description/robots/segbot_full_kinect.urdf.xacro (robot description, xacro)
@@ -10,5 +10,5 @@
   <!-- Add the forward facing kinect sensor for navigation -->
   <include filename="$(find segbot_description)/urdf/sensors/kinect_camera.urdf.xacro" />
-  <kinect_camera name="nav_kinect" parent="base_link">
+  <kinect_camera name="nav_kinect" parent="base">
     <origin xyz="0 0 0.3" rpy="0 0 0" />
   </kinect_camera>

File: segbot_description/robots/segbot_simple_kinect.urdf.xacro (robot description, xacro)
@@ -10,5 +10,5 @@
   <!-- Add the forward facing kinect sensor for navigation -->
   <include filename="$(find segbot_description)/urdf/sensors/kinect_camera.urdf.xacro" />
-  <kinect_camera name="nav_kinect" parent="base_link">
+  <kinect_camera name="nav_kinect" parent="base">
     <origin xyz="0 0 0.3" rpy="0 0 0" />
   </kinect_camera>

File: segbot_description/urdf/sensors/kinect_camera.urdf.xacro (robot description, xacro)
@@ -8,8 +8,8 @@
     <joint name="${name}_frame_joint" type="fixed">
       <insert_block name="origin" />
-      <parent link="${parent}"/>
-      <child link="${name}_frame"/>
+      <parent link="${parent}_link"/>
+      <child link="${name}_link"/>
     </joint>
-    <link name="${name}_frame">
+    <link name="${name}_link">
       <inertial>
         <mass value="0.1" />
@@ -25,4 +25,5 @@
         </geometry>
       </visual>
+<!--
       <collision>
         <origin xyz="0.0 0.012 0" rpy="0 0 0"/>
@@ -31,12 +32,6 @@
         </geometry>
       </collision>
+-->
     </link>
-    <joint name="${name}_optical_joint" type="fixed">
-      <origin xyz="0 0 0"
-                rpy="${-M_PI/2} 0 ${-M_PI/2}" />
-      <parent link="${name}_frame"/>
-      <child link="${name}_optical_frame"/>
-    </joint>
-    <link name="${name}_optical_frame"/>
     <!-- extensions -->
     <xacro:kinect_camera_gazebo name="${name}" />

Commit message: modified default configurations to use new base and chassis macros

File: segbot_description/robots/segbot_full_kinect.urdf.xacro (robot description, xacro)
@@ -2,14 +2,17 @@
 <robot name="segbot">
   <!-- Included URDF Files -->
+  <include filename="$(find segbot_description)/urdf/common.urdf.xacro" />
   <include filename="$(find segbot_description)/urdf/gazebo.xacro" />
   <include filename="$(find segbot_description)/urdf/segbot_base.xacro" />
-  <property name="M_PI" value="3.14159"/>
-  <property name="SCALE" value="0.0254"/>
+  <include filename="$(find segbot_description)/urdf/segbot_chassis.urdf.xacro" />
   <!-- Add the segbot base -->
   <segbot />
+  <segbot_chassis parent="base">
+    <origin xyz="-${2*INCH_TO_M} 0 ${4.25*INCH_TO_M}"/>
+  </segbot_chassis>
   <!-- Add the forward facing kinect sensor for navigation -->
-  <include filename="$(find segbot_description)/urdf/sensors/kinect_camera.urdf.xacro" />
-  <kinect_camera name="nav_kinect" parent="base">
-    <origin xyz="0 0 0.3" rpy="0 0 0" />
-  </kinect_camera>
+  <include filename="$(find segbot_description)/urdf/mounts/kinect_mount.urdf.xacro" />
+  <kinect_mount name="nav_kinect" parent="back_right_vertical_beam" length="${10.75*INCH_TO_M}">
+    <origin xyz="0 ${0.5*INCH_TO_M} ${4*INCH_TO_M}" rpy="-${M_PI/2} -${M_PI/2} 0" />
+  </kinect_mount>
 </robot>

File: segbot_description/robots/segbot_simple_hokuyo.urdf.xacro (robot description, xacro)
@@ -2,14 +2,17 @@
 <robot name="segbot">
   <!-- Included URDF Files -->
+  <include filename="$(find segbot_description)/urdf/common.urdf.xacro" />
   <include filename="$(find segbot_description)/urdf/gazebo_simple.xacro" />
   <include filename="$(find segbot_description)/urdf/segbot_base.xacro" />
-  <property name="M_PI" value="3.14159"/>
-  <property name="SCALE" value="0.0254"/>
+  <include filename="$(find segbot_description)/urdf/segbot_chassis.urdf.xacro" />
   <!-- Add the segbot base -->
   <segbot />
-  <!-- Add the forward facing kinect sensor for navigation -->
-  <include filename="$(find segbot_description)/urdf/sensors/hokuyo_04lx_laser.urdf.xacro" />
-  <hokuyo_04lx_laser name="nav_hokuyo" parent="base" ros_topic="scan" update_rate="10" min_angle="${-M_PI/2}" max_angle="${M_PI/2}">
-    <origin xyz="0.12 0 0.25" rpy="0 0 0" />
-  </hokuyo_04lx_laser>
+  <segbot_chassis parent="base">
+    <origin xyz="-${2*INCH_TO_M} 0 ${4.25*INCH_TO_M}"/>
+  </segbot_chassis>
+  <!-- Add the hokuyo -->
+  <include filename="$(find segbot_description)/urdf/mounts/hokuyo_mount.urdf.xacro" />
+  <hokuyo_mount name="nav_hokuyo" parent="front_right_vertical_beam" length="${10.75*INCH_TO_M}" ros_topic="scan" update_rate="10" min_angle="${-M_PI/2}" max_angle="${M_PI/2}">
+    <origin xyz="0 ${0.5*INCH_TO_M} ${4*INCH_TO_M}" rpy="-${M_PI/2} -${M_PI/2} 0" />
+  </hokuyo_mount>
 </robot>

File: segbot_description/robots/segbot_simple_kinect.urdf.xacro (robot description, xacro)
@@ -2,14 +2,17 @@
 <robot name="segbot">
   <!-- Included URDF Files -->
+  <include filename="$(find segbot_description)/urdf/common.urdf.xacro" />
   <include filename="$(find segbot_description)/urdf/gazebo_simple.xacro" />
   <include filename="$(find segbot_description)/urdf/segbot_base.xacro" />
-  <property name="M_PI" value="3.14159"/>
-  <property name="SCALE" value="0.0254"/>
+  <include filename="$(find segbot_description)/urdf/segbot_chassis.urdf.xacro" />
   <!-- Add the segbot base -->
   <segbot />
+  <segbot_chassis parent="base">
+    <origin xyz="-${2*INCH_TO_M} 0 ${4.25*INCH_TO_M}"/>
+  </segbot_chassis>
   <!-- Add the forward facing kinect sensor for navigation -->
-  <include filename="$(find segbot_description)/urdf/sensors/kinect_camera.urdf.xacro" />
-  <kinect_camera name="nav_kinect" parent="base">
-    <origin xyz="0 0 0.3" rpy="0 0 0" />
-  </kinect_camera>
+  <include filename="$(find segbot_description)/urdf/mounts/kinect_mount.urdf.xacro" />
+  <kinect_mount name="nav_kinect" parent="back_right_vertical_beam" length="${10.75*INCH_TO_M}">
+    <origin xyz="0 ${0.5*INCH_TO_M} ${4*INCH_TO_M}" rpy="-${M_PI/2} -${M_PI/2} 0" />
+  </kinect_mount>
 </robot>
