Commit message: The standard segbot kinect configuration now works on real hardware

File: segbot_description/robots/segbot_kinect.urdf.xacro (robot description, xacro)
@@ -14,6 +14,6 @@
   </xacro:segbot_chassis>
   <!-- Add the forward facing kinect sensor for navigation -->
-  <xacro:kinect_mount name="nav_kinect" parent="back_right_vertical_beam" length="${SENSOR_BEAM_LENGTH*INCH_TO_M}">
-    <origin xyz="0 ${0.5*INCH_TO_M} ${4*INCH_TO_M}" rpy="-${M_PI/2} -${M_PI/2} 0" />
+  <xacro:kinect_mount name="nav_kinect" parent="front_right_vertical_beam" length="${SENSOR_BEAM_LENGTH*INCH_TO_M}">
+    <origin xyz="0 ${0.5*INCH_TO_M} ${17.5*INCH_TO_M}" rpy="-${M_PI/2} -${M_PI/2} 0" />
   </xacro:kinect_mount>
   <xacro:gazebo_segbot_ros_controllers />
