Commit message: removing segbot_iriss and readding segbot (i.e. w/o sensors) configuration file

File: segbot_description/robots/segbot.urdf.xacro (robot description, xacro)
@@ -13,8 +13,4 @@
     <origin xyz="${BASE_PLATE_X_OFFSET*INCH_TO_M} 0 ${BASE_PLATE_Z_OFFSET*INCH_TO_M}"/>
   </xacro:segbot_chassis>
-  <!-- Add the forward facing kinect sensor for navigation -->
-  <xacro:kinect_mount name="nav_kinect" parent="back_right_vertical_beam" length="${SENSOR_BEAM_LENGTH*INCH_TO_M}">
-    <origin xyz="0 ${0.5*INCH_TO_M} ${7.875*INCH_TO_M}" rpy="-${M_PI/2} -${M_PI/2} 0" />
-  </xacro:kinect_mount>
   <xacro:gazebo_segbot_ros_controllers />
 </robot>
