Commit message: segbot_description: coordinate corrections for sensor_mount and hokuyo

File: segbot_description/robots/segbot_default.xacro (robot description, xacro)
@@ -27,5 +27,5 @@
                       ros_topic="scan" update_rate="10"
                       min_angle="${-(5 * M_PI)/12}" max_angle="${(5 * M_PI)/12}">
-    <origin xyz="0 -${0.5*INCH_TO_M} ${6*INCH_TO_M}" rpy="${M_PI/2} ${M_PI/2} 0" />
+    <origin xyz="0 -${0.5*INCH_TO_M} ${7*INCH_TO_M}" rpy="${M_PI/2} ${M_PI/2} 0" />
   </xacro:hokuyo_mount>
   <xacro:gazebo_segbot_ros_controllers />

File: segbot_description/urdf/mounts/sensor_mount.urdf.xacro (robot description, xacro)
@@ -7,19 +7,19 @@
     <!-- add sensor mount plate and its standoffs -->
     <xacro:standoff_632 name="${name}_front_left_standoff" parent="${parent}"
-                        length="${0.5*INCH_TO_M}">
-      <origin xyz="${4.25*INCH_TO_M} ${4.5*INCH_TO_M} ${(1/32)*INCH_TO_M}"
+                        length="${1.5*INCH_TO_M}">
+      <origin xyz="${3.25*INCH_TO_M} ${4.5*INCH_TO_M} ${(1/32)*INCH_TO_M}"
               rpy="0 0 0" />
     </xacro:standoff_632>
     <xacro:standoff_632 name="${name}_front_right_standoff" parent="${parent}"
-                        length="${0.5*INCH_TO_M}">
-      <origin xyz="${4.25*INCH_TO_M} ${-4.5*INCH_TO_M} ${(1/32)*INCH_TO_M}" rpy="0 0 0" />
+                        length="${1.5*INCH_TO_M}">
+      <origin xyz="${3.25*INCH_TO_M} ${-4.5*INCH_TO_M} ${(1/32)*INCH_TO_M}" rpy="0 0 0" />
     </xacro:standoff_632>
     <xacro:standoff_632 name="${name}_back_left_standoff" parent="${parent}"
-                        length="${0.5*INCH_TO_M}">
-      <origin xyz="${2.25*INCH_TO_M} ${4.5*INCH_TO_M} ${(1/32)*INCH_TO_M}" rpy="0 0 0" />
+                        length="${1.5*INCH_TO_M}">
+      <origin xyz="${1.25*INCH_TO_M} ${4.5*INCH_TO_M} ${(1/32)*INCH_TO_M}" rpy="0 0 0" />
     </xacro:standoff_632>
     <xacro:standoff_632 name="${name}_back_right_standoff" parent="${parent}"
-                        length="${0.5*INCH_TO_M}">
-      <origin xyz="${2.25*INCH_TO_M} ${-4.5*INCH_TO_M} ${(1/32)*INCH_TO_M}" rpy="0 0 0" />
+                        length="${1.5*INCH_TO_M}">
+      <origin xyz="${1.25*INCH_TO_M} ${-4.5*INCH_TO_M} ${(1/32)*INCH_TO_M}" rpy="0 0 0" />
     </xacro:standoff_632>
     <xacro:aluminium_sheet name="${name}_plate"
@@ -28,5 +28,5 @@
                            length="${5.875*INCH_TO_M}"
                            width="${9.5*INCH_TO_M}">
-      <origin xyz="${-(11/16)*INCH_TO_M} ${-4.5*INCH_TO_M} ${(17/32)*INCH_TO_M}"
+      <origin xyz="${(11/16)*INCH_TO_M} ${-4.5*INCH_TO_M} ${(1.5+1/32)*INCH_TO_M}"
               rpy="0 0 0" />
     </xacro:aluminium_sheet>
@@ -35,20 +35,20 @@
                         parent="${name}_front_left_standoff"
                         length="${2*INCH_TO_M}">
-      <origin xyz="0 0 ${(1/16)*INCH_TO_M}" rpy="0 0 0" />
+      <origin xyz="0 0 ${(1.5+1/16)*INCH_TO_M}" rpy="0 0 0" />
     </xacro:standoff_632>
     <xacro:standoff_632 name="${name}_top_front_right_standoff"
                         parent="${name}_front_right_standoff"
                         length="${2*INCH_TO_M}">
-      <origin xyz="0 0 ${(1/16)*INCH_TO_M}" rpy="0 0 0" />
+      <origin xyz="0 0 ${(1.5+1/16)*INCH_TO_M}" rpy="0 0 0" />
     </xacro:standoff_632>
     <xacro:standoff_632 name="${name}_top_back_left_standoff"
                         parent="${name}_back_left_standoff"
                         length="${2*INCH_TO_M}">
-      <origin xyz="0 0 ${(1/16)*INCH_TO_M}" rpy="0 0 0" />
+      <origin xyz="0 0 ${(1.5+1/16)*INCH_TO_M}" rpy="0 0 0" />
     </xacro:standoff_632>
     <xacro:standoff_632 name="${name}_top_back_right_standoff"
                         parent="${name}_back_right_standoff"
                         length="${2*INCH_TO_M}">
-      <origin xyz="0 0 ${(1/16)*INCH_TO_M}" rpy="0 0 0" />
+      <origin xyz="0 0 ${(1.5+1/16)*INCH_TO_M}" rpy="0 0 0" />
     </xacro:standoff_632>
     <xacro:aluminium_sheet name="${name}_top_plate"
@@ -57,5 +57,5 @@
                            length="${5.875*INCH_TO_M}"
                            width="${9.5*INCH_TO_M}">
-      <origin xyz="${-(11/16)*INCH_TO_M} ${-4.5*INCH_TO_M} ${(2+1/32)*INCH_TO_M}"
+      <origin xyz="${(11/16)*INCH_TO_M} ${-4.5*INCH_TO_M} ${(2+1/32)*INCH_TO_M}"
               rpy="0 0 0" />
     </xacro:aluminium_sheet>
