Commit message: added some constants for appropriate values (i.e. values used in the final robot urdf files)

File: segbot_description/robots/segbot_hokuyo.urdf.xacro (robot description, xacro)
@@ -1,4 +1,5 @@
 <?xml version="1.0"?>
-<robot name="segbot">
+<robot name="segbot"
+       xmlns:xacro="http://ros.org/wiki/xacro">
   <!-- Included URDF Files -->
   <include filename="$(find segbot_description)/urdf/common.urdf.xacro" />
@@ -6,13 +7,13 @@
   <include filename="$(find segbot_description)/urdf/segbot_base.xacro" />
   <include filename="$(find segbot_description)/urdf/segbot_chassis.urdf.xacro" />
+  <include filename="$(find segbot_description)/urdf/mounts/hokuyo_mount.urdf.xacro" />
   <!-- Add the segbot base -->
-  <segbot />
-  <segbot_chassis parent="base">
-    <origin xyz="-${2*INCH_TO_M} 0 ${4.25*INCH_TO_M}"/>
-  </segbot_chassis>
+  <xacro:segbot />
+  <xacro:segbot_chassis parent="base">
+    <origin xyz="${BASE_PLATE_X_OFFSET*INCH_TO_M} 0 ${BASE_PLATE_Z_OFFSET*INCH_TO_M}"/>
+  </xacro:segbot_chassis>
   <!-- Add the hokuyo -->
-  <include filename="$(find segbot_description)/urdf/mounts/hokuyo_mount.urdf.xacro" />
-  <hokuyo_mount name="nav_hokuyo" parent="front_right_vertical_beam" length="${10.75*INCH_TO_M}" ros_topic="scan" update_rate="10" min_angle="${-M_PI/2}" max_angle="${M_PI/2}">
+  <xacro:hokuyo_mount name="nav_hokuyo" parent="front_right_vertical_beam" length="${SENSOR_BEAM_LENGTH*INCH_TO_M}" ros_topic="scan" update_rate="10" min_angle="${-M_PI/2}" max_angle="${M_PI/2}">
     <origin xyz="0 ${0.5*INCH_TO_M} ${4*INCH_TO_M}" rpy="-${M_PI/2} -${M_PI/2} 0" />
-  </hokuyo_mount>
+  </xacro:hokuyo_mount>
 </robot>

File: segbot_description/robots/segbot_kinect.urdf.xacro (robot description, xacro)
@@ -1,4 +1,5 @@
 <?xml version="1.0"?>
-<robot name="segbot">
+<robot name="segbot"
+       xmlns:xacro="http://ros.org/wiki/xacro">
   <!-- Included URDF Files -->
   <include filename="$(find segbot_description)/urdf/common.urdf.xacro" />
@@ -6,13 +7,13 @@
   <include filename="$(find segbot_description)/urdf/segbot_base.xacro" />
   <include filename="$(find segbot_description)/urdf/segbot_chassis.urdf.xacro" />
+  <include filename="$(find segbot_description)/urdf/mounts/kinect_mount.urdf.xacro" />
   <!-- Add the segbot base -->
-  <segbot />
-  <segbot_chassis parent="base">
-    <origin xyz="-${2*INCH_TO_M} 0 ${4.25*INCH_TO_M}"/>
-  </segbot_chassis>
+  <xacro:segbot />
+  <xacro:segbot_chassis parent="base">
+    <origin xyz="${BASE_PLATE_X_OFFSET*INCH_TO_M} 0 ${BASE_PLATE_Z_OFFSET*INCH_TO_M}"/>
+  </xacro:segbot_chassis>
   <!-- Add the forward facing kinect sensor for navigation -->
-  <include filename="$(find segbot_description)/urdf/mounts/kinect_mount.urdf.xacro" />
-  <kinect_mount name="nav_kinect" parent="back_right_vertical_beam" length="${10.75*INCH_TO_M}">
+  <xacro:kinect_mount name="nav_kinect" parent="back_right_vertical_beam" length="${SENSOR_BEAM_LENGTH*INCH_TO_M}">
     <origin xyz="0 ${0.5*INCH_TO_M} ${4*INCH_TO_M}" rpy="-${M_PI/2} -${M_PI/2} 0" />
-  </kinect_mount>
+  </xacro:kinect_mount>
 </robot>

File: segbot_description/urdf/common.urdf.xacro (robot description, xacro)
@@ -1,12 +1,20 @@
 <?xml version="1.0"?>
 <root xmlns:xacro="http://ros.org/wiki/xacro">
-  <!-- constants -->
-  <xacro:property name="M_PI" value="3.14159"/>
+  <!-- generic constants -->
+  <xacro:property name="M_PI" value="3.14159265359" />
   <xacro:property name="INCH_TO_M" value="0.0254"/>
+  <!-- 80/20 constants -->
+  <xacro:property name="BEAM_WIDTH" value="1" /> <!-- inches -->
+  <!-- robot constants -->
+  <!-- distance between the robot origin and the base plate center along the x axis (robot forward) -->
+  <xacro:property name="BASE_PLATE_X_OFFSET" value="-2" /> <!-- inches -->
+  <!-- distance between the robot origin and the bottom of the base plate along the z axis (robot up) -->
+  <xacro:property name="BASE_PLATE_Z_OFFSET" value="4.25" /> <!-- inches -->
+  <xacro:property name="SENSOR_BEAM_LENGTH" value="10.75" /> <!-- inches -->
   <!-- colors -->
-  <material name="beam_grey">
+  <material name="light_grey">
     <color rgba="0.7 0.7 0.7 1" />
   </material>
-  <material name="sheet_grey">
+  <material name="dark_grey">
     <color rgba="0.5 0.5 0.5 1" />
   </material>

File: segbot_description/urdf/components/aluminium_sheet.urdf.xacro (robot description, xacro)
@@ -20,5 +20,5 @@
           <box size="${length} ${width} ${thickness}" />
         </geometry>
-        <material name="sheet_grey" />
+        <material name="dark_grey" />
       </visual>
     </link>

File: segbot_description/urdf/components/beam_8020.urdf.xacro (robot description, xacro)
@@ -23,5 +23,5 @@
           <box size="${1*INCH_TO_M} ${1*INCH_TO_M} ${length}" />
         </geometry>
-        <material name="beam_grey" />
+        <material name="light_grey" />
       </visual>
     </link>

File: segbot_description/urdf/components/standoff_632.urdf.xacro (robot description, xacro)
@@ -20,5 +20,5 @@
           <cylinder length="${length}" radius="0.003175" />
         </geometry>
-        <material name="beam_grey" />
+        <material name="light_grey" />
       </visual>
     </link>

Commit message: lowered height of hokuyo for simulation

File: segbot_description/robots/segbot_hokuyo.urdf.xacro (robot description, xacro)
@@ -15,5 +15,5 @@
   <!-- Add the hokuyo -->
   <xacro:hokuyo_mount name="nav_hokuyo" parent="front_right_vertical_beam" length="${SENSOR_BEAM_LENGTH*INCH_TO_M}" ros_topic="scan" update_rate="10" min_angle="${-M_PI/2}" max_angle="${M_PI/2}">
-    <origin xyz="0 ${0.5*INCH_TO_M} ${4*INCH_TO_M}" rpy="-${M_PI/2} -${M_PI/2} 0" />
+    <origin xyz="0 ${0.5*INCH_TO_M} ${2*INCH_TO_M}" rpy="-${M_PI/2} -${M_PI/2} 0" />
   </xacro:hokuyo_mount>
 </robot>

Commit message: updated segbot hokuyo configuration to inverted lidar position

File: segbot_description/robots/segbot_hokuyo.urdf.xacro (robot description, xacro)
@@ -14,6 +14,6 @@
   </xacro:segbot_chassis>
   <!-- Add the hokuyo -->
-  <xacro:hokuyo_mount name="nav_hokuyo" parent="front_right_vertical_beam" length="${SENSOR_BEAM_LENGTH*INCH_TO_M}" ros_topic="scan" update_rate="10" min_angle="${-M_PI/2}" max_angle="${M_PI/2}">
-    <origin xyz="0 ${0.5*INCH_TO_M} ${2*INCH_TO_M}" rpy="-${M_PI/2} -${M_PI/2} 0" />
+  <xacro:hokuyo_mount name="nav_hokuyo" parent="front_left_vertical_beam" length="${SENSOR_BEAM_LENGTH*INCH_TO_M}" ros_topic="scan" update_rate="10" min_angle="${-M_PI/2}" max_angle="${M_PI/2}">
+    <origin xyz="0 -${0.5*INCH_TO_M} ${4*INCH_TO_M}" rpy="${M_PI/2} ${M_PI/2} 0" />
   </xacro:hokuyo_mount>
 </robot>

Commit message: raising height of hokuyo to something that might be inaccurate. I am currently seeing returns from wheels in simulation

File: segbot_description/robots/segbot_hokuyo.urdf.xacro (robot description, xacro)
@@ -15,5 +15,5 @@
   <!-- Add the hokuyo -->
   <xacro:hokuyo_mount name="nav_hokuyo" parent="front_left_vertical_beam" length="${SENSOR_BEAM_LENGTH*INCH_TO_M}" ros_topic="scan" update_rate="10" min_angle="${-(5 * M_PI)/12}" max_angle="${(5 * M_PI)/12}">
-    <origin xyz="0 -${0.5*INCH_TO_M} ${4*INCH_TO_M}" rpy="${M_PI/2} ${M_PI/2} 0" />
+    <origin xyz="0 -${0.5*INCH_TO_M} ${6*INCH_TO_M}" rpy="${M_PI/2} ${M_PI/2} 0" />
   </xacro:hokuyo_mount>
   <xacro:gazebo_segbot_ros_controllers />

Commit message: segbot_description: correct height of hokuyo in other robots

File: segbot_description/robots/segbot_hokuyo.urdf.xacro (robot description, xacro)
@@ -15,5 +15,5 @@
   <!-- Add the hokuyo -->
   <xacro:hokuyo_mount name="nav_hokuyo" parent="front_left_vertical_beam" length="${SENSOR_BEAM_LENGTH*INCH_TO_M}" ros_topic="scan" update_rate="10" min_angle="${-(5 * M_PI)/12}" max_angle="${(5 * M_PI)/12}">
-    <origin xyz="0 -${0.5*INCH_TO_M} ${6*INCH_TO_M}" rpy="${M_PI/2} ${M_PI/2} 0" />
+    <origin xyz="0 -${0.5*INCH_TO_M} ${7*INCH_TO_M}" rpy="${M_PI/2} ${M_PI/2} 0" />
   </xacro:hokuyo_mount>
   <xacro:gazebo_segbot_ros_controllers />

File: segbot_description/robots/segbot_navigation.urdf.xacro (robot description, xacro)
@@ -20,5 +20,5 @@
   <!-- Add the hokuyo -->
   <xacro:hokuyo_mount name="nav_hokuyo" parent="front_left_vertical_beam" length="${SENSOR_BEAM_LENGTH*INCH_TO_M}" ros_topic="scan" update_rate="10" min_angle="${-(5 * M_PI)/12}" max_angle="${(5 * M_PI)/12}">
-    <origin xyz="0 -${0.5*INCH_TO_M} ${6*INCH_TO_M}" rpy="${M_PI/2} ${M_PI/2} 0" />
+    <origin xyz="0 -${0.5*INCH_TO_M} ${7*INCH_TO_M}" rpy="${M_PI/2} ${M_PI/2} 0" />
   </xacro:hokuyo_mount>
   <xacro:gazebo_segbot_ros_controllers />
