Commit message: updated and added segbot_v2.arm. fixed some issues with previous commit. closes #34.

File: segbot_description/robots/segbot_v1.hokuyo_only.urdf.xacro (robot description, xacro)
@@ -14,5 +14,5 @@
   </xacro:segbot_chassis>
   <!-- Add the hokuyo -->
-  <xacro:hokuyo_mount name="nav_hokuyo" parent="front_left_vertical_beam" length="${SENSOR_BEAM_LENGTH*INCH_TO_M}" ros_topic="scan" update_rate="10" min_angle="${-(5 * M_PI)/12}" max_angle="${(5 * M_PI)/12}">
+  <xacro:hokuyo_mount name="nav_hokuyo" parent="front_left_vertical_beam" length="${SENSOR_BEAM_LENGTH*INCH_TO_M}" ros_topic="scan" update_rate="10" min_angle="${-(5 * M_PI)/12}" max_angle="${(5 * M_PI)/12}" range="4.0">
     <origin xyz="0 -${0.5*INCH_TO_M} ${7*INCH_TO_M}" rpy="${M_PI/2} ${M_PI/2} 0" />
   </xacro:hokuyo_mount>

File: segbot_description/robots/segbot_v1.urdf.xacro (robot description, xacro)
@@ -19,5 +19,5 @@
   </xacro:kinect_mount>
   <!-- Add the hokuyo -->
-  <xacro:hokuyo_mount name="nav_hokuyo" parent="front_left_vertical_beam" length="${SENSOR_BEAM_LENGTH*INCH_TO_M}" ros_topic="scan" update_rate="10" min_angle="${-(5 * M_PI)/12}" max_angle="${(5 * M_PI)/12}">
+  <xacro:hokuyo_mount name="nav_hokuyo" parent="front_left_vertical_beam" length="${SENSOR_BEAM_LENGTH*INCH_TO_M}" ros_topic="scan" update_rate="10" min_angle="${-(5 * M_PI)/12}" max_angle="${(5 * M_PI)/12}" range="4.0">
     <origin xyz="0 -${0.5*INCH_TO_M} ${7*INCH_TO_M}" rpy="${M_PI/2} ${M_PI/2} 0" />
   </xacro:hokuyo_mount>

File: segbot_description/robots/segbot_v2.arm.urdf.xacro (robot description, xacro)
@@ -12,7 +12,7 @@
   <!-- Add the segbot base -->
   <xacro:segbot />
-  <xacro:segbot_chassis parent="base">
+  <xacro:segbot_chassis_arm parent="base">
     <origin xyz="${BASE_PLATE_X_OFFSET*INCH_TO_M} 0 ${BASE_PLATE_Z_OFFSET*INCH_TO_M}"/>
-  </xacro:segbot_chassis>
+  </xacro:segbot_chassis_arm>
   <!-- Add the forward facing kinect sensor for navigation -->
   <xacro:kinect_mount name="nav_kinect" parent="back_right_vertical_beam" length="${SENSOR_BEAM_LENGTH*INCH_TO_M}">
@@ -29,7 +29,15 @@
   <!-- Add the sensor plate mount -->
   <xacro:sensor_plate_mount_without_beam parent="hokuyo_sonar_sensor_beam" length="${SENSOR_BEAM_LENGTH*INCH_TO_M}"/>
-  <!-- Add a beam at top so that the robot looks complete. We'll probably have a different sensor mount here eventually. -->
-  <xacro:beam_8020 name="front_cap_beam" parent="front_right_vertical_beam" length="${SENSOR_BEAM_LENGTH*INCH_TO_M}">
-    <origin xyz="0 -${0.5*INCH_TO_M} ${36.5*INCH_TO_M}" rpy="-${M_PI/2} 0 0" />
+  <!-- Add the left sensor beam -->
+  <xacro:beam_8020 name="left_sensor_beam" parent="laptop_base_plate" length="${30*INCH_TO_M}">
+    <origin xyz="0 ${8.5*INCH_TO_M} ${0.125*INCH_TO_M}" rpy="0 0 0" />
+  </xacro:beam_8020>
+  <!-- Add the right sensor beam -->
+  <xacro:beam_8020 name="right_sensor_beam" parent="laptop_base_plate" length="${30*INCH_TO_M}">
+    <origin xyz="0 -${8.5*INCH_TO_M} ${0.125*INCH_TO_M}" rpy="0 0 0" />
+  </xacro:beam_8020>
+  <!-- Add the top sensor beam -->
+  <xacro:beam_8020 name="top_sensor_beam" parent="right_sensor_beam" length="${18*INCH_TO_M}">
+    <origin xyz="0 -${0.5*INCH_TO_M} ${30.5*INCH_TO_M}" rpy="-${M_PI/2} 0 0" />
   </xacro:beam_8020>
   <xacro:gazebo_segbot_ros_controllers />

File: segbot_description/urdf/mounts/sensor_plate_mount.urdf.xacro (robot description, xacro)
@@ -7,10 +7,10 @@
   <xacro:include filename="$(find segbot_description)/urdf/components/standoff.urdf.xacro" />
   <xacro:include filename="$(find segbot_description)/urdf/components/aluminium_sheet.urdf.xacro" />
-  <xacro:macro name="sensor_plate_mount_without_beam" params="parent length" />
-  <xacro:standoff name="left_sensor_plate_standoff" parent="${parent}" length="${0.5*INCH_TO_M}" radius="${0.25*INCH_TO_M}">
-      <origin xyz="-${1/2*INCH_TO_M} 0 ${length - 2.5*INCH_TO_M}" rpy="-${M_PI/2} 0 ${M_PI/2}" />
+  <xacro:macro name="sensor_plate_mount_without_beam" params="parent length">
+    <xacro:standoff name="left_sensor_plate_standoff" parent="${parent}" length="${0.5*INCH_TO_M}" radius="${0.25*INCH_TO_M}">
+      <origin xyz="-${1/2*INCH_TO_M} 0 ${length/2 - 2.5*INCH_TO_M}" rpy="-${M_PI/2} 0 ${M_PI/2}" />
     </xacro:standoff>
     <xacro:standoff name="right_sensor_plate_standoff" parent="${parent}" length="${0.5*INCH_TO_M}" radius="${0.25*INCH_TO_M}">
-      <origin xyz="-${1/2*INCH_TO_M} 0 ${length + 2.5*INCH_TO_M}" rpy="-${M_PI/2} 0 ${M_PI/2}" />
+      <origin xyz="-${1/2*INCH_TO_M} 0 ${length/2 + 2.5*INCH_TO_M}" rpy="-${M_PI/2} 0 ${M_PI/2}" />
     </xacro:standoff>
     <xacro:aluminium_sheet name="sensor_plate" parent="left_sensor_plate_standoff" thickness="0.003" length="${4.5*INCH_TO_M}" width="${9*INCH_TO_M}">
@@ -31,5 +31,5 @@
           izz="0.01" />
       </inertial>
-     <visual>
+      <visual>
         <origin xyz="0 0 0" rpy="0 0 0" />
         <geometry>
@@ -52,5 +52,5 @@
           izz="0.01" />
       </inertial>
-     <visual>
+      <visual>
         <origin xyz="0 0 0" rpy="0 0 0" />
         <geometry>
@@ -72,5 +72,5 @@
           izz="0.01" />
       </inertial>
-     <visual>
+      <visual>
         <origin xyz="0 0 0" rpy="0 0 0" />
         <geometry>
@@ -93,5 +93,5 @@
           izz="0.01" />
       </inertial>
-     <visual>
+      <visual>
         <origin xyz="0 0 0" rpy="0 0 0" />
         <geometry>
@@ -114,5 +114,5 @@
           izz="0.01" />
       </inertial>
-     <visual>
+      <visual>
         <origin xyz="0 0 0" rpy="0 0 0" />
         <geometry>
@@ -134,5 +134,5 @@
           izz="0.01" />
       </inertial>
-     <visual>
+      <visual>
         <origin xyz="0 0 0" rpy="0 0 0" />
         <geometry>

File: segbot_description/urdf/v2/segbot_chassis.urdf.xacro (robot description, xacro)
@@ -7,5 +7,5 @@
   <xacro:include filename="$(find segbot_description)/urdf/components/laptop.urdf.xacro" />
   <xacro:include filename="$(find segbot_description)/urdf/components/standoff.urdf.xacro" />
-  <xacro:macro name="segbot_chassis" params="parent *origin">
+  <xacro:macro name="segbot_chassis_parametrized" params="parent *origin front_vertical_beam_length back_vertical_beam_length laptop_plate_length laptop_plate_width">
     <!-- base plate -->
     <xacro:aluminium_sheet name="chassis_base_plate" parent="${parent}"
@@ -39,17 +39,17 @@
     </xacro:beam_8020>
     <!-- 80/20 vertical beams -->
-    <xacro:beam_8020 name="back_left_vertical_beam" parent="back_base_beam" length="${24*INCH_TO_M}">
+    <xacro:beam_8020 name="back_left_vertical_beam" parent="back_base_beam" length="${back_vertical_beam_length}">
       <origin xyz="0 0 ${0.5*INCH_TO_M}"
         rpy="-${M_PI/2} 0 0" />
     </xacro:beam_8020>
-    <xacro:beam_8020 name="front_left_vertical_beam" parent="front_base_beam" length="${36*INCH_TO_M}">
+    <xacro:beam_8020 name="front_left_vertical_beam" parent="front_base_beam" length="${front_vertical_beam_length}">
       <origin xyz="0 0 ${0.5*INCH_TO_M}"
         rpy="-${M_PI/2} 0 0" />
     </xacro:beam_8020>
-    <xacro:beam_8020 name="back_right_vertical_beam" parent="back_base_beam" length="${24*INCH_TO_M}">
+    <xacro:beam_8020 name="back_right_vertical_beam" parent="back_base_beam" length="${back_vertical_beam_length}">
       <origin xyz="0 0 ${11.5*INCH_TO_M}"
         rpy="-${M_PI/2} 0 0" />
     </xacro:beam_8020>
-    <xacro:beam_8020 name="front_right_vertical_beam" parent="front_base_beam" length="${36*INCH_TO_M}">
+    <xacro:beam_8020 name="front_right_vertical_beam" parent="front_base_beam" length="${front_vertical_beam_length}">
       <origin xyz="0 0 ${11.5*INCH_TO_M}"
         rpy="-${M_PI/2} 0 0" />
@@ -58,14 +58,14 @@
     <!-- left laptop support beam (from the back beam) -->
     <xacro:beam_8020 name="left_laptop_support_beam" parent="back_left_vertical_beam" length="${12*INCH_TO_M}">
-      <origin xyz="-${0.5*INCH_TO_M} ${1*INCH_TO_M} ${23.5*INCH_TO_M}"
+      <origin xyz="-${0.5*INCH_TO_M} ${1*INCH_TO_M} ${back_vertical_beam_length - 0.5*INCH_TO_M}"
         rpy="${M_PI} -${M_PI/2} 0" />
     </xacro:beam_8020>
     <xacro:beam_8020 name="right_laptop_support_beam" parent="back_right_vertical_beam" length="${12*INCH_TO_M}">
-      <origin xyz="-${0.5*INCH_TO_M} -${1*INCH_TO_M} ${23.5*INCH_TO_M}"
+      <origin xyz="-${0.5*INCH_TO_M} -${1*INCH_TO_M} ${back_vertical_beam_length - 0.5*INCH_TO_M}"
         rpy="${M_PI} -${M_PI/2} 0" />
     </xacro:beam_8020>
     <!-- laptop base plate -->
     <!-- from the left laptop support beam -->
-    <xacro:aluminium_sheet name="laptop_base_plate" parent="left_laptop_support_beam" thickness="${0.125*INCH_TO_M}" length="${12*INCH_TO_M}" width="${14*INCH_TO_M}">
+    <xacro:aluminium_sheet name="laptop_base_plate" parent="left_laptop_support_beam" thickness="${0.125*INCH_TO_M}" length="${laptop_plate_length}" width="${laptop_plate_width}">
       <origin xyz="${0.5*INCH_TO_M} ${6.5*INCH_TO_M} ${6*INCH_TO_M}"
         rpy="${M_PI} -${M_PI/2} 0" />
@@ -76,3 +76,17 @@
     </xacro:laptop>
   </xacro:macro>
+  <xacro:macro name="segbot_chassis" params="parent *origin">
+    <xacro:segbot_chassis_parametrized parent="${parent}" front_vertical_beam_length="${36*INCH_TO_M}"
+      back_vertical_beam_length="${24*INCH_TO_M}" laptop_plate_length="${12*INCH_TO_M}"
+      laptop_plate_width="${14*INCH_TO_M}">
+      <xacro:insert_block name="origin" />
+    </xacro:segbot_chassis_parametrized>
+  </xacro:macro>
+  <xacro:macro name="segbot_chassis_arm" params="parent *origin">
+    <xacro:segbot_chassis_parametrized parent="${parent}" front_vertical_beam_length="${18*INCH_TO_M}"
+      back_vertical_beam_length="${18*INCH_TO_M}" laptop_plate_length="${16*INCH_TO_M}"
+      laptop_plate_width="${18*INCH_TO_M}">
+      <xacro:insert_block name="origin" />
+    </xacro:segbot_chassis_parametrized>
+  </xacro:macro>
 </root>
