Commit message: Fixed position of sensors in urdf.

File: segbot_description/robots/segbot_v2.urdf.xacro (robot description, xacro)
@@ -16,9 +16,9 @@
   <!-- Add the forward facing kinect sensor for navigation -->
   <xacro:kinect_mount name="nav_kinect" parent="back_right_vertical_beam" length="${SENSOR_BEAM_LENGTH*INCH_TO_M}">
-    <origin xyz="-${1*INCH_TO_M} -${0.5*INCH_TO_M} ${12*INCH_TO_M}" rpy="-${M_PI/2} -${M_PI/2} 0" />
+    <origin xyz="${1*INCH_TO_M} -${0.5*INCH_TO_M} ${11.5*INCH_TO_M}" rpy="-${M_PI/2} -${M_PI/2} 0" />
   </xacro:kinect_mount>
   <!-- Add the hokuyo -->
   <xacro:hokuyo_mount name="nav_hokuyo" parent="front_left_vertical_beam" length="${SENSOR_BEAM_LENGTH*INCH_TO_M}" ros_topic="scan" update_rate="10" min_angle="${-(5 * M_PI)/12}" max_angle="${(5 * M_PI)/12}">
-    <origin xyz="${1*INCH_TO_M} ${0.5*INCH_TO_M} ${5*INCH_TO_M}" rpy="${M_PI/2} ${M_PI/2} 0" />
+    <origin xyz="${1*INCH_TO_M} ${0.5*INCH_TO_M} ${4.5*INCH_TO_M}" rpy="${M_PI/2} ${M_PI/2} 0" />
   </xacro:hokuyo_mount>
   <!-- Add a beam at top so that the robot looks complete. -->

Commit message: raised the back kinect by one more inch.

File: segbot_description/robots/segbot_v2.urdf.xacro (robot description, xacro)
@@ -16,5 +16,5 @@
   <!-- Add the forward facing kinect sensor for navigation -->
   <xacro:kinect_mount name="nav_kinect" parent="back_right_vertical_beam" length="${SENSOR_BEAM_LENGTH*INCH_TO_M}">
-    <origin xyz="${1*INCH_TO_M} -${0.5*INCH_TO_M} ${11.5*INCH_TO_M}" rpy="-${M_PI/2} -${M_PI/2} 0" />
+    <origin xyz="${1*INCH_TO_M} -${0.5*INCH_TO_M} ${12.5*INCH_TO_M}" rpy="-${M_PI/2} -${M_PI/2} 0" />
   </xacro:kinect_mount>
   <!-- Add the hokuyo -->

Commit message: lowered height of kinect by 1 inch

File: segbot_description/robots/segbot_v2.urdf.xacro (robot description, xacro)
@@ -16,5 +16,5 @@
   <!-- Add the forward facing kinect sensor for navigation -->
   <xacro:kinect_mount name="nav_kinect" parent="back_right_vertical_beam" length="${SENSOR_BEAM_LENGTH*INCH_TO_M}">
-    <origin xyz="${1*INCH_TO_M} -${0.5*INCH_TO_M} ${12.5*INCH_TO_M}" rpy="-${M_PI/2} -${M_PI/2} 0" />
+    <origin xyz="${1*INCH_TO_M} -${0.5*INCH_TO_M} ${11.5*INCH_TO_M}" rpy="-${M_PI/2} -${M_PI/2} 0" />
   </xacro:kinect_mount>
   <!-- Add the hokuyo -->

Commit message: added sensor plate and sonars to tf tree.

File: segbot_description/robots/segbot_v2.urdf.xacro (robot description, xacro)
@@ -22,8 +22,142 @@
     <origin xyz="${1*INCH_TO_M} ${0.5*INCH_TO_M} ${4.5*INCH_TO_M}" rpy="${M_PI/2} ${M_PI/2} 0" />
   </xacro:hokuyo_mount>
-  <!-- Add a beam at top so that the robot looks complete. -->
+  <!-- The sensor plate shares the hokuyo mount. Use the beam generated by the hokuyo mount to generate the sensor
+       plate. -->
+  <xacro:standoff name="left_sensor_plate_standoff" parent="nav_hokuyo_sensor_beam" length="${0.5*INCH_TO_M}" radius="${0.25*INCH_TO_M}">
+    <origin xyz="-${1/2*INCH_TO_M} 0 ${3.5*INCH_TO_M}" rpy="-${M_PI/2} 0 ${M_PI/2}" />
+  </xacro:standoff>
+  <xacro:standoff name="right_sensor_plate_standoff" parent="nav_hokuyo_sensor_beam" length="${0.5*INCH_TO_M}" radius="${0.25*INCH_TO_M}">
+    <origin xyz="-${1/2*INCH_TO_M} 0 ${8.5*INCH_TO_M}" rpy="-${M_PI/2} 0 ${M_PI/2}" />
+  </xacro:standoff>
+  <xacro:aluminium_sheet name="sensor_plate" parent="left_sensor_plate_standoff" thickness="0.003" length="${4.5*INCH_TO_M}" width="${9*INCH_TO_M}">
+    <origin xyz="-${1/4*INCH_TO_M} -${2.5*INCH_TO_M} ${1/2*INCH_TO_M}" rpy="0 0 0" />
+  </xacro:aluminium_sheet>
+  <joint name="sonar_center_joint" type="fixed">
+    <origin xyz="-${8.58*INCH_TO_M} 0 ${0.003 + 0.012}" />
+    <parent link="sensor_plate_link"/>
+    <child link="sonar_center_link"/>
+  </joint>
+  <!-- sonar_center_link is an empty link that marks the start -->
+  <link name="sonar_center_link">
+    <inertial>
+      <mass value="0.1" />
+      <origin xyz="0 0 0" rpy="0 0 0"/>
+      <inertia ixx="0.01"  ixy="0.0"  ixz="0.0"
+        iyy="0.01"  iyz="0.0"
+        izz="0.01" />
+    </inertial>
+   <visual>
+      <origin xyz="0 0 0" rpy="0 0 0" />
+      <geometry>
+        <box size="0.001 0.001 0.001" />
+      </geometry>
+    </visual>
+  </link>
+  <!-- sonar0 - right -->
+  <joint name="sonar0_rotated_center_joint" type="fixed">
+    <origin xyz="0 0 0" rpy="0 0 -${M_PI/9}"/>
+    <parent link="sonar_center_link"/>
+    <child link="sonar0_rotated_center_link"/>
+  </joint>
+  <link name="sonar0_rotated_center_link">
+    <inertial>
+      <mass value="0.1" />
+      <origin xyz="0 0 0" rpy="0 0 0"/>
+      <inertia ixx="0.01"  ixy="0.0"  ixz="0.0"
+        iyy="0.01"  iyz="0.0"
+        izz="0.01" />
+    </inertial>
+   <visual>
+      <origin xyz="0 0 0" rpy="0 0 0" />
+      <geometry>
+        <box size="0.001 0.001 0.001" />
+      </geometry>
+    </visual>
+  </link>
+  <joint name="sonar0_joint" type="fixed">
+    <origin xyz="${10.33*INCH_TO_M} 0 0" />
+    <parent link="sonar0_rotated_center_link"/>
+    <child link="sonar0_link"/>
+  </joint>
+  <link name="sonar0_link">
+    <inertial>
+      <mass value="0.1" />
+      <origin xyz="0 0 0" rpy="0 0 0"/>
+      <inertia ixx="0.01"  ixy="0.0"  ixz="0.0"
+        iyy="0.01"  iyz="0.0"
+        izz="0.01" />
+    </inertial>
+   <visual>
+      <origin xyz="0 0 0" rpy="0 0 0" />
+      <geometry>
+        <box size="0.012 0.044 0.023" />
+      </geometry>
+    </visual>
+  </link>
+  <!-- sonar1 - center -->
+  <joint name="sonar1_joint" type="fixed">
+    <origin xyz="${10.33*INCH_TO_M} 0 0" />
+    <parent link="sonar_center_link"/>
+    <child link="sonar1_link"/>
+  </joint>
+  <link name="sonar1_link">
+    <inertial>
+      <mass value="0.1" />
+      <origin xyz="0 0 0" rpy="0 0 0"/>
+      <inertia ixx="0.01"  ixy="0.0"  ixz="0.0"
+        iyy="0.01"  iyz="0.0"
+        izz="0.01" />
+    </inertial>
+   <visual>
+      <origin xyz="0 0 0" rpy="0 0 0" />
+      <geometry>
+        <box size="0.012 0.044 0.023" />
+      </geometry>
+    </visual>
+  </link>
+  <!-- sonar2 - left -->
+  <joint name="sonar2_rotated_center_joint" type="fixed">
+    <origin xyz="0 0 0" rpy="0 0 ${M_PI/9}"/>
+    <parent link="sonar_center_link"/>
+    <child link="sonar2_rotated_center_link"/>
+  </joint>
+  <link name="sonar2_rotated_center_link">
+    <inertial>
+      <mass value="0.1" />
+      <origin xyz="0 0 0" rpy="0 0 0"/>
+      <inertia ixx="0.01"  ixy="0.0"  ixz="0.0"
+        iyy="0.01"  iyz="0.0"
+        izz="0.01" />
+    </inertial>
+   <visual>
+      <origin xyz="0 0 0" rpy="0 0 0" />
+      <geometry>
+        <box size="0.001 0.001 0.001" />
+      </geometry>
+    </visual>
+  </link>
+  <joint name="sonar2_joint" type="fixed">
+    <origin xyz="${10.33*INCH_TO_M} 0 0" />
+    <parent link="sonar2_rotated_center_link"/>
+    <child link="sonar2_link"/>
+  </joint>
+  <link name="sonar2_link">
+    <inertial>
+      <mass value="0.1" />
+      <origin xyz="0 0 0" rpy="0 0 0"/>
+      <inertia ixx="0.01"  ixy="0.0"  ixz="0.0"
+        iyy="0.01"  iyz="0.0"
+        izz="0.01" />
+    </inertial>
+   <visual>
+      <origin xyz="0 0 0" rpy="0 0 0" />
+      <geometry>
+        <box size="0.012 0.044 0.023" />
+      </geometry>
+    </visual>
+  </link>
+  <!-- Add a beam at top so that the robot looks complete. We'll probably have a different sensor mount here eventually. -->
   <xacro:beam_8020 name="front_cap_beam" parent="front_right_vertical_beam" length="${SENSOR_BEAM_LENGTH*INCH_TO_M}">
-    <origin xyz="0 -${0.5*INCH_TO_M} ${36.5*INCH_TO_M}"
-      rpy="-${M_PI/2} 0 0" />
+    <origin xyz="0 -${0.5*INCH_TO_M} ${36.5*INCH_TO_M}" rpy="-${M_PI/2} 0 0" />
   </xacro:beam_8020>
   <xacro:gazebo_segbot_ros_controllers />

Commit message: updated segbot_v2 to use independent sensor plate mount. see #34

File: segbot_description/robots/segbot_v2.urdf.xacro (robot description, xacro)
@@ -9,4 +9,5 @@
   <xacro:include filename="$(find segbot_description)/urdf/mounts/hokuyo_mount.urdf.xacro" />
   <xacro:include filename="$(find segbot_description)/urdf/mounts/kinect_mount.urdf.xacro" />
+  <xacro:include filename="$(find segbot_description)/urdf/mounts/sensor_plate_mount.urdf.xacro" />
   <!-- Add the segbot base -->
   <xacro:segbot />
@@ -18,143 +19,14 @@
     <origin xyz="${1*INCH_TO_M} -${0.5*INCH_TO_M} ${11.5*INCH_TO_M}" rpy="-${M_PI/2} -${M_PI/2} 0" />
   </xacro:kinect_mount>
-  <!-- Add the hokuyo -->
-  <xacro:hokuyo_mount name="nav_hokuyo" parent="front_left_vertical_beam" length="${SENSOR_BEAM_LENGTH*INCH_TO_M}" ros_topic="scan" update_rate="10" min_angle="${-(5 * M_PI)/12}" max_angle="${(5 * M_PI)/12}">
+  <!-- Add the shared beam between the hokuyo and the sensor plate -->
+  <xacro:beam_8020 name="hokuyo_sonar_sensor_beam" parent="${parent}" length="${length}">
     <origin xyz="${1*INCH_TO_M} ${0.5*INCH_TO_M} ${4.5*INCH_TO_M}" rpy="${M_PI/2} ${M_PI/2} 0" />
-  </xacro:hokuyo_mount>
-  <!-- The sensor plate shares the hokuyo mount. Use the beam generated by the hokuyo mount to generate the sensor
-       plate. -->
-  <xacro:standoff name="left_sensor_plate_standoff" parent="nav_hokuyo_sensor_beam" length="${0.5*INCH_TO_M}" radius="${0.25*INCH_TO_M}">
-    <origin xyz="-${1/2*INCH_TO_M} 0 ${3.5*INCH_TO_M}" rpy="-${M_PI/2} 0 ${M_PI/2}" />
-  </xacro:standoff>
-  <xacro:standoff name="right_sensor_plate_standoff" parent="nav_hokuyo_sensor_beam" length="${0.5*INCH_TO_M}" radius="${0.25*INCH_TO_M}">
-    <origin xyz="-${1/2*INCH_TO_M} 0 ${8.5*INCH_TO_M}" rpy="-${M_PI/2} 0 ${M_PI/2}" />
-  </xacro:standoff>
-  <xacro:aluminium_sheet name="sensor_plate" parent="left_sensor_plate_standoff" thickness="0.003" length="${4.5*INCH_TO_M}" width="${9*INCH_TO_M}">
-    <origin xyz="-${1/4*INCH_TO_M} -${2.5*INCH_TO_M} ${1/2*INCH_TO_M}" rpy="0 0 0" />
-  </xacro:aluminium_sheet>
-  <joint name="sonar_center_joint" type="fixed">
-    <origin xyz="-${8.58*INCH_TO_M} 0 ${0.003 + 0.012}" />
-    <parent link="sensor_plate_link"/>
-    <child link="sonar_center_link"/>
-  </joint>
-  <!-- sonar_center_link is an empty link that marks the start -->
-  <link name="sonar_center_link">
-    <inertial>
-      <mass value="0.1" />
-      <origin xyz="0 0 0" rpy="0 0 0"/>
-      <inertia ixx="0.01"  ixy="0.0"  ixz="0.0"
-        iyy="0.01"  iyz="0.0"
-        izz="0.01" />
-    </inertial>
-   <visual>
-      <origin xyz="0 0 0" rpy="0 0 0" />
-      <geometry>
-        <box size="0.001 0.001 0.001" />
-      </geometry>
-    </visual>
-  </link>
-  <!-- sonar0 - right -->
-  <joint name="sonar0_rotated_center_joint" type="fixed">
-    <origin xyz="0 0 0" rpy="0 0 -${M_PI/9}"/>
-    <parent link="sonar_center_link"/>
-    <child link="sonar0_rotated_center_link"/>
-  </joint>
-  <link name="sonar0_rotated_center_link">
-    <inertial>
-      <mass value="0.1" />
-      <origin xyz="0 0 0" rpy="0 0 0"/>
-      <inertia ixx="0.01"  ixy="0.0"  ixz="0.0"
-        iyy="0.01"  iyz="0.0"
-        izz="0.01" />
-    </inertial>
-   <visual>
-      <origin xyz="0 0 0" rpy="0 0 0" />
-      <geometry>
-        <box size="0.001 0.001 0.001" />
-      </geometry>
-    </visual>
-  </link>
-  <joint name="sonar0_joint" type="fixed">
-    <origin xyz="${10.33*INCH_TO_M} 0 0" />
-    <parent link="sonar0_rotated_center_link"/>
-    <child link="sonar0_link"/>
-  </joint>
-  <link name="sonar0_link">
-    <inertial>
-      <mass value="0.1" />
-      <origin xyz="0 0 0" rpy="0 0 0"/>
-      <inertia ixx="0.01"  ixy="0.0"  ixz="0.0"
-        iyy="0.01"  iyz="0.0"
-        izz="0.01" />
-    </inertial>
-   <visual>
-      <origin xyz="0 0 0" rpy="0 0 0" />
-      <geometry>
-        <box size="0.012 0.044 0.023" />
-      </geometry>
-    </visual>
-  </link>
-  <!-- sonar1 - center -->
-  <joint name="sonar1_joint" type="fixed">
-    <origin xyz="${10.33*INCH_TO_M} 0 0" />
-    <parent link="sonar_center_link"/>
-    <child link="sonar1_link"/>
-  </joint>
-  <link name="sonar1_link">
-    <inertial>
-      <mass value="0.1" />
-      <origin xyz="0 0 0" rpy="0 0 0"/>
-      <inertia ixx="0.01"  ixy="0.0"  ixz="0.0"
-        iyy="0.01"  iyz="0.0"
-        izz="0.01" />
-    </inertial>
-   <visual>
-      <origin xyz="0 0 0" rpy="0 0 0" />
-      <geometry>
-        <box size="0.012 0.044 0.023" />
-      </geometry>
-    </visual>
-  </link>
-  <!-- sonar2 - left -->
-  <joint name="sonar2_rotated_center_joint" type="fixed">
-    <origin xyz="0 0 0" rpy="0 0 ${M_PI/9}"/>
-    <parent link="sonar_center_link"/>
-    <child link="sonar2_rotated_center_link"/>
-  </joint>
-  <link name="sonar2_rotated_center_link">
-    <inertial>
-      <mass value="0.1" />
-      <origin xyz="0 0 0" rpy="0 0 0"/>
-      <inertia ixx="0.01"  ixy="0.0"  ixz="0.0"
-        iyy="0.01"  iyz="0.0"
-        izz="0.01" />
-    </inertial>
-   <visual>
-      <origin xyz="0 0 0" rpy="0 0 0" />
-      <geometry>
-        <box size="0.001 0.001 0.001" />
-      </geometry>
-    </visual>
-  </link>
-  <joint name="sonar2_joint" type="fixed">
-    <origin xyz="${10.33*INCH_TO_M} 0 0" />
-    <parent link="sonar2_rotated_center_link"/>
-    <child link="sonar2_link"/>
-  </joint>
-  <link name="sonar2_link">
-    <inertial>
-      <mass value="0.1" />
-      <origin xyz="0 0 0" rpy="0 0 0"/>
-      <inertia ixx="0.01"  ixy="0.0"  ixz="0.0"
-        iyy="0.01"  iyz="0.0"
-        izz="0.01" />
-    </inertial>
-   <visual>
-      <origin xyz="0 0 0" rpy="0 0 0" />
-      <geometry>
-        <box size="0.012 0.044 0.023" />
-      </geometry>
-    </visual>
-  </link>
+  </xacro:beam_8020>
+  <!-- Add the hokuyo mount without the beam -->
+  <xacro:hokuyo_mount_without_beam name="nav_hokuyo" parent="hokuyo_sonar_sensor_beam" length="${SENSOR_BEAM_LENGTH*INCH_TO_M}" ros_topic="scan" update_rate="10" min_angle="${-(5 * M_PI)/12}" max_angle="${(5 * M_PI)/12}" range="20.0">
+    <origin xyz="${0.5*INCH_TO_M} 0 ${SENSOR_BEAM_LENGTH/2*INCH_TO_M}" rpy="${M_PI/2} 0 ${M_PI/2}" />
+  </xacro:hokuyo_mount_without_beam>
+  <!-- Add the sensor plate mount -->
+  <xacro:sensor_plate_mount_without_beam parent="hokuyo_sonar_sensor_beam" length="${SENSOR_BEAM_LENGTH*INCH_TO_M}"/>
   <!-- Add a beam at top so that the robot looks complete. We'll probably have a different sensor mount here eventually. -->
   <xacro:beam_8020 name="front_cap_beam" parent="front_right_vertical_beam" length="${SENSOR_BEAM_LENGTH*INCH_TO_M}">

File: segbot_description/urdf/mounts/hokuyo_mount.urdf.xacro (robot description, xacro)
@@ -7,16 +7,20 @@
   <xacro:include filename="$(find segbot_description)/urdf/components/standoff.urdf.xacro" />
   <xacro:include filename="$(find segbot_description)/urdf/components/aluminium_sheet.urdf.xacro" />
-  <xacro:include filename="$(find segbot_description)/urdf/sensors/hokuyo_04lx_laser.urdf.xacro" />
-  <xacro:macro name="hokuyo_mount" params="name parent *origin length ros_topic update_rate min_angle max_angle">
+  <xacro:include filename="$(find segbot_description)/urdf/sensors/hokuyo_laser.urdf.xacro" />
+  <xacro:macro name="hokuyo_mount_without_beam" params="name parent *origin ros_topic update_rate min_angle max_angle range">
+    <xacro:aluminium_sheet name="${name}_plate" parent="${parent}" thickness="${0.125*INCH_TO_M}" length="0.06" width="0.12">
+      <xacro:insert_block name="origin" />
+    </xacro:aluminium_sheet>
+    <xacro:hokuyo_laser name="${name}" parent="${name}_plate" ros_topic="${ros_topic}" update_rate="${update_rate}" min_angle="${min_angle}" max_angle="${max_angle}" range="${range}">
+      <origin xyz="0 0 ${0.125*INCH_TO_M}" rpy="0 0 0" />
+    </xacro:hokuyo_laser>
+  </xacro:macro>
+  <xacro:macro name="hokuyo_mount" params="name parent *origin length ros_topic update_rate min_angle max_angle range">
     <xacro:beam_8020 name="${name}_sensor_beam" parent="${parent}" length="${length}">
       <xacro:insert_block name="origin" />
     </xacro:beam_8020>
-    <xacro:aluminium_sheet name="${name}_plate" parent="${name}_sensor_beam"
-                          thickness="${0.125*INCH_TO_M}" length="0.06" width="0.12">
-                           <origin xyz="${0.5*INCH_TO_M} 0 ${length/2}" rpy="${M_PI/2} 0 ${M_PI/2}" />
-    </xacro:aluminium_sheet>
-    <xacro:hokuyo_04lx_laser name="${name}" parent="${name}_plate" ros_topic="${ros_topic}" update_rate="${update_rate}" min_angle="${min_angle}" max_angle="${max_angle}">
-      <origin xyz="0 0 ${0.125*INCH_TO_M}" rpy="0 0 0" />
-    </xacro:hokuyo_04lx_laser>
+    <xacro:hokuyo_mount_without_beam name="${name}" parent="${name}_sensor_beam" ros_topic="${ros_topic}" update_rate="${update_rate}" min_angle="${min_angle}" max_angle="${max_angle}" range="${range}">
+      <origin xyz="${0.5*INCH_TO_M} 0 ${length/2}" rpy="${M_PI/2} 0 ${M_PI/2}" />
+    </xacro:hokuyo_mount_without_beam>
   </xacro:macro>
 </root>

File: segbot_description/urdf/sensors/hokuyo_laser.gazebo.xacro (robot description, xacro)
@@ -2,5 +2,5 @@
 <root
       xmlns:xacro="http://ros.org/wiki/xacro">
-  <xacro:macro name="hokuyo_04lx_laser_gazebo" params="name ros_topic update_rate min_angle max_angle">
+  <xacro:macro name="hokuyo_laser_gazebo" params="name ros_topic update_rate min_angle max_angle range">
     <gazebo reference="${name}_link">
       <sensor type="ray" name="${name}">
@@ -20,5 +20,5 @@
           <range>
             <min>0.02</min>
-            <max>21.0</max>
+            <max>${range}</max>
             <resolution>0.03</resolution>
           </range>

File: segbot_description/urdf/sensors/hokuyo_laser.urdf.xacro (robot description, xacro)
@@ -4,6 +4,6 @@
       xmlns:interface="http://playerstage.sourceforge.net/gazebo/xmlschema/#interface"
       xmlns:xacro="http://ros.org/wiki/xacro">
-  <xacro:include filename="$(find segbot_description)/urdf/sensors/hokuyo_04lx_laser.gazebo.xacro" />
-  <xacro:macro name="hokuyo_04lx_laser" params="name parent *origin ros_topic update_rate min_angle max_angle">
+  <xacro:include filename="$(find segbot_description)/urdf/sensors/hokuyo_laser.gazebo.xacro" />
+  <xacro:macro name="hokuyo_laser" params="name parent *origin ros_topic update_rate min_angle max_angle range">
     <joint name="${name}_joint" type="fixed">
       <axis xyz="0 1 0" />
@@ -24,10 +24,5 @@
         </geometry>
       </visual>
-      <!-- <collision> -->
-      <!--   <origin xyz="0 0 0" rpy="0 0 0" /> -->
-      <!--   <geometry> -->
-      <!--     <mesh filename="package://segbot_description/meshes/hokuyo.dae" scale="0.0254 0.0254 0.0254" /> -->
-      <!--   </geometry> -->
-      <!-- </collision> -->
+      <!-- ignore the collision element -->
     </link>
     <!-- go from the base of the laser to the actual sensor location -->
@@ -45,5 +40,5 @@
     </link>
     <!-- gazebo extensions -->
-    <xacro:hokuyo_04lx_laser_gazebo name="${name}_laser" ros_topic="${ros_topic}" update_rate="${update_rate}" min_angle="${min_angle}" max_angle="${max_angle}" />
+    <xacro:hokuyo_laser_gazebo name="${name}_laser" ros_topic="${ros_topic}" update_rate="${update_rate}" min_angle="${min_angle}" max_angle="${max_angle}" range="${range}"/>
   </xacro:macro>
 </root>

Commit message: fixed hokuyo location in segbot v2 and segbot v3.

File: segbot_description/robots/segbot_v2.urdf.xacro (robot description, xacro)
@@ -25,5 +25,5 @@
   <!-- Add the hokuyo mount without the beam -->
   <xacro:hokuyo_mount_without_beam name="nav_hokuyo" parent="hokuyo_sonar_sensor_beam" ros_topic="scan" update_rate="10" min_angle="${-(5 * M_PI)/12}" max_angle="${(5 * M_PI)/12}" range="20.0">
-    <origin xyz="${0.5*INCH_TO_M} 0 ${SENSOR_BEAM_LENGTH/2*INCH_TO_M}" rpy="${M_PI/2} 0 ${M_PI/2}" />
+    <origin xyz="${.5*INCH_TO_M} ${0.75*INCH_TO_M} ${SENSOR_BEAM_LENGTH/2*INCH_TO_M}" rpy="${M_PI/2} 0 ${M_PI/2}" />
   </xacro:hokuyo_mount_without_beam>
   <!-- Add the sensor plate mount -->

File: segbot_description/urdf/mounts/hokuyo_mount.urdf.xacro (robot description, xacro)
@@ -9,5 +9,5 @@
   <xacro:include filename="$(find segbot_description)/urdf/sensors/hokuyo_laser.urdf.xacro" />
   <xacro:macro name="hokuyo_mount_without_beam" params="name parent *origin ros_topic update_rate min_angle max_angle range">
-    <xacro:aluminium_sheet name="${name}_plate" parent="${parent}" thickness="${0.125*INCH_TO_M}" length="0.06" width="0.12">
+    <xacro:aluminium_sheet name="${name}_plate" parent="${parent}" thickness="${0.125*INCH_TO_M}" length="${2.5*INCH_TO_M}" width="${4*INCH_TO_M}">
       <xacro:insert_block name="origin" />
     </xacro:aluminium_sheet>
@@ -21,5 +21,5 @@
     </xacro:beam_8020>
     <xacro:hokuyo_mount_without_beam name="${name}" parent="${name}_sensor_beam" ros_topic="${ros_topic}" update_rate="${update_rate}" min_angle="${min_angle}" max_angle="${max_angle}" range="${range}">
-      <origin xyz="${0.5*INCH_TO_M} 0 ${length/2}" rpy="${M_PI/2} 0 ${M_PI/2}" />
+      <origin xyz="${0.5*INCH_TO_M} ${0.75*INCH_TO_M} ${length/2}" rpy="${M_PI/2} 0 ${M_PI/2}" />
     </xacro:hokuyo_mount_without_beam>
   </xacro:macro>
