Commit message: fixed the basic segbot v3 description, which is now ready for supplanting the chassis. fixed the segbot v3 controller.

File: segbot_description/robots/segbot_v3.urdf.xacro (robot description, xacro)
@@ -1,4 +1,6 @@
 <?xml version="1.0"?>
 <!--
+Original copyright notice from rmp.urdf.xacro from segway_description. This file has been modified to look like a RMP
+110 with rear caster assembly.
 Software License Agreement (BSD)
 \file      rmp.urdf.xacro
@@ -22,92 +24,77 @@
 -->
 <robot name="segway_robot" xmlns:xacro="http://ros.org/wiki/xacro">
-    <!-- Included URDF/XACRO Files -->
-    <xacro:include filename="$(find segway_description)/urdf/segway_components/battery.urdf.xacro" />
-    <xacro:include filename="$(find segway_description)/urdf/segway_components/i2_wheel.urdf.xacro" />
-    <xacro:include filename="$(find segway_description)/urdf/segway_components/caster_assembly.urdf.xacro" />
-    <xacro:include filename="$(find segway_description)/urdf/segway_components/std_gearbox_chassis.urdf.xacro" />
-    <xacro:include filename="$(find segway_description)/urdf/segway_components/single_spacer.urdf.xacro" />
-    <xacro:include filename="$(find segway_description)/urdf/segway_components/ui_box.urdf.xacro" />
-    <xacro:include filename="$(find segway_description)/urdf/segway_components/ui_box_spacer_mount.urdf.xacro" />
-    <xacro:include filename="$(find segway_description)/urdf/accessories.urdf.xacro" />
-    <property name="M_PI" value="3.14159"/>
-    <!-- Wheel Mounting Positions -->
-    <xacro:property name="track" value="0.479111" />
-    <xacro:property name="wheel_vertical_offset" value="0.08255015" />
-    <!-- Wheel Properties -->
-    <xacro:property name="wheel_length" value="0.09224900" />
-    <xacro:property name="wheel_radius" value="0.2405681" />
-    <xacro:macro name="segway_robot">
-        <gazebo>
-          <plugin name="gazebo_ros_control" filename="libgazebo_ros_control.so">
-              <robotNamespace>/</robotNamespace>
-          </plugin>
-        </gazebo>
-        <!-- Base link is the center of the robot's chassis between the motors projected on the ground -->
-        <link name="base_link"/>
-        <!--Chassis -->
-        <xacro:std_gearbox_chassis chassis_prefix="base" parent="base_link">
-            <origin xyz="0 0 ${-wheel_vertical_offset + wheel_radius}" rpy="0 0 0" />
-        </xacro:std_gearbox_chassis>
-        <link name="inertial_collision_link">
-			<inertial>
-				<mass value="36.914402" />
-				<origin xyz="-0.043407 0.000037 0.060079" />
-				<inertia ixx="1.182744"  ixy="0.017957" ixz="-0.077476"
-                         iyx="0.017957"  iyy="0.538664" iyz="0.000018"
-                         izx="-0.077476" izy="0.000018" izz="1.240229" />
-			</inertial>
-            <collision>
-				<geometry>
-					<mesh filename="package://segway_description/meshes/collision/RMP210_chassis_collision.stl" />
-				</geometry>
-			</collision>
-		</link>
-		<joint name="inertial_collision_joint" type="fixed" >
-		    <parent link="base_chassis_link" />
-		    <child link="inertial_collision_link" />
-		</joint>
-        <!--Gearbox Spacers -->
-        <xacro:single_spacer spacer_prefix="left" parent="base_chassis_link">
-            <origin xyz="0 0.19582 0.00665015" rpy="0 0 0" />
-        </xacro:single_spacer>
-        <xacro:single_spacer spacer_prefix="right" parent="base_chassis_link">
-            <origin xyz="0 -0.19582 0.00665015" rpy="0 0 ${M_PI}" />
-        </xacro:single_spacer>
-        <!-- Propulsion Batteries -->
-        <xacro:battery battery_prefix="mcu_1" parent="base_chassis_link">
-            <origin xyz="-0.09298 0 0" rpy="0 0 0" />
-        </xacro:battery>
-        <!-- UI Box -->
-        <!-- <xacro:ui_box_spacer_mount parent="base_chassis_link"> -->
-        <!--     <origin xyz="-0.1016 0 0.1273" rpy="0 0 0" /> -->
-        <!-- </xacro:ui_box_spacer_mount> -->
-        <!-- <xacro:ui_box parent="base_chassis_link"> -->
-        <!--     <origin xyz="-0.1016 0 0.1273" rpy="0 0 0" /> -->
-        <!-- </xacro:ui_box> -->
-        <!-- UI Batteries -->
-        <xacro:battery battery_prefix="aux" parent="base_chassis_link">
-            <origin xyz="-0.07845 0 0.1932753" rpy="${M_PI} 0 0" />
-        </xacro:battery>
-        <!-- Segway wheel macros -->
-        <xacro:i2_wheel wheel_prefix="left" parent="base_chassis_link" visual_rotation="0.0">
-            <origin xyz="0 ${track/2} ${wheel_vertical_offset}" rpy="0 0 0" />
-        </xacro:i2_wheel>
-        <xacro:i2_wheel wheel_prefix="right" parent="base_chassis_link" visual_rotation="${M_PI}">
-            <origin xyz="0 ${-track/2} ${wheel_vertical_offset}" rpy="0 0 0" />
-        </xacro:i2_wheel>
-        <!-- Segway Caster Assembly-->
-        <xacro:if value="$(optenv SEGWAY_HAS_REAR_CASTER false)">
-            <xacro:caster_assembly caster_prefix="rear" parent="base_chassis_link">
-                <origin xyz="-0.31472057 0 0.02425235" rpy="0 0 0" />
-            </xacro:caster_assembly>
-        </xacro:if>
-        <xacro:if value="$(optenv SEGWAY_HAS_FRONT_CASTER false)">
-            <xacro:caster_assembly caster_prefix="front" parent="base_chassis_link">
-                <origin xyz="0.31472057 0 0.02425235" rpy="0 0 ${M_PI}" />
-            </xacro:caster_assembly>
-        </xacro:if>
-        <!-- Setup any accessories defined in the environment -->
-        <xacro:segway_accessories />
-    </xacro:macro>
+  <!-- Included URDF/XACRO Files -->
+  <xacro:include filename="$(find segway_description)/urdf/segway_components/battery.urdf.xacro" />
+  <xacro:include filename="$(find segway_description)/urdf/segway_components/i2_wheel.urdf.xacro" />
+  <xacro:include filename="$(find segway_description)/urdf/segway_components/caster_assembly.urdf.xacro" />
+  <xacro:include filename="$(find segway_description)/urdf/segway_components/std_gearbox_chassis.urdf.xacro" />
+  <xacro:include filename="$(find segway_description)/urdf/segway_components/single_spacer.urdf.xacro" />
+  <xacro:include filename="$(find segway_description)/urdf/segway_components/ui_box.urdf.xacro" />
+  <xacro:include filename="$(find segway_description)/urdf/segway_components/ui_box_spacer_mount.urdf.xacro" />
+  <xacro:include filename="$(find segway_description)/urdf/accessories.urdf.xacro" />
+  <property name="M_PI" value="3.14159"/>
+  <!-- Wheel Mounting Positions -->
+  <xacro:property name="track" value="0.479111" />
+  <xacro:property name="wheel_vertical_offset" value="0.08255015" />
+  <!-- Wheel Properties -->
+  <xacro:property name="wheel_length" value="0.09224900" />
+  <xacro:property name="wheel_radius" value="0.2405681" />
+  <xacro:macro name="segway_robot">
+    <gazebo>
+      <plugin name="gazebo_ros_control" filename="libgazebo_ros_control.so">
+        <robotNamespace>/</robotNamespace>
+      </plugin>
+    </gazebo>
+    <!-- Base link is the center of the robot's chassis between the motors projected on the ground -->
+    <link name="base_link"/>
+    <!--Chassis -->
+    <xacro:std_gearbox_chassis chassis_prefix="base" parent="base_link">
+      <origin xyz="0 0 ${-wheel_vertical_offset + wheel_radius}" rpy="0 0 0" />
+    </xacro:std_gearbox_chassis>
+    <link name="inertial_collision_link">
+      <inertial>
+        <mass value="36.914402" />
+        <origin xyz="-0.043407 0.000037 0.060079" />
+        <inertia ixx="1.182744"  ixy="0.017957" ixz="-0.077476"
+          iyx="0.017957"  iyy="0.538664" iyz="0.000018"
+          izx="-0.077476" izy="0.000018" izz="1.240229" />
+      </inertial>
+      <collision>
+        <geometry>
+          <mesh filename="package://segway_description/meshes/collision/RMP210_chassis_collision.stl" />
+        </geometry>
+      </collision>
+    </link>
+    <joint name="inertial_collision_joint" type="fixed" >
+      <parent link="base_chassis_link" />
+      <child link="inertial_collision_link" />
+    </joint>
+    <!--Gearbox Spacers -->
+    <xacro:single_spacer spacer_prefix="left" parent="base_chassis_link">
+      <origin xyz="0 0.19582 0.00665015" rpy="0 0 0" />
+    </xacro:single_spacer>
+    <xacro:single_spacer spacer_prefix="right" parent="base_chassis_link">
+      <origin xyz="0 -0.19582 0.00665015" rpy="0 0 ${M_PI}" />
+    </xacro:single_spacer>
+    <!-- Propulsion Batteries -->
+    <xacro:battery battery_prefix="mcu_1" parent="base_chassis_link">
+      <origin xyz="-0.09298 0 0" rpy="0 0 0" />
+    </xacro:battery>
+    <!-- UI Batteries -->
+    <xacro:battery battery_prefix="aux" parent="base_chassis_link">
+      <origin xyz="0.09298 0 0" rpy="0 0 ${M_PI}" />
+    </xacro:battery>
+    <!-- Segway wheel macros -->
+    <xacro:i2_wheel wheel_prefix="left" parent="base_chassis_link" visual_rotation="0.0">
+      <origin xyz="0 ${track/2} ${wheel_vertical_offset}" rpy="0 0 0" />
+    </xacro:i2_wheel>
+    <xacro:i2_wheel wheel_prefix="right" parent="base_chassis_link" visual_rotation="${M_PI}">
+      <origin xyz="0 ${-track/2} ${wheel_vertical_offset}" rpy="0 0 0" />
+    </xacro:i2_wheel>
+    <!-- Segway Caster Assembly-->
+    <xacro:caster_assembly caster_prefix="rear" parent="base_chassis_link">
+      <origin xyz="-0.31472057 0 0.02425235" rpy="0 0 0" />
+    </xacro:caster_assembly>
+  </xacro:macro>
+  <xacro:segway_robot/>
 </robot>

Commit message: fixed segbot v3 urdf file.

File: segbot_description/robots/segbot_v3.urdf.xacro (robot description, xacro)
@@ -1,100 +1,13 @@
 <?xml version="1.0"?>
-<!--
-Original copyright notice from rmp.urdf.xacro from segway_description. This file has been modified to look like a RMP
-110 with rear caster assembly.
-Software License Agreement (BSD)
-\file      rmp.urdf.xacro
-\authors   Patrick Hussey
-\copyright Copyright (c) 2015, Stanley Innovation, Inc., All rights reserved.
-Redistribution and use in source and binary forms, with or without modification, are permitted provided that
-the following conditions are met:
- * Redistributions of source code must retain the above copyright notice, this list of conditions and the
-   following disclaimer.
- * Redistributions in binary form must reproduce the above copyright notice, this list of conditions and the
-   following disclaimer in the documentation and/or other materials provided with the distribution.
- * Neither the name of Stanley Innovation, Inc. nor the names of its contributors may be used to endorse or promote
-   products derived from this software without specific prior written permission.
-THIS SOFTWARE IS PROVIDED BY THE COPYRIGHT HOLDERS AND CONTRIBUTORS "AS IS" AND ANY EXPRESS OR IMPLIED WAR-
-RANTIES, INCLUDING, BUT NOT LIMITED TO, THE IMPLIED WARRANTIES OF MERCHANTABILITY AND FITNESS FOR A PARTICULAR
-PURPOSE ARE DISCLAIMED. IN NO EVENT SHALL THE COPYRIGHT HOLDER OR CONTRIBUTORS BE LIABLE FOR ANY DIRECT, IN-
-DIRECT, INCIDENTAL, SPECIAL, EXEMPLARY, OR CONSEQUENTIAL DAMAGES (INCLUDING, BUT NOT LIMITED TO, PROCUREMENT
-OF SUBSTITUTE GOODS OR SERVICES; LOSS OF USE, DATA, OR PROFITS; OR BUSINESS INTERRUPTION) HOWEVER CAUSED AND
-ON ANY THEORY OF LIABILITY, WHETHER IN CONTRACT, STRICT LIABILITY, OR TORT (INCLUDING NEGLIGENCE OR OTHERWISE)
-ARISING IN ANY WAY OUT OF THE USE OF THIS SOFTWARE, EVEN IF ADVISED OF THE POSSIBILITY OF SUCH DAMAGE.
--->
-<robot name="segway_robot" xmlns:xacro="http://ros.org/wiki/xacro">
-  <!-- Included URDF/XACRO Files -->
-  <xacro:include filename="$(find segway_description)/urdf/segway_components/battery.urdf.xacro" />
-  <xacro:include filename="$(find segway_description)/urdf/segway_components/i2_wheel.urdf.xacro" />
-  <xacro:include filename="$(find segway_description)/urdf/segway_components/caster_assembly.urdf.xacro" />
-  <xacro:include filename="$(find segway_description)/urdf/segway_components/std_gearbox_chassis.urdf.xacro" />
-  <xacro:include filename="$(find segway_description)/urdf/segway_components/single_spacer.urdf.xacro" />
-  <xacro:include filename="$(find segway_description)/urdf/segway_components/ui_box.urdf.xacro" />
-  <xacro:include filename="$(find segway_description)/urdf/segway_components/ui_box_spacer_mount.urdf.xacro" />
-  <xacro:include filename="$(find segway_description)/urdf/accessories.urdf.xacro" />
-  <property name="M_PI" value="3.14159"/>
-  <!-- Wheel Mounting Positions -->
-  <xacro:property name="track" value="0.479111" />
-  <xacro:property name="wheel_vertical_offset" value="0.08255015" />
-  <!-- Wheel Properties -->
-  <xacro:property name="wheel_length" value="0.09224900" />
-  <xacro:property name="wheel_radius" value="0.2405681" />
-  <xacro:macro name="segway_robot">
-    <gazebo>
-      <plugin name="gazebo_ros_control" filename="libgazebo_ros_control.so">
-        <robotNamespace>/</robotNamespace>
-      </plugin>
-    </gazebo>
-    <!-- Base link is the center of the robot's chassis between the motors projected on the ground -->
-    <link name="base_link"/>
-    <!--Chassis -->
-    <xacro:std_gearbox_chassis chassis_prefix="base" parent="base_link">
-      <origin xyz="0 0 ${-wheel_vertical_offset + wheel_radius}" rpy="0 0 0" />
-    </xacro:std_gearbox_chassis>
-    <link name="inertial_collision_link">
-      <inertial>
-        <mass value="36.914402" />
-        <origin xyz="-0.043407 0.000037 0.060079" />
-        <inertia ixx="1.182744"  ixy="0.017957" ixz="-0.077476"
-          iyx="0.017957"  iyy="0.538664" iyz="0.000018"
-          izx="-0.077476" izy="0.000018" izz="1.240229" />
-      </inertial>
-      <collision>
-        <geometry>
-          <mesh filename="package://segway_description/meshes/collision/RMP210_chassis_collision.stl" />
-        </geometry>
-      </collision>
-    </link>
-    <joint name="inertial_collision_joint" type="fixed" >
-      <parent link="base_chassis_link" />
-      <child link="inertial_collision_link" />
-    </joint>
-    <!--Gearbox Spacers -->
-    <xacro:single_spacer spacer_prefix="left" parent="base_chassis_link">
-      <origin xyz="0 0.19582 0.00665015" rpy="0 0 0" />
-    </xacro:single_spacer>
-    <xacro:single_spacer spacer_prefix="right" parent="base_chassis_link">
-      <origin xyz="0 -0.19582 0.00665015" rpy="0 0 ${M_PI}" />
-    </xacro:single_spacer>
-    <!-- Propulsion Batteries -->
-    <xacro:battery battery_prefix="mcu_1" parent="base_chassis_link">
-      <origin xyz="-0.09298 0 0" rpy="0 0 0" />
-    </xacro:battery>
-    <!-- UI Batteries -->
-    <xacro:battery battery_prefix="aux" parent="base_chassis_link">
-      <origin xyz="0.09298 0 0" rpy="0 0 ${M_PI}" />
-    </xacro:battery>
-    <!-- Segway wheel macros -->
-    <xacro:i2_wheel wheel_prefix="left" parent="base_chassis_link" visual_rotation="0.0">
-      <origin xyz="0 ${track/2} ${wheel_vertical_offset}" rpy="0 0 0" />
-    </xacro:i2_wheel>
-    <xacro:i2_wheel wheel_prefix="right" parent="base_chassis_link" visual_rotation="${M_PI}">
-      <origin xyz="0 ${-track/2} ${wheel_vertical_offset}" rpy="0 0 0" />
-    </xacro:i2_wheel>
-    <!-- Segway Caster Assembly-->
-    <xacro:caster_assembly caster_prefix="rear" parent="base_chassis_link">
-      <origin xyz="-0.31472057 0 0.02425235" rpy="0 0 0" />
-    </xacro:caster_assembly>
-  </xacro:macro>
-  <xacro:segway_robot/>
+<robot name="segbot"
+       xmlns:xacro="http://ros.org/wiki/xacro">
+  <!-- Included URDF Files -->
+  <xacro:include filename="$(find segbot_description)/urdf/segway_110_base.urdf.xacro" />
+  <xacro:include filename="$(find segbot_description)/urdf/v3/common.urdf.xacro" />
+  <xacro:include filename="$(find segbot_description)/urdf/v3/segbot_chassis.urdf.xacro" />
+  <!-- Add the segbot base -->
+  <xacro:segway_robot />
+  <xacro:segbot_chassis parent="base">
+    <origin xyz="${BASE_PLATE_X_OFFSET*INCH_TO_M} 0 ${BASE_PLATE_Z_OFFSET*INCH_TO_M}"/>
+  </xacro:segbot_chassis>
 </robot>

Commit message: some more updates to segbotv3.

File: segbot_description/robots/segbot_v3.urdf.xacro (robot description, xacro)
@@ -11,3 +11,7 @@
     <origin xyz="${BASE_PLATE_X_OFFSET*INCH_TO_M} 0 ${BASE_PLATE_Z_OFFSET*INCH_TO_M}"/>
   </xacro:segbot_chassis>
+  <!-- Add the velodyne -->
+  <xacro:velodyne_mount name="velodyne" parent="back_left_vertical_beam">
+    <origin xyz="${1*INCH_TO_M} -${0.5*INCH_TO_M} ${11.5*INCH_TO_M}" rpy="-${M_PI/2} -${M_PI/2} 0" />
+  </xacro:velodyne_mount>
 </robot>

Commit message: initial testing on simulation complete. will test now on real robot.

File: segbot_description/robots/segbot_v3.urdf.xacro (robot description, xacro)
@@ -6,4 +6,6 @@
   <xacro:include filename="$(find segbot_description)/urdf/v3/common.urdf.xacro" />
   <xacro:include filename="$(find segbot_description)/urdf/v3/segbot_chassis.urdf.xacro" />
+  <xacro:include filename="$(find segbot_description)/urdf/mounts/velodyne_mount.urdf.xacro" />
+  <xacro:include filename="$(find segbot_description)/gazebo/segbot.gazebo.xacro" />
   <!-- Add the segbot base -->
   <xacro:segway_robot />
@@ -13,5 +15,14 @@
   <!-- Add the velodyne -->
   <xacro:velodyne_mount name="velodyne" parent="back_left_vertical_beam">
-    <origin xyz="${1*INCH_TO_M} -${0.5*INCH_TO_M} ${11.5*INCH_TO_M}" rpy="-${M_PI/2} -${M_PI/2} 0" />
+    <origin xyz="0 0 ${14*INCH_TO_M}" rpy="${M_PI} 0 -${M_PI/2}" />
   </xacro:velodyne_mount>
+  <gazebo>
+    <plugin name="object_controller" filename="libgazebo_ros_planar_move.so">
+      <commandTopic>cmd_vel</commandTopic>
+      <odometryTopic>odom</odometryTopic>
+      <odometryFrame>odom</odometryFrame>
+      <robotBaseFrame>base_footprint</robotBaseFrame>
+      <odometryRate>100</odometryRate>
+    </plugin>
+  </gazebo>
 </robot>

File: segbot_description/urdf/mounts/velodyne_mount.urdf.xacro (robot description, xacro)
@@ -6,5 +6,5 @@
   <xacro:include filename="$(find segbot_description)/urdf/components/standoff.urdf.xacro" />
   <xacro:include filename="$(find segbot_description)/urdf/components/aluminium_sheet.urdf.xacro" />
-  <xacro:include filename="$(find velodyne_description)/urdf/VLP-16.urdf.xacro" />
+  <xacro:include filename="$(find segbot_description)/urdf/sensors/VLP-16.urdf.xacro" />
   <xacro:macro name="velodyne_mount" params="name parent *origin">
     <!-- Create a fake link at the specified spot -->

File: segbot_description/urdf/segway_110_base.urdf.xacro (robot description, xacro)
@@ -41,9 +41,9 @@
   <xacro:property name="wheel_radius" value="0.2405681" />
   <xacro:macro name="segway_robot">
-    <gazebo>
-      <plugin name="gazebo_ros_control" filename="libgazebo_ros_control.so">
-        <robotNamespace>/</robotNamespace>
-      </plugin>
-    </gazebo>
+    <!-- <gazebo> -->
+    <!--   <plugin name="gazebo_ros_control" filename="libgazebo_ros_control.so"> -->
+    <!--     <robotNamespace>/</robotNamespace> -->
+    <!--   </plugin> -->
+    <!-- </gazebo> -->
     <!-- Base footprint is the center of the robot's chassis between the motors projected on the ground -->
     <link name="base_footprint"/>

File: segbot_description/urdf/v3/segbot_chassis.urdf.xacro (robot description, xacro)
@@ -30,14 +30,14 @@
     <!-- 80/20 vertical beams -->
     <xacro:beam_8020 name="back_left_vertical_beam" parent="top_box_plate" length="${24*INCH_TO_M}">
+      <origin xyz="-${5.5*INCH_TO_M} ${5.5*INCH_TO_M} ${0.25*INCH_TO_M}" rpy="0 0 0" />
+    </xacro:beam_8020>
+    <xacro:beam_8020 name="front_left_vertical_beam" parent="top_box_plate" length="${24*INCH_TO_M}">
+      <origin xyz="${5.5*INCH_TO_M} ${5.5*INCH_TO_M} ${0.25*INCH_TO_M}" rpy="0 0 0" />
+    </xacro:beam_8020>
+    <xacro:beam_8020 name="back_right_vertical_beam" parent="top_box_plate" length="${24*INCH_TO_M}">
       <origin xyz="-${5.5*INCH_TO_M} -${5.5*INCH_TO_M} ${0.25*INCH_TO_M}" rpy="0 0 0" />
     </xacro:beam_8020>
-    <xacro:beam_8020 name="front_left_vertical_beam" parent="top_box_plate" length="${24*INCH_TO_M}">
+    <xacro:beam_8020 name="front_right_vertical_beam" parent="top_box_plate" length="${24*INCH_TO_M}">
       <origin xyz="${5.5*INCH_TO_M} -${5.5*INCH_TO_M} ${0.25*INCH_TO_M}" rpy="0 0 0" />
-    </xacro:beam_8020>
-    <xacro:beam_8020 name="back_right_vertical_beam" parent="top_box_plate" length="${24*INCH_TO_M}">
-      <origin xyz="-${5.5*INCH_TO_M} ${5.5*INCH_TO_M} ${0.25*INCH_TO_M}" rpy="0 0 0" />
-    </xacro:beam_8020>
-    <xacro:beam_8020 name="front_right_vertical_beam" parent="top_box_plate" length="${24*INCH_TO_M}">
-      <origin xyz="${5.5*INCH_TO_M} ${5.5*INCH_TO_M} ${0.25*INCH_TO_M}" rpy="0 0 0" />
     </xacro:beam_8020>
     <!-- laptop base plate -->

Commit message: updated for hokuyo on segbot v3

File: segbot_description/robots/segbot_v3.urdf.xacro (robot description, xacro)
@@ -7,4 +7,5 @@
   <xacro:include filename="$(find segbot_description)/urdf/v3/segbot_chassis.urdf.xacro" />
   <xacro:include filename="$(find segbot_description)/urdf/mounts/velodyne_mount.urdf.xacro" />
+  <xacro:include filename="$(find segbot_description)/urdf/mounts/hokuyo_mount.urdf.xacro" />
   <xacro:include filename="$(find segbot_description)/gazebo/segbot.gazebo.xacro" />
   <!-- Add the segbot base -->
@@ -17,4 +18,15 @@
     <origin xyz="0 0 ${14*INCH_TO_M}" rpy="${M_PI} 0 -${M_PI/2}" />
   </xacro:velodyne_mount>
+  <xacro:hokuyo_mount
+    name="nav_hokuyo"
+    parent="front_left_vertical_beam"
+    length="${12*INCH_TO_M}"
+    ros_topic="nav_hokuyo/scan"
+    update_rate="10"
+    min_angle="${-(5 * M_PI)/12}"
+    max_angle="${(5 * M_PI)/12}"
+    range="4.1">
+    <origin xyz="${1*INCH_TO_M} ${0.5*INCH_TO_M} ${3.75*INCH_TO_M}" rpy="${M_PI/2} ${M_PI/2} 0" />
+  </xacro:hokuyo_mount>
   <gazebo>
     <!-- <plugin name="object_controller" filename="libgazebo_ros_planar_move.so"> -->

Commit message: added in kinect mount and frame. not positioned correctly.

File: segbot_description/robots/segbot_v3.urdf.xacro (robot description, xacro)
@@ -9,4 +9,6 @@
   <xacro:include filename="$(find segbot_description)/urdf/mounts/hokuyo_mount.urdf.xacro" />
   <xacro:include filename="$(find segbot_description)/gazebo/segbot.gazebo.xacro" />
+  <xacro:include filename="$(find segbot_description)/urdf/mounts/kinect_mount.urdf.xacro" />
+  <xacro:property name="SENSOR_BEAM_LENGTH" value="10.75" /> <!-- inches -->
   <!-- Add the segbot base -->
   <xacro:segway_robot />
@@ -18,4 +20,8 @@
     <origin xyz="0 0 ${14*INCH_TO_M}" rpy="${M_PI} 0 -${M_PI/2}" />
   </xacro:velodyne_mount>
+  <!-- Add the forward facing kinect sensor for navigation -->
+  <xacro:kinect_mount name="nav_kinect" parent="back_right_vertical_beam" length="${SENSOR_BEAM_LENGTH*INCH_TO_M}">
+    <origin xyz="${1*INCH_TO_M} -${0.5*INCH_TO_M} ${11.5*INCH_TO_M}" rpy="-${M_PI/2} -${M_PI/2} 0" />
+  </xacro:kinect_mount>
   <xacro:hokuyo_mount
     name="nav_hokuyo"
