Commit message: adjusted the kinect's height in a very temporary way

File: segbot_description/robots/segbot_v3.urdf.xacro (robot description, xacro)
@@ -22,5 +22,8 @@
   <!-- Add the forward facing kinect sensor for navigation -->
   <xacro:kinect_mount name="nav_kinect" parent="back_right_vertical_beam" length="${SENSOR_BEAM_LENGTH*INCH_TO_M}">
+    <!--
     <origin xyz="${1*INCH_TO_M} -${0.5*INCH_TO_M} ${11.5*INCH_TO_M}" rpy="-${M_PI/2} -${M_PI/2} 0" />
+    -->
+    <origin xyz="${15*INCH_TO_M} -${0.5*INCH_TO_M} ${31.5*INCH_TO_M}" rpy="-${M_PI/2} -${M_PI/2} 0" />
   </xacro:kinect_mount>
   <xacro:hokuyo_mount

Commit message: added kinect mount to model

File: segbot_description/robots/segbot_v3.urdf.xacro (robot description, xacro)
@@ -9,4 +9,7 @@
   <xacro:include filename="$(find segbot_description)/urdf/mounts/hokuyo_mount.urdf.xacro" />
   <xacro:include filename="$(find segbot_description)/gazebo/segbot.gazebo.xacro" />
+  <xacro:include filename="$(find segbot_description)/urdf/mounts/kinect_mount.urdf.xacro" />
+  <xacro:include filename="$(find segbot_description)/urdf/mounts/kinect_mount.urdf.xacro" />
+  <xacro:property name="SENSOR_BEAM_LENGTH" value="10.75" /> <!-- inches -->
   <!-- Add the segbot base -->
   <xacro:segway_robot />
@@ -18,4 +21,11 @@
     <origin xyz="0 0 ${14*INCH_TO_M}" rpy="${M_PI} 0 -${M_PI/2}" />
   </xacro:velodyne_mount>
+  <!-- Add the forward facing kinect sensor for navigation -->
+  <xacro:kinect_mount name="nav_kinect" parent="back_right_vertical_beam" length="${SENSOR_BEAM_LENGTH*INCH_TO_M}">
+    <!--
+    <origin xyz="${1*INCH_TO_M} -${0.5*INCH_TO_M} ${11.5*INCH_TO_M}" rpy="-${M_PI/2} -${M_PI/2} 0" />
+    -->
+    <origin xyz="${15*INCH_TO_M} -${0.5*INCH_TO_M} ${31.5*INCH_TO_M}" rpy="-${M_PI/2} -${M_PI/2} 0" />
+  </xacro:kinect_mount>
   <xacro:hokuyo_mount
     name="nav_hokuyo"
