Commit message: added the segbot arm to the urdf file, added a new urdf for the arm version of the chasis

File: segbot_description/robots/segbot_v2.arm.urdf.xacro (robot description, xacro)
@@ -10,4 +10,5 @@
   <xacro:include filename="$(find segbot_description)/urdf/mounts/kinect_mount.urdf.xacro" />
   <xacro:include filename="$(find segbot_description)/urdf/mounts/sensor_plate_mount.urdf.xacro" />
+  <xacro:include filename="$(find jaco_model)/urdf/mico_arm.xacro" />
   <!-- Add the segbot base -->
   <xacro:segbot />
@@ -31,9 +32,9 @@
   <!-- Add the left sensor beam -->
   <xacro:beam_8020 name="left_sensor_beam" parent="laptop_base_plate" length="${30*INCH_TO_M}">
-    <origin xyz="0 ${8.5*INCH_TO_M} ${0.125*INCH_TO_M}" rpy="0 0 0" />
+    <origin xyz="${-4.5*INCH_TO_M} ${8.5*INCH_TO_M} ${0.125*INCH_TO_M}" rpy="0 0 0" />
   </xacro:beam_8020>
   <!-- Add the right sensor beam -->
   <xacro:beam_8020 name="right_sensor_beam" parent="laptop_base_plate" length="${30*INCH_TO_M}">
-    <origin xyz="0 -${8.5*INCH_TO_M} ${0.125*INCH_TO_M}" rpy="0 0 0" />
+    <origin xyz="${-4.5*INCH_TO_M} -${8.5*INCH_TO_M} ${0.125*INCH_TO_M}" rpy="0 0 0" />
   </xacro:beam_8020>
   <!-- Add the top sensor beam -->
@@ -41,4 +42,31 @@
     <origin xyz="0 -${0.5*INCH_TO_M} ${30.5*INCH_TO_M}" rpy="-${M_PI/2} 0 0" />
   </xacro:beam_8020>
+  <!-- add the arm -->
+  <!--this is needed as the mico_arm xacro file doesn't accept origin as argument -->
+  <joint name="arm_fixed_joint" type="fixed">
+	  <origin xyz="${6*INCH_TO_M} 0 0" rpy="0 0 ${M_PI/2}" />
+      <parent link="laptop_base_plate_link"/>
+      <child link="arm_link"/>
+    </joint>
+	<link name="arm_link">
+      <visual>
+	<origin xyz="0 0 0" rpy="0 0 0" />
+	<geometry>
+	  <box size = "0 0 0"/> <!--making it slightly bigger in x and z direction-->
+	</geometry>
+	<!--<material name="Black" /> -->
+      </visual>
+    <collision>
+	<origin xyz="0 0 0" rpy="0 0 0" />
+	<geometry>
+	  <box size = "0 0 0"/> <!--making it slightly bigger in x and z direction-->
+	</geometry>
+      </collision>
+    </link>
+  <xacro:mico_arm parent="arm_link"/>
+  <!-- add the xtion -->
+  <xacro:kinect_camera name="camera" parent="arm">
+      <origin xyz="0.05 +0.245 0.75" rpy="0 0.74 ${-M_PI/2}" />
+    </xacro:kinect_camera>
   <xacro:gazebo_segbot_ros_controllers />
 </robot>

Commit message: rotated arm around to match physical robot

File: segbot_description/robots/segbot_v2.arm.urdf.xacro (robot description, xacro)
@@ -45,5 +45,5 @@
   <!--this is needed as the mico_arm xacro file doesn't accept origin as argument -->
   <joint name="arm_fixed_joint" type="fixed">
-	  <origin xyz="${6*INCH_TO_M} 0 0" rpy="0 0 ${M_PI/2}" />
+	  <origin xyz="${6*INCH_TO_M} 0 ${1.5*INCH_TO_M}" rpy="0 0 ${0.0*M_PI/2}" />
       <parent link="laptop_base_plate_link"/>
       <child link="arm_link"/>
@@ -67,5 +67,6 @@
   <!-- add the xtion -->
   <xacro:kinect_camera name="xtion_camera" parent="arm">
-      <origin xyz="0.05 +0.245 0.75" rpy="0 0.74 ${-M_PI/2}" />
+     <!-- <origin xyz="0.05 +0.245 0.75" rpy="0 0.74 ${M_PI/2}" /> -->
+      <origin xyz="-0.245 +0.05 0.75" rpy="0 0.74 0" />
     </xacro:kinect_camera>
   <xacro:gazebo_segbot_ros_controllers />

File: segbot_description/urdf/v2/segbot_chassis.urdf.arm.xacro (robot description, xacro)
@@ -73,5 +73,5 @@
     <!-- laptop -->
     <xacro:laptop name="laptop" parent="laptop_base_plate">
-      <origin xyz="-${6.0*INCH_TO_M} 0 ${0.125*INCH_TO_M}" rpy="0 0 0" />
+      <origin xyz="-${3.0*INCH_TO_M} 0 ${0.125*INCH_TO_M}" rpy="0 0 0" />
     </xacro:laptop>
   </xacro:macro>

Commit message: moved the camera to match the physical changed

File: segbot_description/robots/segbot_v2.arm.urdf.xacro (robot description, xacro)
@@ -68,5 +68,5 @@
   <xacro:kinect_camera name="xtion_camera" parent="arm">
      <!-- <origin xyz="0.05 +0.245 0.75" rpy="0 0.74 ${M_PI/2}" /> -->
-      <origin xyz="-0.245 +0.05 0.75" rpy="0 0.74 0" />
+      <origin xyz="-0.265 +0.17 0.7" rpy="0 0.78 0" />
     </xacro:kinect_camera>
   <xacro:gazebo_segbot_ros_controllers />

Commit message: necessary launch files for arm

File: segbot_description/robots/segbot_v2.arm.urdf.xacro (robot description, xacro)
@@ -68,5 +68,5 @@
   <xacro:kinect_camera name="xtion_camera" parent="arm">
      <!-- <origin xyz="0.05 +0.245 0.75" rpy="0 0.74 ${M_PI/2}" /> -->
-      <origin xyz="-0.265 +0.17 0.7" rpy="0 0.78 0" />
+      <origin xyz="-0.265 +0.17 0.74" rpy="0 0.78 0" />
     </xacro:kinect_camera>
   <xacro:gazebo_segbot_ros_controllers />

Commit message: Support arm simulation
Add joint state source for simulator specific arm joint state topic
Add inorder xacro argument to silence deprecation notice

File: segbot_description/robots/segbot_v2.arm.urdf.xacro (robot description, xacro)
@@ -53,5 +53,5 @@
 	<origin xyz="0 0 0" rpy="0 0 0" />
 	<geometry>
-	  <box size = "0 0 0"/> <!--making it slightly bigger in x and z direction-->
+	  <box size = "0.001 0.001 0.001"/> <!--making it slightly bigger in x and z direction-->
 	</geometry>
 	<!--<material name="Black" /> -->
@@ -60,5 +60,5 @@
 	<origin xyz="0 0 0" rpy="0 0 0" />
 	<geometry>
-	  <box size = "0 0 0"/> <!--making it slightly bigger in x and z direction-->
+	  <box size = "0.001 0.001 0.001"/>
 	</geometry>
       </collision>

Commit message: adds xtion mount description files and integrates them into the v2.arm robot

File: segbot_description/robots/segbot_v2.arm.urdf.xacro (robot description, xacro)
@@ -13,4 +13,5 @@
   <xacro:include filename="$(find segbot_description)/urdf/mounts/sensor_plate_mount.urdf.xacro" />
   <xacro:include filename="$(find kinova_description)/urdf/m1n6s200.xacro" />
+  <xacro:include filename="$(find segbot_description)/urdf/sensors/xtion_camera.urdf.xacro"/>
   <!--  <xacro:include filename="$(find segbot_description)/urdf/components/fat_beam_8020.urdf.xacro" /> -->
   <!-- Add the segbot base -->
@@ -72,8 +73,7 @@
   <xacro:m1n6s200 base_parent="arm_link"/>
   <!-- add the xtion -->
-  <xacro:kinect_camera name="xtion_camera" parent="arm">
-     <!-- <origin xyz="0.05 +0.245 0.75" rpy="0 0.74 ${M_PI/2}" /> -->
-      <origin xyz="-0.245 +0.165 0.75" rpy="0 0.74 0" />
-  </xacro:kinect_camera>
+  <xacro:xtion_camera name="xtion_camera" parent="arm">
+      <origin xyz="-0.267 0.0955 0.7525" rpy="0 0 1.57" />
+  </xacro:xtion_camera>
   <xacro:gazebo_segbot_ros_controllers />
 </robot>
