Commit message: azure kinect camera urdf model added to segbot_v4 roslaunch

File: segbot_description/robots/segbot_v4-prism.urdf.xacro (robot description, xacro)
@@ -10,4 +10,5 @@
   <xacro:include filename="$(find segbot_description)/gazebo/segbot.gazebo.xacro" />
   <xacro:include filename="$(find segbot_description)/urdf/mounts/kinect_mount.urdf.xacro" />
+  <xacro:include filename="$(find segbot_description)/urdf/mounts/azure_kinect_mount-prism.urdf.xacro" />
   <xacro:property name="SENSOR_BEAM_LENGTH" value="10.75" /> <!-- inches -->
   <!-- Add the segbot base -->
@@ -27,4 +28,8 @@
     <origin xyz="${15*INCH_TO_M} -${0.5*INCH_TO_M} ${31.5*INCH_TO_M}" rpy="-${M_PI/2} -${M_PI/2} 0" />
   </xacro:kinect_mount>
+  <!-- Add the forward facing azure kinect sensor for navigation -->
+  <xacro:azure_kinect_mount name="azure_kinect" parent="back_right_vertical_beam" length="${SENSOR_BEAM_LENGTH*INCH_TO_M}">
+    <origin xyz="${15*INCH_TO_M} -${0.5*INCH_TO_M} ${21.5*INCH_TO_M}" rpy="-${M_PI/2} -${M_PI/2} 0" />
+  </xacro:azure_kinect_mount>
   <xacro:hokuyo_mount
     name="nav_hokuyo"

File: segbot_description/urdf/mounts/azure_kinect_mount-prism.urdf.xacro (robot description, xacro)
@@ -7,6 +7,8 @@
   <xacro:include filename="$(find segbot_description)/urdf/components/standoff.urdf.xacro" />
   <xacro:include filename="$(find segbot_description)/urdf/components/aluminium_sheet.urdf.xacro" />
-  <xacro:include filename="$(find segbot_description)/urdf/sensors/kinect_camera.urdf.xacro" />
-  <xacro:macro name="kinect_mount" params="name parent *origin length">
+  <!---->
+  <xacro:include filename="$(find segbot_description)/urdf/sensors/azure_camera.urdf.xacro" />
+  <!---->
+  <xacro:macro name="azure_kinect_mount" params="name parent *origin length">
     <xacro:beam_8020 name="${name}_sensor_beam" parent="${parent}" length="${length}">
       <xacro:insert_block name="origin" />
@@ -37,7 +39,17 @@
               rpy="0 0 0" />
     </xacro:aluminium_sheet>
+    <!--
     <xacro:kinect_camera name="${name}" parent="${name}_top_plate">
       <origin xyz="${1.23*INCH_TO_M} -${0.54*INCH_TO_M}0 ${0.88*INCH_TO_M}" rpy="0 0 0" />
     </xacro:kinect_camera>
+    -->
+    <!---->
+    <xacro:azure_kinect_camera name="${name}" parent="${name}_top_plate">
+      <origin xyz="${1.23*INCH_TO_M} -${0.54*INCH_TO_M}0 ${0.88*INCH_TO_M}" rpy="0 0 0" />
+    </xacro:azure_kinect_camera>
+    <!---->
+    <!--
+    <xacro:command="xacro $(find azure_kinect_ros_driver)/urdf/azure_kinect.urdf.xacro" />
+    -->
   </xacro:macro>
 </root>

Commit message: changes for prism experiments

File: segbot_description/robots/segbot_v4-prism.urdf.xacro (robot description, xacro)
@@ -30,5 +30,5 @@
   <!-- Add the forward facing azure kinect sensor for navigation -->
   <xacro:azure_kinect_mount name="azure_kinect" parent="back_right_vertical_beam" length="${SENSOR_BEAM_LENGTH*INCH_TO_M}">
-    <origin xyz="${15*INCH_TO_M} -${0.5*INCH_TO_M} ${21.5*INCH_TO_M}" rpy="-${M_PI/2} -${M_PI/2} 0" />
+    <origin xyz="${15*INCH_TO_M} -${0.5*INCH_TO_M} ${33.8*INCH_TO_M}" rpy="-${M_PI/2} -${M_PI/2} 0" />
   </xacro:azure_kinect_mount>
   <xacro:hokuyo_mount
