Commit message: refactor: update segbot setups for Bing

File: segbot_description/robots/segbot_bu.urdf.xacro (robot description, xacro)
@@ -1,13 +1,10 @@
 <?xml version="1.0"?>
-<robot name="segbot"
-       xmlns:xacro="http://ros.org/wiki/xacro">
+<robot name="segbot" xmlns:xacro="http://ros.org/wiki/xacro">
   <!-- Included URDF Files -->
   <xacro:include filename="$(find segbot_description)/urdf/segway_110_base.urdf.xacro" />
   <xacro:include filename="$(find segbot_description)/urdf/v3/common.urdf.xacro" />
   <xacro:include filename="$(find segbot_description)/urdf/v3/segbot_chassis.urdf.xacro" />
-  <!-- <xacro:include filename="$(find segbot_description)/urdf/mounts/velodyne_mount.urdf.xacro" /> -->
-  <!-- <xacro:include filename="$(find segbot_description)/urdf/mounts/hokuyo_mount.urdf.xacro" /> -->
+  <xacro:include filename="$(find segbot_description)/urdf/mounts/sick_tim_mount.urdf.xacro" />
   <xacro:include filename="$(find segbot_description)/gazebo/segbot.gazebo.xacro" />
-  <!-- <xacro:include filename="$(find segbot_description)/urdf/mounts/kinect_mount.urdf.xacro" />    -->
   <xacro:property name="SENSOR_BEAM_LENGTH" value="10.75" /> <!-- inches -->
   <!-- Add the segbot base -->
@@ -16,26 +13,8 @@
     <origin xyz="${BASE_PLATE_X_OFFSET*INCH_TO_M} 0 ${BASE_PLATE_Z_OFFSET*INCH_TO_M}"/>
   </xacro:segbot_chassis>
-  <!-- Add the velodyne -->
-  <!-- <xacro:velodyne_mount name="velodyne" parent="back_left_vertical_beam">
-    <origin xyz="0 0 ${14*INCH_TO_M}" rpy="${M_PI} 0 -${M_PI/2}" />
-  </xacro:velodyne_mount> -->
-  <!-- Add the forward facing kinect sensor for navigation -->
-  <!-- <xacro:kinect_mount name="nav_kinect" parent="back_right_vertical_beam" length="${SENSOR_BEAM_LENGTH*INCH_TO_M}"> -->
-    <!--
-    <origin xyz="${1*INCH_TO_M} -${0.5*INCH_TO_M} ${11.5*INCH_TO_M}" rpy="-${M_PI/2} -${M_PI/2} 0" />
-    -->
-    <!-- <origin xyz="${15*INCH_TO_M} -${0.5*INCH_TO_M} ${31.5*INCH_TO_M}" rpy="-${M_PI/2} -${M_PI/2} 0" />
-  </xacro:kinect_mount> -->
-  <!-- <xacro:hokuyo_mount
-    name="nav_hokuyo"
-    parent="front_left_vertical_beam"
-    length="${12*INCH_TO_M}"
-    ros_topic="nav_hokuyo/scan"
-    update_rate="10"
-    min_angle="${-(5 * M_PI)/12}"
-    max_angle="${(5 * M_PI)/12}"
-    range="4.1">
-    <origin xyz="${1*INCH_TO_M} ${0.5*INCH_TO_M} ${3.75*INCH_TO_M}" rpy="${M_PI/2} ${M_PI/2} 0" />
-  </xacro:hokuyo_mount> -->
+  <!-- Add the forward facing sick_tim  for navigation -->
+  <xacro:sick_tim_mount name="sick_tim" parent="back_left_vertical_beam" ros_topic="sick_tim/scan">
+    <origin xyz="0 0 ${0.125*INCH_TO_M}" rpy="0 0 0" />
+  </xacro:sick_tim_mount>
   <gazebo>
     <!-- <plugin name="object_controller" filename="libgazebo_ros_planar_move.so"> -->
@@ -48,8 +27,6 @@
     <plugin name="differential_drive_controller" filename="libgazebo_ros_diff_drive.so">
       <updateRate>100</updateRate>
-      <!-- <leftJoint>left_wheel</leftJoint>
-      <rightJoint>right_wheel</rightJoint> -->
-      <leftJoint>right_wheel</leftJoint>
-      <rightJoint>left_wheel</rightJoint>
+      <leftJoint>left_wheel</leftJoint>
+      <rightJoint>right_wheel</rightJoint>
       <wheelSeparation>0.479111</wheelSeparation>
       <wheelDiameter>0.46228</wheelDiameter>

Commit message: updating urdf

File: segbot_description/robots/segbot_bu.urdf.xacro (robot description, xacro)
@@ -3,6 +3,8 @@
   <!-- Included URDF Files -->
   <xacro:include filename="$(find segbot_description)/urdf/segway_110_base.urdf.xacro" />
-  <xacro:include filename="$(find segbot_description)/urdf/v3/common.urdf.xacro" />
-  <xacro:include filename="$(find segbot_description)/urdf/v3/segbot_chassis.urdf.xacro" />
+  <xacro:include filename="$(find segbot_description)/urdf/vbu/common.urdf.xacro" />
+  <xacro:include filename="$(find segbot_description)/urdf/vbu/segbot_chassis.urdf.xacro" />
+  <!-- <xacro:include filename="$(find segbot_description)/urdf/v3/common.urdf.xacro" /> -->
+  <!-- <xacro:include filename="$(find segbot_description)/urdf/v3/segbot_chassis.urdf.xacro" /> -->
   <xacro:include filename="$(find segbot_description)/urdf/mounts/sick_tim_mount.urdf.xacro" />
   <xacro:include filename="$(find segbot_description)/gazebo/segbot.gazebo.xacro" />
@@ -10,11 +12,15 @@
   <!-- Add the segbot base -->
   <xacro:segway_robot />
+  <!-- Segway Caster Assembly-->
+  <xacro:caster_assembly caster_prefix="front" parent="base_chassis_link">
+    <origin xyz="0.31472057 0 0.02425235" rpy="0 0 ${M_PI}" />
+  </xacro:caster_assembly>
   <xacro:segbot_chassis parent="base">
     <origin xyz="${BASE_PLATE_X_OFFSET*INCH_TO_M} 0 ${BASE_PLATE_Z_OFFSET*INCH_TO_M}"/>
   </xacro:segbot_chassis>
   <!-- Add the forward facing sick_tim  for navigation -->
-  <xacro:sick_tim_mount name="sick_tim" parent="back_left_vertical_beam" ros_topic="sick_tim/scan">
-    <origin xyz="0 0 ${0.125*INCH_TO_M}" rpy="0 0 0" />
-  </xacro:sick_tim_mount>
+  <!-- <xacro:sick_tim_mount name="sick_tim" parent="back_left_vertical_beam" ros_topic="sick_tim/scan"> -->
+    <!-- <origin xyz="0 0 ${0.125*INCH_TO_M}" rpy="0 0 0" /> -->
+  <!-- </xacro:sick_tim_mount> -->
   <gazebo>
     <!-- <plugin name="object_controller" filename="libgazebo_ros_planar_move.so"> -->

Commit message: refactor: update robot descriptions

File: segbot_description/robots/segbot_bu.urdf.xacro (robot description, xacro)
@@ -5,6 +5,4 @@
   <xacro:include filename="$(find segbot_description)/urdf/vbu/common.urdf.xacro" />
   <xacro:include filename="$(find segbot_description)/urdf/vbu/segbot_chassis.urdf.xacro" />
-  <!-- <xacro:include filename="$(find segbot_description)/urdf/v3/common.urdf.xacro" /> -->
-  <!-- <xacro:include filename="$(find segbot_description)/urdf/v3/segbot_chassis.urdf.xacro" /> -->
   <xacro:include filename="$(find segbot_description)/urdf/mounts/sick_tim_mount.urdf.xacro" />
   <xacro:include filename="$(find segbot_description)/gazebo/segbot.gazebo.xacro" />
@@ -12,15 +10,12 @@
   <!-- Add the segbot base -->
   <xacro:segway_robot />
-  <!-- Segway Caster Assembly-->
-  <xacro:caster_assembly caster_prefix="front" parent="base_chassis_link">
-    <origin xyz="0.31472057 0 0.02425235" rpy="0 0 ${M_PI}" />
-  </xacro:caster_assembly>
-  <xacro:segbot_chassis parent="base">
+  <xacro:segbot_chassis parent="base_chassis">
     <origin xyz="${BASE_PLATE_X_OFFSET*INCH_TO_M} 0 ${BASE_PLATE_Z_OFFSET*INCH_TO_M}"/>
   </xacro:segbot_chassis>
   <!-- Add the forward facing sick_tim  for navigation -->
-  <!-- <xacro:sick_tim_mount name="sick_tim" parent="back_left_vertical_beam" ros_topic="sick_tim/scan"> -->
-    <!-- <origin xyz="0 0 ${0.125*INCH_TO_M}" rpy="0 0 0" /> -->
-  <!-- </xacro:sick_tim_mount> -->
+  <xacro:sick_tim_mount name="sick_tim" parent="base_chassis" ros_topic="sick_tim/scan">
+    <!-- <origin xyz="${0.125*INCH_TO_M} 0 0" rpy="0 0 0" /> -->
+    <origin xyz="${12.75*INCH_TO_M} 0 ${2.25*INCH_TO_M}" rpy="0 0 0"/>
+  </xacro:sick_tim_mount>
   <gazebo>
     <!-- <plugin name="object_controller" filename="libgazebo_ros_planar_move.so"> -->

File: segbot_description/urdf/vbu/segbot_chassis.urdf.xacro (robot description, xacro)
@@ -8,4 +8,8 @@
   <xacro:include filename="$(find segbot_description)/urdf/components/standoff.urdf.xacro" />
   <xacro:macro name="segbot_chassis" params="parent *origin">
+    <!-- Segway Caster Assembly-->
+    <xacro:caster_assembly caster_prefix="front" parent="${parent}_link">
+      <origin xyz="0.31472057 0 0.02425235" rpy="0 0 ${M_PI}" />
+    </xacro:caster_assembly>
     <!-- bottom box plate -->
     <!-- <xacro:aluminium_sheet name="bottom_box_plate" parent="${parent}"
@@ -30,24 +34,24 @@
     <!-- 80/20 vertical beams -->
     <xacro:beam_8020 name="back_left_vertical_beam" parent="${parent}" length="${24*INCH_TO_M}">
-      <origin xyz="-${5.5*INCH_TO_M} ${5.5*INCH_TO_M} ${10.2*INCH_TO_M}" rpy="0 0 0" />
+      <origin xyz="-${5.0*INCH_TO_M} ${6.0*INCH_TO_M} ${2.25*INCH_TO_M}" rpy="0 0 0" />
     </xacro:beam_8020>
     <xacro:beam_8020 name="front_left_vertical_beam" parent="${parent}" length="${24*INCH_TO_M}">
-      <origin xyz="${5.5*INCH_TO_M} ${5.5*INCH_TO_M} ${10.2*INCH_TO_M}" rpy="0 0 0" />
+      <origin xyz="${5.0*INCH_TO_M} ${6.0*INCH_TO_M} ${2.25*INCH_TO_M}" rpy="0 0 0" />
     </xacro:beam_8020>
     <xacro:beam_8020 name="back_right_vertical_beam" parent="${parent}" length="${24*INCH_TO_M}">
-      <origin xyz="-${5.5*INCH_TO_M} -${5.5*INCH_TO_M} ${10.2*INCH_TO_M}" rpy="0 0 0" />
+      <origin xyz="-${5.0*INCH_TO_M} -${6.0*INCH_TO_M} ${2.25*INCH_TO_M}" rpy="0 0 0" />
     </xacro:beam_8020>
     <xacro:beam_8020 name="front_right_vertical_beam" parent="${parent}" length="${24*INCH_TO_M}">
-      <origin xyz="${5.5*INCH_TO_M} -${5.5*INCH_TO_M} ${10.2*INCH_TO_M}" rpy="0 0 0" />
+      <origin xyz="${5.0*INCH_TO_M} -${6.0*INCH_TO_M} ${2.25*INCH_TO_M}" rpy="0 0 0" />
     </xacro:beam_8020>
     <!-- laptop base plate -->
     <!-- from the left laptop support beam -->
     <xacro:aluminium_sheet name="laptop_base_plate" parent="${parent}"
-                           thickness="${0.125*INCH_TO_M}" length="${12*INCH_TO_M}" width="${14*INCH_TO_M}">
-      <origin xyz="0 0 ${24.25*INCH_TO_M}" rpy="0 0 0" />
+                           thickness="${0.125*INCH_TO_M}" length="${11*INCH_TO_M}" width="${13*INCH_TO_M}">
+      <origin xyz="0 0 ${26.25*INCH_TO_M}" rpy="0 0 0" />
     </xacro:aluminium_sheet>
     <!-- laptop -->
     <xacro:laptop name="laptop" parent="laptop_base_plate">
-      <origin xyz="-${2.1*INCH_TO_M} 0 ${0.125*INCH_TO_M}" rpy="0 0 0" />
+      <origin xyz="0 0 ${0.125*INCH_TO_M}" rpy="0 0 0" />
     </xacro:laptop>
   </xacro:macro>

Commit message: refactor: update navigation settings
This change includes updates of urdf models

File: segbot_description/robots/segbot_bu.urdf.xacro (robot description, xacro)
@@ -1,4 +1,4 @@
 <?xml version="1.0"?>
-<robot name="segbot" xmlns:xacro="http://ros.org/wiki/xacro">
+<robot name="segbot_bu" xmlns:xacro="http://ros.org/wiki/xacro">
   <!-- Included URDF Files -->
   <xacro:include filename="$(find segbot_description)/urdf/segway_110_base.urdf.xacro" />
@@ -11,10 +11,10 @@
   <xacro:segway_robot />
   <xacro:segbot_chassis parent="base_chassis">
-    <origin xyz="${BASE_PLATE_X_OFFSET*INCH_TO_M} 0 ${BASE_PLATE_Z_OFFSET*INCH_TO_M}"/>
+    <origin xyz="${BASE_PLATE_X_OFFSET*INCH_TO_M} 0 ${BASE_PLATE_Z_OFFSET*INCH_TO_M}" rpy="0 0 ${M_PI}"/>
   </xacro:segbot_chassis>
   <!-- Add the forward facing sick_tim  for navigation -->
   <xacro:sick_tim_mount name="sick_tim" parent="base_chassis" ros_topic="sick_tim/scan">
     <!-- <origin xyz="${0.125*INCH_TO_M} 0 0" rpy="0 0 0" /> -->
-    <origin xyz="${12.75*INCH_TO_M} 0 ${2.25*INCH_TO_M}" rpy="0 0 0"/>
+    <origin xyz="${12.75*INCH_TO_M} 0 -${2.25*INCH_TO_M}" rpy="0 0 0"/>
   </xacro:sick_tim_mount>
   <gazebo>

File: segbot_description/robots/segbot_v4.urdf.xacro (robot description, xacro)
@@ -1,4 +1,4 @@
 <?xml version="1.0"?>
-<robot name="segbot"
+<robot name="segbot_v4"
        xmlns:xacro="http://ros.org/wiki/xacro">
   <!-- Included URDF Files -->

Commit message: refactor: update robot description

File: segbot_description/robots/segbot_bu.urdf.xacro (robot description, xacro)
@@ -16,5 +16,5 @@
   <xacro:sick_tim_mount name="sick_tim" parent="base_chassis" ros_topic="sick_tim/scan">
     <!-- <origin xyz="${0.125*INCH_TO_M} 0 0" rpy="0 0 0" /> -->
-    <origin xyz="${12.75*INCH_TO_M} 0 -${2.25*INCH_TO_M}" rpy="0 0 0"/>
+    <origin xyz="${12.75*INCH_TO_M} 0 ${2.25*INCH_TO_M}" rpy="0 0 0"/>
   </xacro:sick_tim_mount>
   <gazebo>

Commit message: basic integration of arm and base

File: segbot_description/robots/segbot_bu.urdf.xacro (robot description, xacro)
@@ -8,4 +8,17 @@
   <xacro:include filename="$(find segbot_description)/gazebo/segbot.gazebo.xacro" />
   <xacro:property name="SENSOR_BEAM_LENGTH" value="10.75" /> <!-- inches -->
+  <xacro:include filename="$(find ur_description)/urdf/inc/ur5e_macro.xacro"/>
+  <xacro:ur5e_robot prefix="" />
+  <joint name="arm_joint" type="fixed">
+    <parent link="laptop_base_plate_link" />
+    <child link = "ur5e_base_link" />
+    <origin xyz="0.0 0.0 0.0" rpy="0.0 0.0 ${M_PI / 2.0}" />
+  </joint>
+  <xacro:include filename="$(find robotiq_2f_140_gripper_visualization)/urdf/robotiq_arg2f_140_model.xacro" />
+  <joint name="gripper_joint" type="fixed">
+    <parent link="tool0" />
+    <child link = "robotiq_arg2f_base_link" />
+    <origin xyz="0.0 0.0 0.01" rpy="0.0 0.0 ${pi/2}" />
+  </joint>
   <!-- Add the segbot base -->
   <xacro:segway_robot />

File: segbot_description/urdf/vbu/segbot_chassis.urdf.xacro (robot description, xacro)
@@ -5,6 +5,7 @@
   <xacro:include filename="$(find segbot_description)/urdf/components/battery_box.urdf.xacro" />
   <xacro:include filename="$(find segbot_description)/urdf/components/beam_8020.urdf.xacro" />
-  <xacro:include filename="$(find segbot_description)/urdf/components/laptop.urdf.xacro" />
+  <!-- <xacro:include filename="$(find segbot_description)/urdf/components/laptop.urdf.xacro" /> -->
   <xacro:include filename="$(find segbot_description)/urdf/components/standoff.urdf.xacro" />
+  <xacro:include filename="$(find segbot_description)/urdf/components/front_wall.urdf.xacro" />
   <xacro:macro name="segbot_chassis" params="parent *origin">
     <!-- Segway Caster Assembly-->
@@ -51,8 +52,12 @@
       <origin xyz="0 0 ${26.25*INCH_TO_M}" rpy="0 0 0" />
     </xacro:aluminium_sheet>
+    <xacro:front_wall name="front_wall" parent="laptop_base_plate" thickness="${0.125*INCH_TO_M}" length="${25*INCH_TO_M}" width="${12*INCH_TO_M}">
+      <origin xyz="${8.0*INCH_TO_M} ${0.0*INCH_TO_M} ${12.5*INCH_TO_M}"
+        rpy="0 ${M_PI/2} 0" />
+    </xacro:front_wall>
     <!-- laptop -->
-    <xacro:laptop name="laptop" parent="laptop_base_plate">
+    <!-- <xacro:laptop name="laptop" parent="laptop_base_plate">
       <origin xyz="0 0 ${0.125*INCH_TO_M}" rpy="0 0 0" />
-    </xacro:laptop>
+    </xacro:laptop> -->
   </xacro:macro>
 </root>
