Commit message: constructed a mesh model for the hokuyo and replaced it in the urdf file. Now the hokuyo needs a separate frame for the laser location

File: segbot_description/urdf/sensors/hokuyo_04lx_laser.urdf.xacro (robot description, xacro)
@@ -21,5 +21,6 @@
         <origin xyz="0 0 0" rpy="0 0 0" />
         <geometry>
-          <box size="0.05 0.05 0.07" />
+          <!-- <box size="0.05 0.05 0.07" /> -->
+          <mesh filename="package://segbot_description/meshes/hokuyo.dae" scale="0.0254 0.0254 0.0254" />
         </geometry>
       </visual>
