Commit message: some relocation/renaming of the gazebo specific urdf files

File: segbot_description/gazebo/common.gazebo.xacro (robot description, xacro)
@@ -3,6 +3,7 @@
   xmlns:sensor="http://playerstage.sourceforge.net/gazebo/xmlschema/#sensor"
   xmlns:controller="http://playerstage.sourceforge.net/gazebo/xmlschema/#controller"
-  xmlns:interface="http://playerstage.sourceforge.net/gazebo/xmlschema/#interface">
-  <macro name="gazebo_segbot_base_link_surface">
+  xmlns:interface="http://playerstage.sourceforge.net/gazebo/xmlschema/#interface"
+  xmlns:xacro="http://ros.org/wiki/xacro">
+  <xacro:macro name="gazebo_segbot_base_link_surface">
     <gazebo reference="base_link">
       <mu1 value="100.0" />
@@ -11,6 +12,6 @@
       <kd  value="1.0" />
     </gazebo>
-  </macro>
-  <macro name="gazebo_segbot_castor_wheel_link_surface">
+  </xacro:macro>
+  <xacro:macro name="gazebo_segbot_castor_wheel_link_surface">
     <gazebo reference="caster_wheel_link">
       <mu1 value="10.0" />
@@ -19,42 +20,42 @@
       <kd  value="1.0" />
     </gazebo>
-  </macro>
-  <macro name="segbot_base_link_mesh">
+  </xacro:macro>
+  <xacro:macro name="segbot_base_link_mesh">
     <origin xyz="0 0 0" rpy="0 0 0" />
     <geometry>
       <mesh filename="package://segbot_description/meshes/rmp50-base-link.dae" scale="0.0254 0.0254 0.0254"/>
     </geometry>
-  </macro>
-  <macro name="segbot_base_link_cylinder">
+  </xacro:macro>
+  <xacro:macro name="segbot_base_link_cylinder">
     <origin xyz="0 0 0" rpy="0 0 0" />
     <geometry>
       <cylinder length="0.4330" radius="0.6" />
     </geometry>
-  </macro>
-  <macro name="segbot_castor_wheel_link_mesh">
+  </xacro:macro>
+  <xacro:macro name="segbot_castor_wheel_link_mesh">
     <origin xyz="0 0 0" rpy="0 0 0" />
     <geometry>
       <mesh filename="package://segbot_description/meshes/rmp50-castor-wheel.dae" scale="0.0254 0.0254 0.0254"/>
     </geometry>
-  </macro>
-  <macro name="segbot_collision_none">
+  </xacro:macro>
+  <xacro:macro name="segbot_collision_none">
     <origin xyz="0 0 0" rpy="0 0 0" />
     <geometry>
       <box size="0.01 0.01 0.01" />
     </geometry>
-  </macro>
-  <macro name="segbot_castor_support_link_mesh">
+  </xacro:macro>
+  <xacro:macro name="segbot_castor_support_link_mesh">
     <origin xyz="0 0 0" rpy="0 0 0" />
     <geometry>
       <mesh filename="package://segbot_description/meshes/rmp50-castor-link.dae" scale="0.0254 0.0254 0.0254"/>
     </geometry>
-  </macro>
-  <macro name="segbot_wheel_mesh" params="suffix">
+  </xacro:macro>
+  <xacro:macro name="segbot_wheel_mesh" params="suffix">
     <origin xyz="0 0 0" rpy="0 0 0" />
     <geometry>
       <mesh filename="package://segbot_description/meshes/rmp50-${suffix}-wheel.dae" scale="0.0254 0.0254 0.0254"/>
     </geometry>
-  </macro>
-  <macro name="gazebo_segbot_wheel_surface">
+  </xacro:macro>
+  <xacro:macro name="gazebo_segbot_wheel_surface">
     <gazebo reference="${parent}_${suffix}_wheel_link" >
       <mu1 value="10.0" />
@@ -63,6 +64,6 @@
       <kd  value="1.0" />
     </gazebo>
-  </macro>
-  <macro name="gazebo_segbot_controllers_common">
+  </xacro:macro>
+  <xacro:macro name="gazebo_segbot_controllers_common">
     <canonicalBody>base_footprint</canonicalBody>
     <controller:gazebo_ros_controller_manager name="gazebo_ros_controller_manager" plugin="libgazebo_ros_controller_manager.so">
@@ -71,6 +72,6 @@
       <interface:audio name="gazebo_ros_controller_manager_dummy_iface" />
     </controller:gazebo_ros_controller_manager>
-  </macro>
-  <macro name="gazebo_segbot_drive_parameters">
+  </xacro:macro>
+  <xacro:macro name="gazebo_segbot_drive_parameters">
     <alwaysOn>true</alwaysOn>
     <update>100</update>
@@ -83,14 +84,14 @@
     <interface:position name="position_iface_0"/>
     <topicName>cmd_vel</topicName>
-  </macro>
-  <macro name="gazebo_segbot_simple_drive_plugin">
+  </xacro:macro>
+  <xacro:macro name="gazebo_segbot_simple_drive_plugin">
     <controller:segbotsimpledrive_plugin name="differential_drive_controller" plugin="libsegbotsimpledrive_plugin.so">
       <gazebo_segbot_drive_parameters />
     </controller:segbotsimpledrive_plugin>
-  </macro>
-  <macro name="gazebo_segbot_drive_plugin">
+  </xacro:macro>
+  <xacro:macro name="gazebo_segbot_drive_plugin">
     <controller:segbotdrive_plugin name="differential_drive_controller" plugin="libsegbotdrive_plugin.so">
       <gazebo_segbot_drive_parameters />
     </controller:segbotdrive_plugin>
-  </macro>
+  </xacro:macro>
 </robot>

File: segbot_description/gazebo/full_collision.gazebo.xacro (robot description, xacro)
@@ -1,11 +1,14 @@
 <?xml version="1.0"?>
-<robot>
+<robot
+  xmlns:sensor="http://playerstage.sourceforge.net/gazebo/xmlschema/#sensor"
+  xmlns:controller="http://playerstage.sourceforge.net/gazebo/xmlschema/#controller"
+  xmlns:interface="http://playerstage.sourceforge.net/gazebo/xmlschema/#interface">
   <!-- Included URDF Files -->
-  <include filename="$(find segbot_description)/urdf/gazebo_common.xacro" />
+  <include filename="$(find segbot_description)/gazebo/common.gazebo.xacro" />
   <macro name="segbot_base_link_visual" >
     <segbot_base_link_mesh />
   </macro>
   <macro name="segbot_base_link_collision" >
-    <segbot_base_link_cylinder />
+    <segbot_base_link_mesh />
   </macro>
   <macro name="segbot_castor_support_link_visual" >
@@ -13,5 +16,5 @@
   </macro>
   <macro name="segbot_castor_support_link_collision" >
-    <segbot_collision_none />
+    <segbot_castor_support_link_mesh />
   </macro>
   <macro name="segbot_castor_wheel_link_visual" >
@@ -19,5 +22,5 @@
   </macro>
   <macro name="segbot_castor_wheel_link_collision" >
-    <segbot_collision_none />
+    <segbot_castor_wheel_link_mesh />
   </macro>
   <macro name="segbot_wheel_visual" params="suffix">
@@ -25,9 +28,9 @@
   </macro>
   <macro name="segbot_wheel_collision" params="suffix">
-    <segbot_collision_none />
+    <segbot_wheel_mesh suffix="${suffix}" />
   </macro>
   <macro name="gazebo_segbot_ros_controllers">
     <gazebo>
-      <gazebo_segbot_simple_drive_plugin />
+      <gazebo_segbot_drive_plugin />
       <gazebo_segbot_controllers_common />
     </gazebo>

File: segbot_description/gazebo/simple_collision.gazebo.xacro (robot description, xacro)
@@ -1,14 +1,11 @@
 <?xml version="1.0"?>
-<robot
-  xmlns:sensor="http://playerstage.sourceforge.net/gazebo/xmlschema/#sensor"
-  xmlns:controller="http://playerstage.sourceforge.net/gazebo/xmlschema/#controller"
-  xmlns:interface="http://playerstage.sourceforge.net/gazebo/xmlschema/#interface">
+<robot>
   <!-- Included URDF Files -->
-  <include filename="$(find segbot_description)/urdf/gazebo_common.xacro" />
+  <include filename="$(find segbot_description)/gazebo/common.gazebo.xacro" />
   <macro name="segbot_base_link_visual" >
     <segbot_base_link_mesh />
   </macro>
   <macro name="segbot_base_link_collision" >
-    <segbot_base_link_mesh />
+    <segbot_base_link_cylinder />
   </macro>
   <macro name="segbot_castor_support_link_visual" >
@@ -16,5 +13,5 @@
   </macro>
   <macro name="segbot_castor_support_link_collision" >
-    <segbot_castor_support_link_mesh />
+    <segbot_collision_none />
   </macro>
   <macro name="segbot_castor_wheel_link_visual" >
@@ -22,5 +19,5 @@
   </macro>
   <macro name="segbot_castor_wheel_link_collision" >
-    <segbot_castor_wheel_link_mesh />
+    <segbot_collision_none />
   </macro>
   <macro name="segbot_wheel_visual" params="suffix">
@@ -28,9 +25,9 @@
   </macro>
   <macro name="segbot_wheel_collision" params="suffix">
-    <segbot_wheel_mesh suffix="${suffix}" />
+    <segbot_collision_none />
   </macro>
   <macro name="gazebo_segbot_ros_controllers">
     <gazebo>
-      <gazebo_segbot_drive_plugin />
+      <gazebo_segbot_simple_drive_plugin />
       <gazebo_segbot_controllers_common />
     </gazebo>

File: segbot_description/robots/segbot_hokuyo.urdf.xacro (robot description, xacro)
@@ -4,5 +4,5 @@
   <!-- Included URDF Files -->
   <include filename="$(find segbot_description)/urdf/common.urdf.xacro" />
-  <include filename="$(find segbot_description)/urdf/gazebo_simple.xacro" />
+  <include filename="$(find segbot_description)/gazebo/simple_collision.gazebo.xacro" />
   <include filename="$(find segbot_description)/urdf/segbot_base.xacro" />
   <include filename="$(find segbot_description)/urdf/segbot_chassis.urdf.xacro" />

File: segbot_description/robots/segbot_kinect.urdf.xacro (robot description, xacro)
@@ -4,5 +4,5 @@
   <!-- Included URDF Files -->
   <include filename="$(find segbot_description)/urdf/common.urdf.xacro" />
-  <include filename="$(find segbot_description)/urdf/gazebo_simple.xacro" />
+  <include filename="$(find segbot_description)/gazebo/simple_collision.gazebo.xacro" />
   <include filename="$(find segbot_description)/urdf/segbot_base.xacro" />
   <include filename="$(find segbot_description)/urdf/segbot_chassis.urdf.xacro" />

Commit message: more cleanup in the gazebo launch files

File: segbot_description/gazebo/common.gazebo.xacro (robot description, xacro)
@@ -1,4 +1,4 @@
 <?xml version="1.0"?>
-<robot
+<root
   xmlns:sensor="http://playerstage.sourceforge.net/gazebo/xmlschema/#sensor"
   xmlns:controller="http://playerstage.sourceforge.net/gazebo/xmlschema/#controller"
@@ -95,3 +95,3 @@
     </controller:segbotdrive_plugin>
   </xacro:macro>
-</robot>
+</root>

File: segbot_description/gazebo/full_collision.gazebo.xacro (robot description, xacro)
@@ -1,38 +1,36 @@
 <?xml version="1.0"?>
-<robot
-  xmlns:sensor="http://playerstage.sourceforge.net/gazebo/xmlschema/#sensor"
-  xmlns:controller="http://playerstage.sourceforge.net/gazebo/xmlschema/#controller"
-  xmlns:interface="http://playerstage.sourceforge.net/gazebo/xmlschema/#interface">
+<root
+  xmlns:xacro="http://ros.org/wiki/xacro">
   <!-- Included URDF Files -->
   <include filename="$(find segbot_description)/gazebo/common.gazebo.xacro" />
-  <macro name="segbot_base_link_visual" >
-    <segbot_base_link_mesh />
-  </macro>
-  <macro name="segbot_base_link_collision" >
-    <segbot_base_link_mesh />
-  </macro>
-  <macro name="segbot_castor_support_link_visual" >
-    <segbot_castor_support_link_mesh />
-  </macro>
-  <macro name="segbot_castor_support_link_collision" >
-    <segbot_castor_support_link_mesh />
-  </macro>
-  <macro name="segbot_castor_wheel_link_visual" >
-    <segbot_castor_wheel_link_mesh />
-  </macro>
-  <macro name="segbot_castor_wheel_link_collision" >
-    <segbot_castor_wheel_link_mesh />
-  </macro>
-  <macro name="segbot_wheel_visual" params="suffix">
-    <segbot_wheel_mesh suffix="${suffix}" />
-  </macro>
-  <macro name="segbot_wheel_collision" params="suffix">
-    <segbot_wheel_mesh suffix="${suffix}" />
-  </macro>
-  <macro name="gazebo_segbot_ros_controllers">
+  <xacro:macro name="segbot_base_link_visual" >
+    <xacro:segbot_base_link_mesh />
+  </xacro:macro>
+  <xacro:macro name="segbot_base_link_collision" >
+    <xacro:segbot_base_link_mesh />
+  </xacro:macro>
+  <xacro:macro name="segbot_castor_support_link_visual" >
+    <xacro:segbot_castor_support_link_mesh />
+  </xacro:macro>
+  <xacro:macro name="segbot_castor_support_link_collision" >
+    <xacro:segbot_castor_support_link_mesh />
+  </xacro:macro>
+  <xacro:macro name="segbot_castor_wheel_link_visual" >
+    <xacro:segbot_castor_wheel_link_mesh />
+  </xacro:macro>
+  <xacro:macro name="segbot_castor_wheel_link_collision" >
+    <xacro:segbot_castor_wheel_link_mesh />
+  </xacro:macro>
+  <xacro:macro name="segbot_wheel_visual" params="suffix">
+    <xacro:segbot_wheel_mesh suffix="${suffix}" />
+  </xacro:macro>
+  <xacro:macro name="segbot_wheel_collision" params="suffix">
+    <xacro:segbot_wheel_mesh suffix="${suffix}" />
+  </xacro:macro>
+  <xacro:macro name="gazebo_segbot_ros_controllers">
     <gazebo>
-      <gazebo_segbot_drive_plugin />
-      <gazebo_segbot_controllers_common />
+      <xacro:gazebo_segbot_drive_plugin />
+      <xacro:gazebo_segbot_controllers_common />
     </gazebo>
-  </macro>
-</robot>
+  </xacro:macro>
+</root>

File: segbot_description/gazebo/simple_collision.gazebo.xacro (robot description, xacro)
@@ -1,35 +1,36 @@
 <?xml version="1.0"?>
-<robot>
+<root
+  xmlns:xacro="http://ros.org/wiki/xacro">
   <!-- Included URDF Files -->
   <include filename="$(find segbot_description)/gazebo/common.gazebo.xacro" />
-  <macro name="segbot_base_link_visual" >
-    <segbot_base_link_mesh />
-  </macro>
-  <macro name="segbot_base_link_collision" >
-    <segbot_base_link_cylinder />
-  </macro>
-  <macro name="segbot_castor_support_link_visual" >
-    <segbot_castor_support_link_mesh />
-  </macro>
-  <macro name="segbot_castor_support_link_collision" >
-    <segbot_collision_none />
-  </macro>
-  <macro name="segbot_castor_wheel_link_visual" >
-    <segbot_castor_wheel_link_mesh />
-  </macro>
-  <macro name="segbot_castor_wheel_link_collision" >
-    <segbot_collision_none />
-  </macro>
-  <macro name="segbot_wheel_visual" params="suffix">
-    <segbot_wheel_mesh suffix="${suffix}" />
-  </macro>
-  <macro name="segbot_wheel_collision" params="suffix">
-    <segbot_collision_none />
-  </macro>
-  <macro name="gazebo_segbot_ros_controllers">
+  <xacro:macro name="segbot_base_link_visual" >
+    <xacro:segbot_base_link_mesh />
+  </xacro:macro>
+  <xacro:macro name="segbot_base_link_collision" >
+    <xacro:segbot_base_link_cylinder />
+  </xacro:macro>
+  <xacro:macro name="segbot_castor_support_link_visual" >
+    <xacro:segbot_castor_support_link_mesh />
+  </xacro:macro>
+  <xacro:macro name="segbot_castor_support_link_collision" >
+    <xacro:segbot_collision_none />
+  </xacro:macro>
+  <xacro:macro name="segbot_castor_wheel_link_visual" >
+    <xacro:segbot_castor_wheel_link_mesh />
+  </xacro:macro>
+  <xacro:macro name="segbot_castor_wheel_link_collision" >
+    <xacro:segbot_collision_none />
+  </xacro:macro>
+  <xacro:macro name="segbot_wheel_visual" params="suffix">
+    <xacro:segbot_wheel_mesh suffix="${suffix}" />
+  </xacro:macro>
+  <xacro:macro name="segbot_wheel_collision" params="suffix">
+    <xacro:segbot_collision_none />
+  </xacro:macro>
+  <xacro:macro name="gazebo_segbot_ros_controllers">
     <gazebo>
-      <gazebo_segbot_simple_drive_plugin />
-      <gazebo_segbot_controllers_common />
+      <xacro:gazebo_segbot_simple_drive_plugin />
+      <xacro:gazebo_segbot_controllers_common />
     </gazebo>
-  </macro>
-</robot>
+  </xacro:macro>
+</root>

Commit message: fixed some surface properties, removed transmission as recommended by ros wiki page

File: segbot_description/gazebo/common.gazebo.xacro (robot description, xacro)
@@ -57,5 +57,5 @@
     </geometry>
   </xacro:macro>
-  <xacro:macro name="gazebo_segbot_wheel_surface">
+  <xacro:macro name="gazebo_segbot_wheel_surface" params="parent suffix">
     <gazebo reference="${parent}_${suffix}_wheel_link" >
       <mu1 value="10.0" />

File: segbot_description/urdf/segbot_base.urdf.xacro (robot description, xacro)
@@ -7,5 +7,5 @@
     <!-- root link, on the ground just below the robot origin -->
     <link name="base_footprint">
-      <visual>
+     <visual>
         <origin xyz="0 0 0" rpy="0 0 0" />
         <geometry>
@@ -22,9 +22,9 @@
     <link name="base_link">
       <inertial>
-        <mass value="0.01" />
-        <origin xyz="0 0 0" />
-        <inertia ixx="1.0" ixy="0.0" ixz="0.0"
-          iyy="1.0" iyz="0.0"
-          izz="1.0" />
+        <mass value="30" />
+        <origin xyz="-0.1 0 -0.075" />
+        <inertia ixx="3.0" ixy="0.0" ixz="0.0"
+          iyy="3.0" iyz="0.0"
+          izz="2.0" />
       </inertial>
       <visual>
@@ -37,18 +37,18 @@
     <xacro:gazebo_segbot_base_link_surface />
     <!-- pushing the center of mass of the body to a more appropriate pos -->
-    <joint name="base_center_of_mass_joint" type="fixed">
-      <origin xyz="-0.1 0 -0.075" rpy="0 0 0" />
-      <parent link="base_link"/>
-      <child link="base_center_of_mass_link" />
-    </joint>
-    <link name="base_center_of_mass_link">
-      <inertial>
-        <mass value="30" />
-        <origin xyz="0 0 0" />
-        <inertia ixx="1.0" ixy="0.0" ixz="0.0"
-          iyy="1.0" iyz="0.0"
-          izz="1.0" />
-      </inertial>
-    </link>
+    <!-- <joint name="base_center_of_mass_joint" type="fixed"> -->
+    <!--   <origin xyz="-0.1 0 -0.075" rpy="0 0 0" /> -->
+    <!--   <parent link="base_link"/> -->
+    <!--   <child link="base_center_of_mass_link" /> -->
+    <!-- </joint> -->
+    <!-- <link name="base_center_of_mass_link"> -->
+    <!--   <inertial> -->
+    <!--     <mass value="30" /> -->
+    <!--     <origin xyz="0 0 0" /> -->
+    <!--     <inertia ixx="1.0" ixy="0.0" ixz="0.0" -->
+    <!--       iyy="1.0" iyz="0.0"  -->
+    <!--       izz="1.0" /> -->
+    <!--   </inertial> -->
+    <!-- </link> -->
     <!-- castor joint and wheel -->
     <joint name="base_caster_support_joint" type="continuous">
@@ -81,4 +81,10 @@
       </collision>
     </link>
+    <gazebo reference="base_caster_support_link">
+      <mu1 value="100.0" />
+      <mu2 value="100.0" />
+      <kp  value="1000000.0" />
+      <kd  value="1.0" />
+    </gazebo>
     <joint name="caster_wheel_joint" type="continuous">
       <origin xyz="-0.0397 0 -0.0918" rpy="0 0 0" />
@@ -90,9 +96,9 @@
       <joint_properties damping="0.0" friction="0.0" />
     </joint>
-    <transmission type="pr2_mechanism_model/SimpleTransmission" name="caster_wheel_trans">
-      <actuator name="caster_wheel_motor" />
-      <joint name="caster_wheel_joint" />
-      <mechanicalReduction>1.0</mechanicalReduction>
-    </transmission>
+    <!-- <transmission type="pr2_mechanism_model/SimpleTransmission" name="caster_wheel_trans"> -->
+    <!--   <actuator name="caster_wheel_motor" /> -->
+    <!--   <joint name="caster_wheel_joint" /> -->
+    <!--   <mechanicalReduction>1.0</mechanicalReduction> -->
+    <!-- </transmission> -->
     <link name="caster_wheel_link">
       <inertial>

File: segbot_description/urdf/segbot_chassis.urdf.xacro (robot description, xacro)
@@ -48,4 +48,10 @@
       </collision>
     </link>
+    <gazebo reference="battery_box_link">
+      <mu1 value="100.0" />
+      <mu2 value="100.0" />
+      <kp  value="1000000.0" />
+      <kd  value="1.0" />
+    </gazebo>
     <!-- 80/20 base beams -->
     <!-- left beam -->

File: segbot_description/urdf/segbot_wheel.urdf.xacro (robot description, xacro)
@@ -27,10 +27,10 @@
       </collision>
     </link>
-    <xacro:gazebo_segbot_wheel_surface />
-    <transmission type="pr2_mechanism_model/SimpleTransmission" name="${parent}_${suffix}_wheel_trans">
-      <actuator name="${parent}_${suffix}_wheel_motor" />
-      <joint name="${parent}_${suffix}_wheel_joint" />
-      <mechanicalReduction>1.0</mechanicalReduction>
-    </transmission>
+    <xacro:gazebo_segbot_wheel_surface parent="${parent}" suffix="${suffix}" />
+    <!-- <transmission type="pr2_mechanism_model/SimpleTransmission" name="${parent}_${suffix}_wheel_trans"> -->
+    <!--   <actuator name="${parent}_${suffix}_wheel_motor" /> -->
+    <!--   <joint name="${parent}_${suffix}_wheel_joint" /> -->
+    <!--   <mechanicalReduction>1.0</mechanicalReduction> -->
+    <!-- </transmission> -->
   </xacro:macro>
 </root>
