Commit message: some minor urdf cleanup

File: segbot_description/gazebo/common.gazebo.xacro (robot description, xacro)
@@ -5,4 +5,5 @@
   xmlns:interface="http://playerstage.sourceforge.net/gazebo/xmlschema/#interface"
   xmlns:xacro="http://ros.org/wiki/xacro">
+  <xacro:property name="SIMPLE_ROBOT_RADIUS" value="0.4" />
   <xacro:macro name="gazebo_segbot_base_link_surface">
     <gazebo reference="base_link">
@@ -28,7 +29,7 @@
   </xacro:macro>
   <xacro:macro name="segbot_base_link_cylinder">
-    <origin xyz="0 0 0" rpy="0 0 0" />
+    <origin xyz="0 0 0.2" rpy="0 0 0" />
     <geometry>
-      <cylinder length="0.4330" radius="0.6" />
+      <cylinder length="0.8330" radius="${SIMPLE_ROBOT_RADIUS}" />
     </geometry>
   </xacro:macro>
@@ -73,24 +74,19 @@
     </controller:gazebo_ros_controller_manager>
   </xacro:macro>
-  <xacro:macro name="gazebo_segbot_drive_parameters">
-    <alwaysOn>true</alwaysOn>
-    <updateRate>100.0</updateRate>
-    <leftJoint>base_link_right_wheel_joint</leftJoint>
-    <rightJoint>base_link_left_wheel_joint</rightJoint>
-    <wheelSeparation>0.5380</wheelSeparation>
-    <wheelDiameter>0.2410</wheelDiameter>
-    <torque>20</torque>
-    <topicName>cmd_vel</topicName>
-    <!-- <interface:position name="position_iface_0"/> -->
-  </xacro:macro>
-  <xacro:macro name="gazebo_segbot_simple_drive_plugin">
+  <xacro:macro name="gazebo_segbot_drive_plugin" params="use_simple_model update_rate">
     <controller:segbotdrive_plugin name="differential_drive_controller" plugin="libsegbotdrive_plugin.so">
+      <alwaysOn>true</alwaysOn>
+      <updateRate>${update_rate}</updateRate>
+      <leftJoint>base_link_right_wheel_joint</leftJoint>
+      <rightJoint>base_link_left_wheel_joint</rightJoint>
+      <wheelSeparation>0.5380</wheelSeparation>
+      <wheelDiameter>0.2410</wheelDiameter>
+      <torque>20</torque>
+      <topicName>cmd_vel</topicName>
       <gazebo_segbot_drive_parameters />
-      <useSimpleModel>true</useSimpleModel>
-    </controller:segbotdrive_plugin>
-  </xacro:macro>
-  <xacro:macro name="gazebo_segbot_drive_plugin">
-    <controller:segbotdrive_plugin name="differential_drive_controller" plugin="libsegbotdrive_plugin.so">
-      <gazebo_segbot_drive_parameters />
+      <useSimpleModel>${use_simple_model}</useSimpleModel>
+      <simpleMapTopic>map</simpleMapTopic>
+      <simpleModelRadius>${SIMPLE_ROBOT_RADIUS}</simpleModelRadius>
+      <simpleRobotPadding>0.025</simpleRobotPadding>
     </controller:segbotdrive_plugin>
   </xacro:macro>

File: segbot_description/gazebo/full_collision.gazebo.xacro (robot description, xacro)
@@ -30,5 +30,5 @@
   <xacro:macro name="gazebo_segbot_ros_controllers">
     <gazebo>
-      <xacro:gazebo_segbot_drive_plugin />
+      <xacro:gazebo_segbot_drive_plugin use_simple_model="false" update_rate="100" />
       <xacro:gazebo_segbot_controllers_common />
     </gazebo>

File: segbot_description/gazebo/simple_collision.gazebo.xacro (robot description, xacro)
@@ -30,5 +30,5 @@
   <xacro:macro name="gazebo_segbot_ros_controllers">
     <gazebo>
-      <xacro:gazebo_segbot_simple_drive_plugin />
+      <xacro:gazebo_segbot_drive_plugin use_simple_model="true" update_rate="1000" />
       <xacro:gazebo_segbot_controllers_common />
     </gazebo>

File: segbot_description/urdf/segbot_base.urdf.xacro (robot description, xacro)
@@ -19,5 +19,5 @@
       <child link="base_link" />
     </joint>
-    <!-- This is the robot origin, middle of the wheel axis -->
+    <!-- This is the robot origin, center of the 2 wheels (axis of rotation) -->
     <link name="base_link">
       <inertial>
@@ -36,20 +36,5 @@
     </link>
     <xacro:gazebo_segbot_base_link_surface />
-    <!-- pushing the center of mass of the body to a more appropriate pos -->
-    <!-- <joint name="base_center_of_mass_joint" type="fixed"> -->
-    <!--   <origin xyz="-0.1 0 -0.075" rpy="0 0 0" /> -->
-    <!--   <parent link="base_link"/> -->
-    <!--   <child link="base_center_of_mass_link" /> -->
-    <!-- </joint> -->
-    <!-- <link name="base_center_of_mass_link"> -->
-    <!--   <inertial> -->
-    <!--     <mass value="30" /> -->
-    <!--     <origin xyz="0 0 0" /> -->
-    <!--     <inertia ixx="1.0" ixy="0.0" ixz="0.0" -->
-    <!--       iyy="1.0" iyz="0.0"  -->
-    <!--       izz="1.0" /> -->
-    <!--   </inertial> -->
-    <!-- </link> -->
-    <!-- castor joint and wheel -->
+    <!-- castor joint -->
     <joint name="base_caster_support_joint" type="continuous">
       <origin xyz="-0.3292 0 -0.0485" rpy="0 0 0" />
@@ -87,4 +72,5 @@
       <kd  value="1.0" />
     </gazebo>
+    <!-- castor wheel -->
     <joint name="caster_wheel_joint" type="continuous">
       <origin xyz="-0.0397 0 -0.0918" rpy="0 0 0" />

Commit message: fixed collision issues between simple and full model

File: segbot_description/gazebo/common.gazebo.xacro (robot description, xacro)
@@ -22,39 +22,11 @@
     </gazebo>
   </xacro:macro>
-  <xacro:macro name="segbot_base_link_mesh">
-    <origin xyz="0 0 0" rpy="0 0 0" />
-    <geometry>
-      <mesh filename="package://segbot_description/meshes/rmp50-base-link.dae" scale="0.0254 0.0254 0.0254"/>
-    </geometry>
-  </xacro:macro>
-  <xacro:macro name="segbot_base_link_cylinder">
-    <origin xyz="0 0 0.2" rpy="0 0 0" />
-    <geometry>
-      <cylinder length="0.8330" radius="${SIMPLE_ROBOT_RADIUS}" />
-    </geometry>
-  </xacro:macro>
-  <xacro:macro name="segbot_castor_wheel_link_mesh">
-    <origin xyz="0 0 0" rpy="0 0 0" />
-    <geometry>
-      <mesh filename="package://segbot_description/meshes/rmp50-castor-wheel.dae" scale="0.0254 0.0254 0.0254"/>
-    </geometry>
-  </xacro:macro>
-  <xacro:macro name="segbot_collision_none">
-    <origin xyz="0 0 0" rpy="0 0 0" />
-    <geometry>
-      <box size="0.01 0.01 0.01" />
-    </geometry>
-  </xacro:macro>
-  <xacro:macro name="segbot_castor_support_link_mesh">
-    <origin xyz="0 0 0" rpy="0 0 0" />
-    <geometry>
-      <mesh filename="package://segbot_description/meshes/rmp50-castor-link.dae" scale="0.0254 0.0254 0.0254"/>
-    </geometry>
-  </xacro:macro>
-  <xacro:macro name="segbot_wheel_mesh" params="suffix">
-    <origin xyz="0 0 0" rpy="0 0 0" />
-    <geometry>
-      <mesh filename="package://segbot_description/meshes/rmp50-${suffix}-wheel.dae" scale="0.0254 0.0254 0.0254"/>
-    </geometry>
+  <xacro:macro name="segbot_simple_collision">
+    <collision>
+      <origin xyz="0 0 0.2" rpy="0 0 0" />
+      <geometry>
+        <cylinder length="0.8330" radius="${SIMPLE_ROBOT_RADIUS}" />
+      </geometry>
+    </collision>
   </xacro:macro>
   <xacro:macro name="gazebo_segbot_wheel_surface" params="parent suffix">

File: segbot_description/gazebo/full_collision.gazebo.xacro (robot description, xacro)
@@ -4,27 +4,67 @@
   <!-- Included URDF Files -->
   <include filename="$(find segbot_description)/gazebo/common.gazebo.xacro" />
-  <xacro:macro name="segbot_base_link_visual" >
-    <xacro:segbot_base_link_mesh />
-  </xacro:macro>
   <xacro:macro name="segbot_base_link_collision" >
-    <xacro:segbot_base_link_mesh />
-  </xacro:macro>
-  <xacro:macro name="segbot_castor_support_link_visual" >
-    <xacro:segbot_castor_support_link_mesh />
+    <collision>
+      <origin xyz="0 0 0" rpy="0 0 0" />
+      <geometry>
+        <mesh filename="package://segbot_description/meshes/rmp50-base-link.dae" scale="0.0254 0.0254 0.0254"/>
+      </geometry>
+    </collision>
   </xacro:macro>
   <xacro:macro name="segbot_castor_support_link_collision" >
-    <xacro:segbot_castor_support_link_mesh />
-  </xacro:macro>
-  <xacro:macro name="segbot_castor_wheel_link_visual" >
-    <xacro:segbot_castor_wheel_link_mesh />
+    <collision>
+      <origin xyz="0 0 0" rpy="0 0 0" />
+      <geometry>
+        <mesh filename="package://segbot_description/meshes/rmp50-castor-link.dae" scale="0.0254 0.0254 0.0254"/>
+      </geometry>
+    </collision>
   </xacro:macro>
   <xacro:macro name="segbot_castor_wheel_link_collision" >
-    <xacro:segbot_castor_wheel_link_mesh />
-  </xacro:macro>
-  <xacro:macro name="segbot_wheel_visual" params="suffix">
-    <xacro:segbot_wheel_mesh suffix="${suffix}" />
+    <collision>
+      <origin xyz="0 0 0" rpy="0 0 0" />
+      <geometry>
+        <mesh filename="package://segbot_description/meshes/rmp50-castor-wheel.dae" scale="0.0254 0.0254 0.0254"/>
+      </geometry>
+    </collision>
   </xacro:macro>
   <xacro:macro name="segbot_wheel_collision" params="suffix">
-    <xacro:segbot_wheel_mesh suffix="${suffix}" />
+    <collision>
+      <origin xyz="0 0 0" rpy="0 0 0" />
+      <geometry>
+        <mesh filename="package://segbot_description/meshes/rmp50-${suffix}-wheel.dae" scale="0.0254 0.0254 0.0254"/>
+      </geometry>
+    </collision>
+  </xacro:macro>
+  <xacro:macro name="segbot_battery_box_collision">
+    <collision>
+      <origin xyz="0 0 ${5.5*INCH_TO_M}" rpy="0 0 0"/>
+      <geometry>
+        <box size="${7*INCH_TO_M} ${14*INCH_TO_M} ${11*INCH_TO_M}" />
+      </geometry>
+    </collision>
+  </xacro:macro>
+  <xacro:macro name="aluminium_sheet_collision" params="thickness length width">
+    <collision>
+      <origin xyz="0 0 ${thickness/2}" rpy="0 0 0"/>
+      <geometry>
+        <box size="${length} ${width} ${thickness}" />
+      </geometry>
+    </collision>
+  </xacro:macro>
+  <xacro:macro name="beam_8020_collision" params="length">
+    <collision>
+      <origin xyz="0 0 ${length/2}" rpy="0 0 0"/>
+      <geometry>
+        <box size="${1*INCH_TO_M} ${1*INCH_TO_M} ${length}" />
+      </geometry>
+    </collision>
+  </xacro:macro>
+  <xacro:macro name="standoff_632_collision" params="length">
+    <collision>
+      <origin xyz="0 0 ${length/2}" rpy="0 0 0"/>
+      <geometry>
+        <cylinder length="${length}" radius="0.003175" />
+      </geometry>
+    </collision>
   </xacro:macro>
   <xacro:macro name="gazebo_segbot_ros_controllers">

File: segbot_description/gazebo/simple_collision.gazebo.xacro (robot description, xacro)
@@ -4,27 +4,27 @@
   <!-- Included URDF Files -->
   <include filename="$(find segbot_description)/gazebo/common.gazebo.xacro" />
-  <xacro:macro name="segbot_base_link_visual" >
-    <xacro:segbot_base_link_mesh />
-  </xacro:macro>
   <xacro:macro name="segbot_base_link_collision" >
-    <xacro:segbot_base_link_cylinder />
-  </xacro:macro>
-  <xacro:macro name="segbot_castor_support_link_visual" >
-    <xacro:segbot_castor_support_link_mesh />
+    <xacro:segbot_simple_collision />
   </xacro:macro>
   <xacro:macro name="segbot_castor_support_link_collision" >
-    <xacro:segbot_collision_none />
-  </xacro:macro>
-  <xacro:macro name="segbot_castor_wheel_link_visual" >
-    <xacro:segbot_castor_wheel_link_mesh />
+    <!-- simple model has no collision -->
   </xacro:macro>
   <xacro:macro name="segbot_castor_wheel_link_collision" >
-    <xacro:segbot_collision_none />
-  </xacro:macro>
-  <xacro:macro name="segbot_wheel_visual" params="suffix">
-    <xacro:segbot_wheel_mesh suffix="${suffix}" />
+    <!-- simple model has no collision -->
   </xacro:macro>
   <xacro:macro name="segbot_wheel_collision" params="suffix">
-    <xacro:segbot_collision_none />
+    <!-- simple model has no collision -->
+  </xacro:macro>
+  <xacro:macro name="segbot_battery_box_collision">
+    <!-- simple model has no collision -->
+  </xacro:macro>
+  <xacro:macro name="aluminium_sheet_collision" params="thickness length width">
+    <!-- simple model has no collision -->
+  </xacro:macro>
+  <xacro:macro name="beam_8020_collision" params="length">
+    <!-- simple model has no collision -->
+  </xacro:macro>
+  <xacro:macro name="standoff_632_collision" params="length">
+    <!-- simple model has no collision -->
   </xacro:macro>
   <xacro:macro name="gazebo_segbot_ros_controllers">

File: segbot_description/urdf/components/aluminium_sheet.urdf.xacro (robot description, xacro)
@@ -22,10 +22,5 @@
         <material name="dark_grey" />
       </visual>
-      <collision>
-        <origin xyz="0 0 ${thickness/2}" rpy="0 0 0"/>
-        <geometry>
-          <box size="${length} ${width} ${thickness}" />
-        </geometry>
-      </collision>
+      <xacro:aluminium_sheet_collision thickness="${thickness}" length="${length}" width="${width}"/>
     </link>
     <gazebo reference="${name}_link">

File: segbot_description/urdf/components/beam_8020.urdf.xacro (robot description, xacro)
@@ -24,10 +24,5 @@
         <material name="light_grey" />
       </visual>
-      <collision>
-        <origin xyz="0 0 ${length/2}" rpy="0 0 0"/>
-        <geometry>
-          <box size="${1*INCH_TO_M} ${1*INCH_TO_M} ${length}" />
-        </geometry>
-      </collision>
+      <xacro:beam_8020_collision length="${length}" />
     </link>
     <gazebo reference="${name}_link">

File: segbot_description/urdf/components/standoff_632.urdf.xacro (robot description, xacro)
@@ -22,10 +22,4 @@
         <material name="light_grey" />
       </visual>
-      <collision>
-        <origin xyz="0 0 ${length/2}" rpy="0 0 0"/>
-        <geometry>
-          <cylinder length="${length}" radius="0.003175" />
-        </geometry>
-      </collision>
     </link>
     <gazebo reference="${name}_link">

File: segbot_description/urdf/segbot_base.urdf.xacro (robot description, xacro)
@@ -29,9 +29,10 @@
       </inertial>
       <visual>
-        <xacro:segbot_base_link_visual />
+        <origin xyz="0 0 0" rpy="0 0 0" />
+        <geometry>
+          <mesh filename="package://segbot_description/meshes/rmp50-base-link.dae" scale="0.0254 0.0254 0.0254"/>
+        </geometry>
       </visual>
-      <collision>
-        <xacro:segbot_base_link_collision />
-      </collision>
+      <xacro:segbot_base_link_collision />
     </link>
     <xacro:gazebo_segbot_base_link_surface />
@@ -60,9 +61,10 @@
       </inertial>
       <visual>
-        <segbot_castor_support_link_visual />
+        <origin xyz="0 0 0" rpy="0 0 0" />
+        <geometry>
+          <mesh filename="package://segbot_description/meshes/rmp50-castor-link.dae" scale="0.0254 0.0254 0.0254"/>
+        </geometry>
       </visual>
-      <collision>
-        <segbot_castor_support_link_collision />
-      </collision>
+      <xacro:segbot_castor_support_link_collision />
     </link>
     <gazebo reference="base_caster_support_link">
@@ -96,9 +98,10 @@
       </inertial>
       <visual>
-        <xacro:segbot_castor_wheel_link_visual />
+        <origin xyz="0 0 0" rpy="0 0 0" />
+        <geometry>
+          <mesh filename="package://segbot_description/meshes/rmp50-castor-wheel.dae" scale="0.0254 0.0254 0.0254"/>
+        </geometry>
       </visual>
-      <collision>
-        <xacro:segbot_castor_wheel_link_collision />
-      </collision>
+      <xacro:segbot_castor_wheel_link_collision />
     </link>
     <xacro:gazebo_segbot_castor_wheel_link_surface />

File: segbot_description/urdf/segbot_chassis.urdf.xacro (robot description, xacro)
@@ -41,10 +41,5 @@
         <material name="almost_black" />
       </visual>
-      <collision>
-        <origin xyz="0 0 ${5.5*INCH_TO_M}" rpy="0 0 0"/>
-        <geometry>
-          <box size="${7*INCH_TO_M} ${14*INCH_TO_M} ${11*INCH_TO_M}" />
-        </geometry>
-      </collision>
+      <xacro:segbot_battery_box_collision />
     </link>
     <gazebo reference="battery_box_link">

File: segbot_description/urdf/segbot_wheel.urdf.xacro (robot description, xacro)
@@ -21,9 +21,10 @@
       </inertial>
       <visual>
-        <xacro:segbot_wheel_visual suffix="${suffix}" />
+        <origin xyz="0 0 0" rpy="0 0 0" />
+        <geometry>
+          <mesh filename="package://segbot_description/meshes/rmp50-${suffix}-wheel.dae" scale="0.0254 0.0254 0.0254"/>
+        </geometry>
       </visual>
-      <collision>
-        <xacro:segbot_wheel_collision suffix="${suffix}" />
-      </collision>
+      <xacro:segbot_wheel_collision suffix="${suffix}" />
     </link>
     <xacro:gazebo_segbot_wheel_surface parent="${parent}" suffix="${suffix}" />

File: segbot_description/urdf/sensors/hokuyo_04lx_laser.urdf.xacro (robot description, xacro)
@@ -21,15 +21,13 @@
         <origin xyz="0 0 0" rpy="0 0 0" />
         <geometry>
-          <!-- <box size="0.05 0.05 0.07" /> -->
           <mesh filename="package://segbot_description/meshes/hokuyo.dae" scale="0.0254 0.0254 0.0254" />
         </geometry>
       </visual>
-      <collision>
-        <origin xyz="0 0 0" rpy="0 0 0" />
-        <geometry>
-          <!-- <box size="0.05 0.05 0.07" /> -->
-          <mesh filename="package://segbot_description/meshes/hokuyo.dae" scale="0.0254 0.0254 0.0254" />
-        </geometry>
-      </collision>
+      <!-- <collision> -->
+      <!--   <origin xyz="0 0 0" rpy="0 0 0" /> -->
+      <!--   <geometry> -->
+      <!--     <mesh filename="package://segbot_description/meshes/hokuyo.dae" scale="0.0254 0.0254 0.0254" /> -->
+      <!--   </geometry> -->
+      <!-- </collision> -->
     </link>
     <!-- go from the base of the laser to the actual sensor location -->

File: segbot_description/urdf/sensors/kinect_camera.urdf.xacro (robot description, xacro)
@@ -25,10 +25,10 @@
         </geometry>
       </visual>
-      <collision>
-        <origin xyz="0.0 0.012 0" rpy="0 0 0"/>
-        <geometry>
-          <mesh filename="package://pr2_description/meshes/sensors/kinect_v0/kinect.dae" scale="0.001 0.001 0.001" />
-        </geometry>
-      </collision>
+      <!-- <collision> -->
+      <!--   <origin xyz="0.0 0.012 0" rpy="0 0 0"/> -->
+      <!--   <geometry> -->
+      <!--     <mesh filename="package://pr2_description/meshes/sensors/kinect_v0/kinect.dae" scale="0.001 0.001 0.001" /> -->
+      <!--   </geometry> -->
+      <!-- </collision> -->
     </link>
     <!-- extensions -->

Commit message: using the significantly improved (unpublished) object controller plugin from bwi_gazebo_entities for the simple controller

File: segbot_description/gazebo/common.gazebo.xacro (robot description, xacro)
@@ -46,5 +46,5 @@
     </controller:gazebo_ros_controller_manager>
   </xacro:macro>
-  <xacro:macro name="gazebo_segbot_drive_plugin" params="use_simple_model update_rate">
+  <xacro:macro name="gazebo_segbot_drive_plugin" params="update_rate">
     <controller:segbotdrive_plugin name="differential_drive_controller" plugin="libsegbotdrive_plugin.so">
       <alwaysOn>true</alwaysOn>
@@ -56,10 +56,15 @@
       <torque>20</torque>
       <topicName>cmd_vel</topicName>
-      <gazebo_segbot_drive_parameters />
-      <useSimpleModel>${use_simple_model}</useSimpleModel>
-      <simpleMapTopic>map</simpleMapTopic>
-      <simpleModelRadius>${SIMPLE_ROBOT_RADIUS}</simpleModelRadius>
-      <simpleRobotPadding>0.025</simpleRobotPadding>
     </controller:segbotdrive_plugin>
   </xacro:macro>
+  <xacro:macro name="gazebo_object_controller_plugin" params="update_rate">
+    <controller:object_controller_plugin name="object_controller" plugin="libobject_controller_plugin.so">
+      <alwaysOn>true</alwaysOn>
+      <updateRate>${update_rate}</updateRate>
+      <topicName>cmd_vel</topicName>
+      <mapTopic>map</mapTopic>
+      <modelRadius>${SIMPLE_ROBOT_RADIUS}</modelRadius>
+      <modelPadding>0.025</modelPadding>
+    </controller:object_controller_plugin>
+  </xacro:macro>
 </root>

File: segbot_description/gazebo/full_collision.gazebo.xacro (robot description, xacro)
@@ -70,6 +70,6 @@
   <xacro:macro name="gazebo_segbot_ros_controllers">
     <gazebo>
-      <xacro:gazebo_segbot_drive_plugin use_simple_model="false" update_rate="100" />
-      <xacro:gazebo_segbot_controllers_common />
+      <xacro:gazebo_segbot_drive_plugin update_rate="100" />
+      <!-- <xacro:gazebo_segbot_controllers_common /> -->
     </gazebo>
   </xacro:macro>

File: segbot_description/gazebo/simple_collision.gazebo.xacro (robot description, xacro)
@@ -30,6 +30,6 @@
   <xacro:macro name="gazebo_segbot_ros_controllers">
     <gazebo>
-      <xacro:gazebo_segbot_drive_plugin use_simple_model="true" update_rate="1000" />
-      <xacro:gazebo_segbot_controllers_common />
+      <xacro:gazebo_object_controller_plugin update_rate="50" />
+      <!-- <xacro:gazebo_segbot_controllers_common /> -->
     </gazebo>
   </xacro:macro>

Commit message: reduced model size for the simple robot model

File: segbot_description/gazebo/common.gazebo.xacro (robot description, xacro)
@@ -5,5 +5,5 @@
   xmlns:interface="http://playerstage.sourceforge.net/gazebo/xmlschema/#interface"
   xmlns:xacro="http://ros.org/wiki/xacro">
-  <xacro:property name="SIMPLE_ROBOT_RADIUS" value="0.4" />
+  <xacro:property name="SIMPLE_ROBOT_RADIUS" value="0.3" />
   <xacro:macro name="gazebo_segbot_base_link_surface">
     <gazebo reference="base_link">

Commit message: reduced the radius of the robot further

File: segbot_description/gazebo/common.gazebo.xacro (robot description, xacro)
@@ -5,5 +5,5 @@
   xmlns:interface="http://playerstage.sourceforge.net/gazebo/xmlschema/#interface"
   xmlns:xacro="http://ros.org/wiki/xacro">
-  <xacro:property name="SIMPLE_ROBOT_RADIUS" value="0.3" />
+  <xacro:property name="SIMPLE_ROBOT_RADIUS" value="0.25" />
   <xacro:macro name="gazebo_segbot_base_link_surface">
     <gazebo reference="base_link">
@@ -65,5 +65,5 @@
       <mapTopic>map</mapTopic>
       <modelRadius>${SIMPLE_ROBOT_RADIUS}</modelRadius>
-      <modelPadding>0.025</modelPadding>
+      <modelPadding>0.05</modelPadding>
     </controller:object_controller_plugin>
   </xacro:macro>
