Commit message: updating all plugins to sdf

File: segbot_description/gazebo/common.gazebo.xacro (robot description, xacro)
@@ -1,7 +1,4 @@
 <?xml version="1.0"?>
 <root
-  xmlns:sensor="http://playerstage.sourceforge.net/gazebo/xmlschema/#sensor"
-  xmlns:controller="http://playerstage.sourceforge.net/gazebo/xmlschema/#controller"
-  xmlns:interface="http://playerstage.sourceforge.net/gazebo/xmlschema/#interface"
   xmlns:xacro="http://ros.org/wiki/xacro">
   <xacro:property name="SIMPLE_ROBOT_RADIUS" value="0.25" />
@@ -40,12 +37,11 @@
   <xacro:macro name="gazebo_segbot_controllers_common">
     <canonicalBody>base_footprint</canonicalBody>
-    <controller:gazebo_ros_controller_manager name="gazebo_ros_controller_manager" plugin="libgazebo_ros_controller_manager.so">
+    <plugin name="gazebo_ros_controller_manager" filename="libgazebo_ros_controller_manager.so">
       <alwaysOn>true</alwaysOn>
       <updateRate>5.0</updateRate>
-      <interface:audio name="gazebo_ros_controller_manager_dummy_iface" />
-    </controller:gazebo_ros_controller_manager>
+    </plugin>
   </xacro:macro>
   <xacro:macro name="gazebo_segbot_drive_plugin" params="update_rate">
-    <controller:segbotdrive_plugin name="differential_drive_controller" plugin="libsegbotdrive_plugin.so">
+    <plugin name="differential_drive_controller" filename="libsegbotdrive_plugin.so">
       <alwaysOn>true</alwaysOn>
       <updateRate>${update_rate}</updateRate>
@@ -56,8 +52,8 @@
       <torque>20</torque>
       <topicName>cmd_vel</topicName>
-    </controller:segbotdrive_plugin>
+    </plugin>
   </xacro:macro>
   <xacro:macro name="gazebo_object_controller_plugin" params="update_rate">
-    <controller:object_controller_plugin name="object_controller" plugin="libobject_controller_plugin.so">
+    <plugin name="object_controller" filename="libobject_controller_plugin.so">
       <alwaysOn>true</alwaysOn>
       <updateRate>${update_rate}</updateRate>
@@ -66,5 +62,5 @@
       <modelRadius>${SIMPLE_ROBOT_RADIUS}</modelRadius>
       <modelPadding>0.05</modelPadding>
-    </controller:object_controller_plugin>
+    </plugin>
   </xacro:macro>
 </root>

File: segbot_description/urdf/components/laptop.urdf.xacro (robot description, xacro)
@@ -59,11 +59,11 @@
     </link>
     <gazebo reference="${name}_screen_link">
-      <visual>
-        <controller:laptop_visual_plugin name="${name}_video_controller" filename="libgazebo_ros_video.so">
-          <height>120</height>
-          <width>160</width>
-          <topicName>image</topicName>
-        </controller:laptop_visual_plugin>
-    </visual>
+    <!--   <visual> -->
+    <!--     <controller:laptop_visual_plugin name="${name}_video_controller" filename="libgazebo_ros_video.so"> -->
+    <!--       <height>120</height> -->
+    <!--       <width>160</width> -->
+    <!--       <topicName>image</topicName> -->
+    <!--     </controller:laptop_visual_plugin> -->
+    <!-- </visual> -->
       <material>Gazebo/Grey</material>
       <mu1 value="100.0" />

File: segbot_description/urdf/sensors/hokuyo_04lx_laser.gazebo.xacro (robot description, xacro)
@@ -1,30 +1,35 @@
 <?xml version="1.0"?>
-<root xmlns:sensor="http://playerstage.sourceforge.net/gazebo/xmlschema/#sensor"
-      xmlns:controller="http://playerstage.sourceforge.net/gazebo/xmlschema/#controller"
-      xmlns:interface="http://playerstage.sourceforge.net/gazebo/xmlschema/#interface"
+<root
       xmlns:xacro="http://ros.org/wiki/xacro">
   <xacro:macro name="hokuyo_04lx_laser_gazebo" params="name ros_topic update_rate min_angle max_angle">
     <gazebo reference="${name}_link">
-      <sensor:ray name="${name}">
-        <rayCount>640</rayCount>
-        <rangeCount>640</rangeCount>
-        <laserCount>1</laserCount>
-        <origin>0.0 0.0 0.0</origin>
-        <displayRays>false</displayRays>
-        <minAngle>${min_angle*180.0/M_PI}</minAngle>
-        <maxAngle>${max_angle*180.0/M_PI}</maxAngle>
-        <minRange>0.02</minRange>
-        <maxRange>4.0</maxRange>
-        <resRange>0.03</resRange>
-        <updateRate>${update_rate}</updateRate>
-        <controller:gazebo_ros_laser name="gazebo_ros_${name}_controller" plugin="libgazebo_ros_laser.so">
-          <gaussianNoise>0.03</gaussianNoise>
+      <sensor type="ray" name="${name}">
+        <always_on>true</always_on>
+        <update_rate>${update_rate}</update_rate>
+        <pose>0 0 0 0 0 0</pose>
+        <visualize>false</visualize>
+        <ray>
+          <scan>
+            <horizontal>
+              <samples>640</samples>
+              <resolution>1</resolution>
+              <min_angle>${min_angle}</min_angle>
+              <max_angle>${max_angle}</max_angle>
+            </horizontal>
+          </scan>
+          <range>
+            <min>0.02</min>
+            <max>4.0</max>
+            <resolution>0.03</resolution>
+          </range>
+        </ray>
+        <plugin name="gazebo_ros_${name}_controller" filename="libgazebo_ros_laser.so">
+          <gaussianNoise>0.0</gaussianNoise>
           <alwaysOn>true</alwaysOn>
           <updateRate>${update_rate}</updateRate>
           <topicName>${ros_topic}</topicName>
           <frameName>${name}_link</frameName>
-          <interface:laser name="gazebo_ros_${name}_iface" />
-        </controller:gazebo_ros_laser>
-      </sensor:ray>
+        </plugin>
+      </sensor>
     </gazebo>
   </xacro:macro>

File: segbot_description/urdf/sensors/kinect_camera.gazebo.xacro (robot description, xacro)
@@ -6,13 +6,20 @@
 <xacro:macro name="kinect_camera_gazebo" params="name">
   <gazebo reference="${name}_link">
-    <sensor:camera name="${name}_link_sensor">
-      <imageFormat>R8G8B8</imageFormat>
-      <imageSize>640 480</imageSize>
-      <hfov>57</hfov>
-      <nearClip>0.01</nearClip>
-      <farClip>5</farClip>
-      <updateRate>20.0</updateRate>
-      <baseline>0.2</baseline>
-      <controller:gazebo_ros_openni_kinect name="${name}_frame_controller" plugin="libgazebo_ros_openni_kinect.so">
+    <sensor:camera type="depth" name="${name}_link_sensor">
+      <always_on>true</always_on>
+      <update_rate>20.0</update_rate>
+      <camera>
+        <horizontal_fov>${57.0*M_PI/180.0}</horizontal_fov>
+        <image>
+          <format>R8G8B8</format>
+          <width>640</width>
+          <height>480</height>
+        </image>
+        <clip>
+          <near>0.01</near>
+          <far>5</far>
+        </clip>
+      </camera>
+      <plugin name="${name}_frame_controller" filename="libgazebo_ros_openni_kinect.so">
         <alwaysOn>true</alwaysOn>
         <updateRate>20.0</updateRate>
@@ -30,6 +37,6 @@
         <distortionT1>0.00000001</distortionT1>
         <distortionT2>0.00000001</distortionT2>
-      </controller:gazebo_ros_openni_kinect>
-    </sensor:camera>
+      </plugin>
+    </sensor>
   </gazebo>
 </xacro:macro>

Commit message: updating dependencies now that libsegwayrmp and segway_rmp have been successfully catkinized

File: segbot_description/gazebo/common.gazebo.xacro (robot description, xacro)
@@ -2,5 +2,5 @@
 <root
   xmlns:xacro="http://ros.org/wiki/xacro">
-  <xacro:property name="SIMPLE_ROBOT_RADIUS" value="0.25" />
+  <xacro:property name="SIMPLE_ROBOT_RADIUS" value="0.05" />
   <xacro:macro name="gazebo_segbot_base_link_surface">
     <gazebo reference="base_link">

File: segbot_description/urdf/components/laptop.urdf.xacro (robot description, xacro)
@@ -59,11 +59,11 @@
     </link>
     <gazebo reference="${name}_screen_link">
-    <!--   <visual> -->
-    <!--     <controller:laptop_visual_plugin name="${name}_video_controller" filename="libgazebo_ros_video.so"> -->
-    <!--       <height>120</height> -->
-    <!--       <width>160</width> -->
-    <!--       <topicName>image</topicName> -->
-    <!--     </controller:laptop_visual_plugin> -->
-    <!-- </visual> -->
+      <visual>
+        <plugin name="${name}_video_controller" filename="libgazebo_ros_video.so">
+          <height>120</height>
+          <width>160</width>
+          <topicName>image</topicName>
+        </plugin>
+      </visual>
       <material>Gazebo/Grey</material>
       <mu1 value="100.0" />

Commit message: reverted robot radius

File: segbot_description/gazebo/common.gazebo.xacro (robot description, xacro)
@@ -2,5 +2,5 @@
 <root
   xmlns:xacro="http://ros.org/wiki/xacro">
-  <xacro:property name="SIMPLE_ROBOT_RADIUS" value="0.05" />
+  <xacro:property name="SIMPLE_ROBOT_RADIUS" value="0.30" />
   <xacro:macro name="gazebo_segbot_base_link_surface">
     <gazebo reference="base_link">

Commit message: significantly cleaned up segbot_description. need new version of xacro to be released before merging with devel. closes #7, #12

File: segbot_description/gazebo/common.gazebo.xacro (robot description, xacro)
@@ -2,37 +2,4 @@
 <root
   xmlns:xacro="http://ros.org/wiki/xacro">
-  <xacro:property name="SIMPLE_ROBOT_RADIUS" value="0.30" />
-  <xacro:macro name="gazebo_segbot_base_link_surface">
-    <gazebo reference="base_link">
-      <mu1 value="100.0" />
-      <mu2 value="100.0" />
-      <kp  value="1000000.0" />
-      <kd  value="1.0" />
-    </gazebo>
-  </xacro:macro>
-  <xacro:macro name="gazebo_segbot_castor_wheel_link_surface">
-    <gazebo reference="caster_wheel_link">
-      <mu1 value="10.0" />
-      <mu2 value="10.0" />
-      <kp  value="1000000.0" />
-      <kd  value="1.0" />
-    </gazebo>
-  </xacro:macro>
-  <xacro:macro name="segbot_simple_collision">
-    <collision>
-      <origin xyz="0 0 0.2" rpy="0 0 0" />
-      <geometry>
-        <cylinder length="0.8330" radius="${SIMPLE_ROBOT_RADIUS}" />
-      </geometry>
-    </collision>
-  </xacro:macro>
-  <xacro:macro name="gazebo_segbot_wheel_surface" params="parent suffix">
-    <gazebo reference="${parent}_${suffix}_wheel_link" >
-      <mu1 value="10.0" />
-      <mu2 value="10.0" />
-      <kp  value="1000000.0" />
-      <kd  value="1.0" />
-    </gazebo>
-  </xacro:macro>
   <xacro:macro name="gazebo_segbot_controllers_common">
     <canonicalBody>base_footprint</canonicalBody>
@@ -43,25 +10,6 @@
   </xacro:macro>
   <xacro:macro name="gazebo_segbot_drive_plugin" params="update_rate">
-    <plugin name="differential_drive_controller" filename="libgazebo_ros_diff_drive.so">
-      <updateRate>${update_rate}</updateRate>
-      <leftJoint>base_link_right_wheel_joint</leftJoint>
-      <rightJoint>base_link_left_wheel_joint</rightJoint>
-      <wheelSeparation>0.5380</wheelSeparation>
-      <wheelDiameter>0.2410</wheelDiameter>
-      <torque>20</torque>
-      <commandTopic>cmd_vel</commandTopic>
-      <odometryTopic>odom</odometryTopic>
-      <odometryFrame>odom</odometryFrame>
-      <robotBaseFrame>base_footprint</robotBaseFrame>
-    </plugin>
   </xacro:macro>
   <xacro:macro name="gazebo_object_controller_plugin" params="update_rate">
-    <plugin name="object_controller" filename="libgazebo_ros_planar_move.so">
-      <commandTopic>cmd_vel</commandTopic>
-      <odometryTopic>odom</odometryTopic>
-      <odometryFrame>odom</odometryFrame>
-      <robotBaseFrame>base_footprint</robotBaseFrame>
-      <odometryRate>${update_rate}</odometryRate>
-    </plugin>
   </xacro:macro>
 </root>

File: segbot_description/gazebo/full_collision.gazebo.xacro (robot description, xacro)
@@ -3,5 +3,5 @@
   xmlns:xacro="http://ros.org/wiki/xacro">
   <!-- Included URDF Files -->
-  <include filename="$(find segbot_description)/gazebo/common.gazebo.xacro" />
+  <xacro:include filename="$(find segbot_description)/gazebo/common.gazebo.xacro" />
   <xacro:macro name="segbot_base_link_collision" >
     <collision>

File: segbot_description/gazebo/simple_collision.gazebo.xacro (robot description, xacro)
@@ -3,5 +3,5 @@
   xmlns:xacro="http://ros.org/wiki/xacro">
   <!-- Included URDF Files -->
-  <include filename="$(find segbot_description)/gazebo/common.gazebo.xacro" />
+  <xacro:include filename="$(find segbot_description)/gazebo/common.gazebo.xacro" />
   <xacro:macro name="segbot_base_link_collision" >
     <xacro:segbot_simple_collision />

File: segbot_description/robots/segbot.urdf.xacro (robot description, xacro)
@@ -3,9 +3,9 @@
        xmlns:xacro="http://ros.org/wiki/xacro">
   <!-- Included URDF Files -->
-  <include filename="$(find segbot_description)/urdf/common.urdf.xacro" />
-  <include filename="$(find segbot_description)/gazebo/full_collision.gazebo.xacro" />
-  <include filename="$(find segbot_description)/urdf/segbot_base.urdf.xacro" />
-  <include filename="$(find segbot_description)/urdf/segbot_chassis.urdf.xacro" />
-  <include filename="$(find segbot_description)/urdf/mounts/kinect_mount.urdf.xacro" />
+  <xacro:include filename="$(find segbot_description)/urdf/common.urdf.xacro" />
+  <xacro:include filename="$(find segbot_description)/gazebo/segbot.gazebo.xacro" />
+  <xacro:include filename="$(find segbot_description)/urdf/segbot_base.urdf.xacro" />
+  <xacro:include filename="$(find segbot_description)/urdf/segbot_chassis.urdf.xacro" />
+  <xacro:include filename="$(find segbot_description)/urdf/mounts/kinect_mount.urdf.xacro" />
   <!-- Add the segbot base -->
   <xacro:segbot />

File: segbot_description/robots/segbot_hokuyo.urdf.xacro (robot description, xacro)
@@ -3,9 +3,9 @@
        xmlns:xacro="http://ros.org/wiki/xacro">
   <!-- Included URDF Files -->
-  <include filename="$(find segbot_description)/urdf/common.urdf.xacro" />
-  <include filename="$(find segbot_description)/gazebo/full_collision.gazebo.xacro" />
-  <include filename="$(find segbot_description)/urdf/segbot_base.urdf.xacro" />
-  <include filename="$(find segbot_description)/urdf/segbot_chassis.urdf.xacro" />
-  <include filename="$(find segbot_description)/urdf/mounts/hokuyo_mount.urdf.xacro" />
+  <xacro:include filename="$(find segbot_description)/urdf/common.urdf.xacro" />
+  <xacro:include filename="$(find segbot_description)/gazebo/segbot.gazebo.xacro" />
+  <xacro:include filename="$(find segbot_description)/urdf/segbot_base.urdf.xacro" />
+  <xacro:include filename="$(find segbot_description)/urdf/segbot_chassis.urdf.xacro" />
+  <xacro:include filename="$(find segbot_description)/urdf/mounts/hokuyo_mount.urdf.xacro" />
   <!-- Add the segbot base -->
   <xacro:segbot />

File: segbot_description/robots/segbot_kinect.urdf.xacro (robot description, xacro)
@@ -3,9 +3,9 @@
        xmlns:xacro="http://ros.org/wiki/xacro">
   <!-- Included URDF Files -->
-  <include filename="$(find segbot_description)/urdf/common.urdf.xacro" />
-  <include filename="$(find segbot_description)/gazebo/full_collision.gazebo.xacro" />
-  <include filename="$(find segbot_description)/urdf/segbot_base.urdf.xacro" />
-  <include filename="$(find segbot_description)/urdf/segbot_chassis.urdf.xacro" />
-  <include filename="$(find segbot_description)/urdf/mounts/kinect_mount.urdf.xacro" />
+  <xacro:include filename="$(find segbot_description)/urdf/common.urdf.xacro" />
+  <xacro:include filename="$(find segbot_description)/gazebo/segbot.gazebo.xacro" />
+  <xacro:include filename="$(find segbot_description)/urdf/segbot_base.urdf.xacro" />
+  <xacro:include filename="$(find segbot_description)/urdf/segbot_chassis.urdf.xacro" />
+  <xacro:include filename="$(find segbot_description)/urdf/mounts/kinect_mount.urdf.xacro" />
   <!-- Add the segbot base -->
   <xacro:segbot />

File: segbot_description/test/hokuyo_mount.test.xacro (robot description, xacro)
@@ -3,6 +3,6 @@
        xmlns:xacro="http://ros.org/wiki/xacro">
   <!-- Included URDF Files -->
-  <include filename="$(find segbot_description)/urdf/common.urdf.xacro" />
-  <include filename="$(find segbot_description)/urdf/mounts/hokuyo_mount.urdf.xacro" />
+  <xacro:include filename="$(find segbot_description)/urdf/common.urdf.xacro" />
+  <xacro:include filename="$(find segbot_description)/urdf/mounts/hokuyo_mount.urdf.xacro" />
   <!-- add the root link -->
   <link name="base_link">

File: segbot_description/test/kinect_mount.test.xacro (robot description, xacro)
@@ -3,6 +3,6 @@
        xmlns:xacro="http://ros.org/wiki/xacro">
   <!-- Included URDF Files -->
-  <include filename="$(find segbot_description)/urdf/common.urdf.xacro" />
-  <include filename="$(find segbot_description)/urdf/mounts/kinect_mount.urdf.xacro" />
+  <xacro:include filename="$(find segbot_description)/urdf/common.urdf.xacro" />
+  <xacro:include filename="$(find segbot_description)/urdf/mounts/kinect_mount.urdf.xacro" />
   <!-- add the root link -->
   <link name="base_link">

File: segbot_description/test/segbot_chassis.test.xacro (robot description, xacro)
@@ -3,6 +3,6 @@
        xmlns:xacro="http://ros.org/wiki/xacro">
   <!-- Included URDF Files -->
-  <include filename="$(find segbot_description)/urdf/common.urdf.xacro" />
-  <include filename="$(find segbot_description)/urdf/segbot_chassis.urdf.xacro" />
+  <xacro:include filename="$(find segbot_description)/urdf/common.urdf.xacro" />
+  <xacro:include filename="$(find segbot_description)/urdf/segbot_chassis.urdf.xacro" />
   <!-- add the root link -->
   <link name="base_link">

File: segbot_description/urdf/mounts/hokuyo_mount.urdf.xacro (robot description, xacro)
@@ -4,8 +4,8 @@
       xmlns:interface="http://playerstage.sourceforge.net/gazebo/xmlschema/#interface"
       xmlns:xacro="http://ros.org/wiki/xacro">
-  <include filename="$(find segbot_description)/urdf/components/beam_8020.urdf.xacro" />
-  <include filename="$(find segbot_description)/urdf/components/standoff_632.urdf.xacro" />
-  <include filename="$(find segbot_description)/urdf/components/aluminium_sheet.urdf.xacro" />
-  <include filename="$(find segbot_description)/urdf/sensors/hokuyo_04lx_laser.urdf.xacro" />
+  <xacro:include filename="$(find segbot_description)/urdf/components/beam_8020.urdf.xacro" />
+  <xacro:include filename="$(find segbot_description)/urdf/components/standoff_632.urdf.xacro" />
+  <xacro:include filename="$(find segbot_description)/urdf/components/aluminium_sheet.urdf.xacro" />
+  <xacro:include filename="$(find segbot_description)/urdf/sensors/hokuyo_04lx_laser.urdf.xacro" />
   <xacro:macro name="hokuyo_mount" params="name parent *origin length ros_topic update_rate min_angle max_angle">
     <xacro:beam_8020 name="${name}_sensor_beam" parent="${parent}" length="${length}">

File: segbot_description/urdf/mounts/kinect_mount.urdf.xacro (robot description, xacro)
@@ -4,8 +4,8 @@
       xmlns:interface="http://playerstage.sourceforge.net/gazebo/xmlschema/#interface"
       xmlns:xacro="http://ros.org/wiki/xacro">
-  <include filename="$(find segbot_description)/urdf/components/beam_8020.urdf.xacro" />
-  <include filename="$(find segbot_description)/urdf/components/standoff_632.urdf.xacro" />
-  <include filename="$(find segbot_description)/urdf/components/aluminium_sheet.urdf.xacro" />
-  <include filename="$(find segbot_description)/urdf/sensors/kinect_camera.urdf.xacro" />
+  <xacro:include filename="$(find segbot_description)/urdf/components/beam_8020.urdf.xacro" />
+  <xacro:include filename="$(find segbot_description)/urdf/components/standoff_632.urdf.xacro" />
+  <xacro:include filename="$(find segbot_description)/urdf/components/aluminium_sheet.urdf.xacro" />
+  <xacro:include filename="$(find segbot_description)/urdf/sensors/kinect_camera.urdf.xacro" />
   <xacro:macro name="kinect_mount" params="name parent *origin length">
     <xacro:beam_8020 name="${name}_sensor_beam" parent="${parent}" length="${length}">

File: segbot_description/urdf/segbot_base.urdf.xacro (robot description, xacro)
@@ -3,5 +3,5 @@
       xmlns:xacro="http://ros.org/wiki/xacro">
   <!-- Included URDF Files -->
-  <include filename="$(find segbot_description)/urdf/segbot_wheel.urdf.xacro" />
+  <xacro:include filename="$(find segbot_description)/urdf/segbot_wheel.urdf.xacro" />
   <xacro:macro name="segbot">
     <!-- root link, on the ground just below the robot origin -->

File: segbot_description/urdf/segbot_chassis.urdf.xacro (robot description, xacro)
@@ -2,8 +2,8 @@
 <root xmlns:xacro="http://ros.org/wiki/xacro">
   <!-- Included URDF Files -->
-  <include filename="$(find segbot_description)/urdf/components/beam_8020.urdf.xacro" />
-  <include filename="$(find segbot_description)/urdf/components/aluminium_sheet.urdf.xacro" />
-  <include filename="$(find segbot_description)/urdf/components/battery_box.urdf.xacro" />
-  <include filename="$(find segbot_description)/urdf/components/laptop.urdf.xacro" />
+  <xacro:include filename="$(find segbot_description)/urdf/components/beam_8020.urdf.xacro" />
+  <xacro:include filename="$(find segbot_description)/urdf/components/aluminium_sheet.urdf.xacro" />
+  <xacro:include filename="$(find segbot_description)/urdf/components/battery_box.urdf.xacro" />
+  <xacro:include filename="$(find segbot_description)/urdf/components/laptop.urdf.xacro" />
   <xacro:macro name="segbot_chassis" params="parent *origin">
     <!-- base plate -->

File: segbot_description/urdf/sensors/hokuyo_04lx_laser.urdf.xacro (robot description, xacro)
@@ -4,5 +4,5 @@
       xmlns:interface="http://playerstage.sourceforge.net/gazebo/xmlschema/#interface"
       xmlns:xacro="http://ros.org/wiki/xacro">
-  <include filename="$(find segbot_description)/urdf/sensors/hokuyo_04lx_laser.gazebo.xacro" />
+  <xacro:include filename="$(find segbot_description)/urdf/sensors/hokuyo_04lx_laser.gazebo.xacro" />
   <xacro:macro name="hokuyo_04lx_laser" params="name parent *origin ros_topic update_rate min_angle max_angle">
     <joint name="${name}_joint" type="fixed">

File: segbot_description/urdf/sensors/kinect_camera.urdf.xacro (robot description, xacro)
@@ -4,5 +4,5 @@
       xmlns:interface="http://playerstage.sourceforge.net/gazebo/xmlschema/#interface"
       xmlns:xacro="http://ros.org/wiki/xacro">
-  <include filename="$(find segbot_description)/urdf/sensors/kinect_camera.gazebo.xacro" />
+  <xacro:include filename="$(find segbot_description)/urdf/sensors/kinect_camera.gazebo.xacro" />
   <xacro:macro name="kinect_camera" params="name parent *origin">
     <joint name="${name}_joint" type="fixed">
