Commit message: added inertial and collision changes that make the robot move properly under the simple model assumption in gazebo. The collision model of the robot no longer receives returns from the laser.

File: segbot_description/gazebo/segbot.gazebo.xacro (robot description, xacro)
@@ -2,5 +2,4 @@
 <root
   xmlns:xacro="http://ros.org/wiki/xacro">
-  <xacro:property name="SIMPLE_ROBOT_RADIUS" value="0.30" />
   <xacro:macro name="gazebo_segbot_base_link_surface">
     <gazebo reference="base_link">
@@ -27,4 +26,24 @@
     </gazebo>
   </xacro:macro>
+  <xacro:macro name="segbot_base_link_inertial" >
+    <xacro:if value="$(arg use_full_gazebo_model)">
+      <inertial>
+        <mass value="30" />
+        <origin xyz="-0.1 0 -0.075" />
+        <inertia ixx="3.0" ixy="0.0" ixz="0.0"
+          iyy="3.0" iyz="0.0"
+          izz="2.0" />
+      </inertial>
+    </xacro:if>
+    <xacro:unless value="$(arg use_full_gazebo_model)">
+      <inertial>
+        <mass value="30" />
+        <origin xyz="0 0 -0.2165" />
+        <inertia ixx="300.0" ixy="0.0" ixz="0.0"
+          iyy="300.0" iyz="0.0"
+          izz="300.0" />
+      </inertial>
+    </xacro:unless>
+  </xacro:macro>
   <xacro:macro name="segbot_base_link_collision" >
     <xacro:if value="$(arg use_full_gazebo_model)">
@@ -38,7 +57,7 @@
     <xacro:unless value="$(arg use_full_gazebo_model)">
       <collision>
-        <origin xyz="0 0 0.2" rpy="0 0 0" />
+        <origin xyz="-0.15 0 0" rpy="0 0 0" />
         <geometry>
-          <cylinder length="0.8330" radius="${SIMPLE_ROBOT_RADIUS}" />
+          <box size="0.5 0.4 0.4330" />
         </geometry>
       </collision>

File: segbot_description/urdf/segbot_base.urdf.xacro (robot description, xacro)
@@ -21,11 +21,5 @@
     <!-- This is the robot origin, center of the 2 wheels (axis of rotation) -->
     <link name="base_link">
-      <inertial>
-        <mass value="30" />
-        <origin xyz="-0.1 0 -0.075" />
-        <inertia ixx="3.0" ixy="0.0" ixz="0.0"
-          iyy="3.0" iyz="0.0"
-          izz="2.0" />
-      </inertial>
+      <xacro:segbot_base_link_inertial />
       <visual>
         <origin xyz="0 0 0" rpy="0 0 0" />

Commit message: increased model height to make the robots more visible

File: segbot_description/gazebo/segbot.gazebo.xacro (robot description, xacro)
@@ -57,7 +57,7 @@
     <xacro:unless value="$(arg use_full_gazebo_model)">
       <collision>
-        <origin xyz="-0.15 0 0" rpy="0 0 0" />
+        <origin xyz="-0.15 0 0.1" rpy="0 0 0" />
         <geometry>
-          <box size="0.5 0.4 0.4330" />
+          <box size="0.5 0.4 0.6330" />
         </geometry>
       </collision>

Commit message: increasing inertia to keep robot vertical

File: segbot_description/gazebo/segbot.gazebo.xacro (robot description, xacro)
@@ -40,7 +40,7 @@
         <mass value="30" />
         <origin xyz="0 0 -0.2165" />
-        <inertia ixx="300.0" ixy="0.0" ixz="0.0"
-          iyy="300.0" iyz="0.0"
-          izz="300.0" />
+        <inertia ixx="3000.0" ixy="0.0" ixz="0.0"
+          iyy="3000.0" iyz="0.0"
+          izz="3000.0" />
       </inertial>
     </xacro:unless>

Commit message: added an obstacle that would make the robot somewhat visible in gazebo

File: segbot_description/gazebo/segbot.gazebo.xacro (robot description, xacro)
@@ -57,9 +57,39 @@
     <xacro:unless value="$(arg use_full_gazebo_model)">
       <collision>
-        <origin xyz="-0.15 0 0.1" rpy="0 0 0" />
-        <geometry>
-          <box size="0.5 0.4 0.6330" />
-        </geometry>
-      </collision>
+        <origin xyz="0 0 0" rpy="0 0 0" />
+        <geometry>
+          <cylinder radius="0.305" length="0.4330" />
+        </geometry>
+      </collision>
+    </xacro:unless>
+  </xacro:macro>
+  <xacro:macro name="gazebo_laser_obstacle">
+    <xacro:unless value="$(arg use_full_gazebo_model)">
+      <joint name="laser_obstacle_joint" type="fixed">
+        <origin xyz="0.0 0 0.4165" rpy="0 0 0" />
+        <parent link="base_link"/>
+        <child link="laser_obstacle" />
+      </joint>
+      <link name="laser_obstacle">
+        <inertial>
+          <mass value="0.1" />
+          <origin xyz="0 0 0" rpy="0 0 0"/>
+          <inertia ixx="0.01"  ixy="0.0"  ixz="0.0"
+                   iyy="0.01"  iyz="0.0"
+                   izz="0.01" />
+        </inertial>
+       <visual>
+          <origin xyz="0 0 0" rpy="0 0 0" />
+          <geometry>
+            <box size="0.001 0.001 0.001" />
+          </geometry>
+        </visual>
+        <collision>
+          <origin xyz="0 0 0" rpy="0 0 0" />
+          <geometry>
+            <box size="0.25 0.6 0.4" />
+          </geometry>
+        </collision>
+      </link>
     </xacro:unless>
   </xacro:macro>

File: segbot_description/urdf/segbot_base.urdf.xacro (robot description, xacro)
@@ -30,4 +30,5 @@
       <xacro:segbot_base_link_collision />
     </link>
+    <xacro:gazebo_laser_obstacle />
     <xacro:gazebo_segbot_base_link_surface />
     <!-- castor joint -->

Commit message: updated description bringup to remove unneeded segbot v1 models, better naming for segbot v1 models, and introduced the segbot v2 model.

File: segbot_description/gazebo/segbot.gazebo.xacro (robot description, xacro)
@@ -57,7 +57,7 @@
     <xacro:unless value="$(arg use_full_gazebo_model)">
       <collision>
-        <origin xyz="0 0 0" rpy="0 0 0" />
-        <geometry>
-          <cylinder radius="0.305" length="0.4330" />
+        <origin xyz="0 0 -0.05" rpy="0 0 0" />
+        <geometry>
+          <cylinder radius="0.305" length="0.3330" />
         </geometry>
       </collision>

File: segbot_description/robots/segbot_v1.no_sensors.urdf.xacro (robot description, xacro)
@@ -3,9 +3,8 @@
        xmlns:xacro="http://ros.org/wiki/xacro">
   <!-- Included URDF Files -->
-  <xacro:include filename="$(find segbot_description)/urdf/common.urdf.xacro" />
+  <xacro:include filename="$(find segbot_description)/urdf/v1/common.urdf.xacro" />
   <xacro:include filename="$(find segbot_description)/gazebo/segbot.gazebo.xacro" />
   <xacro:include filename="$(find segbot_description)/urdf/segbot_base.urdf.xacro" />
-  <xacro:include filename="$(find segbot_description)/urdf/segbot_chassis.urdf.xacro" />
-  <xacro:include filename="$(find segbot_description)/urdf/mounts/kinect_mount.urdf.xacro" />
+  <xacro:include filename="$(find segbot_description)/urdf/v1/segbot_chassis.urdf.xacro" />
   <!-- Add the segbot base -->
   <xacro:segbot />

File: segbot_description/robots/segbot_v1.urdf.xacro (robot description, xacro)
@@ -3,9 +3,10 @@
        xmlns:xacro="http://ros.org/wiki/xacro">
   <!-- Included URDF Files -->
-  <xacro:include filename="$(find segbot_description)/urdf/common.urdf.xacro" />
+  <xacro:include filename="$(find segbot_description)/urdf/v1/common.urdf.xacro" />
   <xacro:include filename="$(find segbot_description)/gazebo/segbot.gazebo.xacro" />
   <xacro:include filename="$(find segbot_description)/urdf/segbot_base.urdf.xacro" />
-  <xacro:include filename="$(find segbot_description)/urdf/segbot_chassis.urdf.xacro" />
+  <xacro:include filename="$(find segbot_description)/urdf/v1/segbot_chassis.urdf.xacro" />
   <xacro:include filename="$(find segbot_description)/urdf/mounts/hokuyo_mount.urdf.xacro" />
+  <xacro:include filename="$(find segbot_description)/urdf/mounts/kinect_mount.urdf.xacro" />
   <!-- Add the segbot base -->
   <xacro:segbot />
@@ -13,4 +14,8 @@
     <origin xyz="${BASE_PLATE_X_OFFSET*INCH_TO_M} 0 ${BASE_PLATE_Z_OFFSET*INCH_TO_M}"/>
   </xacro:segbot_chassis>
+  <!-- Add the forward facing kinect sensor for navigation -->
+  <xacro:kinect_mount name="nav_kinect" parent="back_right_vertical_beam" length="${SENSOR_BEAM_LENGTH*INCH_TO_M}">
+    <origin xyz="0 ${0.5*INCH_TO_M} ${10.5*INCH_TO_M}" rpy="-${M_PI/2} -${M_PI/2} 0" />
+  </xacro:kinect_mount>
   <!-- Add the hokuyo -->
   <xacro:hokuyo_mount name="nav_hokuyo" parent="front_left_vertical_beam" length="${SENSOR_BEAM_LENGTH*INCH_TO_M}" ros_topic="scan" update_rate="10" min_angle="${-(5 * M_PI)/12}" max_angle="${(5 * M_PI)/12}">

File: segbot_description/robots/segbot_v2.urdf.xacro (robot description, xacro)
@@ -3,8 +3,8 @@
        xmlns:xacro="http://ros.org/wiki/xacro">
   <!-- Included URDF Files -->
-  <xacro:include filename="$(find segbot_description)/urdf/common.urdf.xacro" />
+  <xacro:include filename="$(find segbot_description)/urdf/v2/common.urdf.xacro" />
   <xacro:include filename="$(find segbot_description)/gazebo/segbot.gazebo.xacro" />
   <xacro:include filename="$(find segbot_description)/urdf/segbot_base.urdf.xacro" />
-  <xacro:include filename="$(find segbot_description)/urdf/segbot_chassis.urdf.xacro" />
+  <xacro:include filename="$(find segbot_description)/urdf/v2/segbot_chassis.urdf.xacro" />
   <xacro:include filename="$(find segbot_description)/urdf/mounts/hokuyo_mount.urdf.xacro" />
   <xacro:include filename="$(find segbot_description)/urdf/mounts/kinect_mount.urdf.xacro" />
@@ -16,10 +16,15 @@
   <!-- Add the forward facing kinect sensor for navigation -->
   <xacro:kinect_mount name="nav_kinect" parent="back_right_vertical_beam" length="${SENSOR_BEAM_LENGTH*INCH_TO_M}">
-    <origin xyz="0 ${0.5*INCH_TO_M} ${10.5*INCH_TO_M}" rpy="-${M_PI/2} -${M_PI/2} 0" />
+    <origin xyz="-${1*INCH_TO_M} -${0.5*INCH_TO_M} ${12*INCH_TO_M}" rpy="-${M_PI/2} -${M_PI/2} 0" />
   </xacro:kinect_mount>
   <!-- Add the hokuyo -->
   <xacro:hokuyo_mount name="nav_hokuyo" parent="front_left_vertical_beam" length="${SENSOR_BEAM_LENGTH*INCH_TO_M}" ros_topic="scan" update_rate="10" min_angle="${-(5 * M_PI)/12}" max_angle="${(5 * M_PI)/12}">
-    <origin xyz="0 -${0.5*INCH_TO_M} ${7*INCH_TO_M}" rpy="${M_PI/2} ${M_PI/2} 0" />
+    <origin xyz="${1*INCH_TO_M} ${0.5*INCH_TO_M} ${5*INCH_TO_M}" rpy="${M_PI/2} ${M_PI/2} 0" />
   </xacro:hokuyo_mount>
+  <!-- Add a beam at top so that the robot looks complete. -->
+  <xacro:beam_8020 name="front_cap_beam" parent="front_right_vertical_beam" length="${SENSOR_BEAM_LENGTH*INCH_TO_M}">
+    <origin xyz="0 -${0.5*INCH_TO_M} ${36.5*INCH_TO_M}"
+      rpy="-${M_PI/2} 0 0" />
+  </xacro:beam_8020>
   <xacro:gazebo_segbot_ros_controllers />
 </robot>

File: segbot_description/urdf/components/laptop.urdf.xacro (robot description, xacro)
@@ -37,5 +37,5 @@
     <!-- laptop screen -->
     <joint name="${name}_screen_joint" type="fixed">
-      <origin xyz="${4.5*INCH_TO_M} 0 ${0.75*INCH_TO_M}" rpy="0 -${M_PI/3} 0"/>
+      <origin xyz="${4.5*INCH_TO_M} 0 ${0.75*INCH_TO_M}" rpy="0 -${21/48*M_PI} 0"/>
       <parent link="${name}_link" />
       <child link="${name}_screen_link" />

File: segbot_description/urdf/v1/segbot_chassis.urdf.xacro (robot description, xacro)
@@ -2,8 +2,9 @@
 <root xmlns:xacro="http://ros.org/wiki/xacro">
   <!-- Included URDF Files -->
-  <xacro:include filename="$(find segbot_description)/urdf/components/beam_8020.urdf.xacro" />
   <xacro:include filename="$(find segbot_description)/urdf/components/aluminium_sheet.urdf.xacro" />
   <xacro:include filename="$(find segbot_description)/urdf/components/battery_box.urdf.xacro" />
+  <xacro:include filename="$(find segbot_description)/urdf/components/beam_8020.urdf.xacro" />
   <xacro:include filename="$(find segbot_description)/urdf/components/laptop.urdf.xacro" />
+  <xacro:include filename="$(find segbot_description)/urdf/components/standoff_632.urdf.xacro" />
   <xacro:macro name="segbot_chassis" params="parent *origin">
     <!-- base plate -->

Commit message: fixed location of laser obstacle for gazebo.

File: segbot_description/gazebo/segbot.gazebo.xacro (robot description, xacro)
@@ -67,5 +67,5 @@
     <xacro:unless value="$(arg use_full_gazebo_model)">
       <joint name="laser_obstacle_joint" type="fixed">
-        <origin xyz="0.0 0 0.4165" rpy="0 0 0" />
+        <origin xyz="0.0 0 0.3165" rpy="0 0 0" />
         <parent link="base_link"/>
         <child link="laser_obstacle" />
