Commit message: make standoff urdf more generic. dropped the 632 suffix and added radius as a parameter

File: segbot_description/gazebo/segbot.gazebo.xacro (robot description, xacro)
@@ -174,10 +174,10 @@
     </xacro:if>
   </xacro:macro>
-  <xacro:macro name="standoff_632_collision" params="length">
+  <xacro:macro name="standoff_collision" params="radius length">
     <xacro:if value="$(arg use_full_gazebo_model)">
       <collision>
         <origin xyz="0 0 ${length/2}" rpy="0 0 0"/>
         <geometry>
-          <cylinder length="${length}" radius="0.003175" />
+          <cylinder length="${length}" radius="${radius}" />
         </geometry>
       </collision>

File: segbot_description/urdf/components/standoff.urdf.xacro (robot description, xacro)
@@ -1,5 +1,5 @@
 <?xml version="1.0"?>
 <root xmlns:xacro="http://ros.org/wiki/xacro">
-  <xacro:macro name="standoff_632" params="name parent length *origin">
+  <xacro:macro name="standoff" params="name parent length radius *origin">
     <joint name="${name}_joint" type="fixed">
       <xacro:insert_block name="origin" />
@@ -18,8 +18,9 @@
         <origin xyz="0 0 ${length/2}" rpy="0 0 0"/>
         <geometry>
-          <cylinder length="${length}" radius="0.003175" />
+          <cylinder length="${length}" radius="${radius}" />
         </geometry>
         <material name="light_grey" />
       </visual>
+      <xacro:standoff_collision radius="${radius}" length="${length}" />
     </link>
     <gazebo reference="${name}_link">

File: segbot_description/urdf/mounts/hokuyo_mount.urdf.xacro (robot description, xacro)
@@ -5,5 +5,5 @@
       xmlns:xacro="http://ros.org/wiki/xacro">
   <xacro:include filename="$(find segbot_description)/urdf/components/beam_8020.urdf.xacro" />
-  <xacro:include filename="$(find segbot_description)/urdf/components/standoff_632.urdf.xacro" />
+  <xacro:include filename="$(find segbot_description)/urdf/components/standoff.urdf.xacro" />
   <xacro:include filename="$(find segbot_description)/urdf/components/aluminium_sheet.urdf.xacro" />
   <xacro:include filename="$(find segbot_description)/urdf/sensors/hokuyo_04lx_laser.urdf.xacro" />

File: segbot_description/urdf/mounts/kinect_mount.urdf.xacro (robot description, xacro)
@@ -5,5 +5,5 @@
       xmlns:xacro="http://ros.org/wiki/xacro">
   <xacro:include filename="$(find segbot_description)/urdf/components/beam_8020.urdf.xacro" />
-  <xacro:include filename="$(find segbot_description)/urdf/components/standoff_632.urdf.xacro" />
+  <xacro:include filename="$(find segbot_description)/urdf/components/standoff.urdf.xacro" />
   <xacro:include filename="$(find segbot_description)/urdf/components/aluminium_sheet.urdf.xacro" />
   <xacro:include filename="$(find segbot_description)/urdf/sensors/kinect_camera.urdf.xacro" />
@@ -16,20 +16,20 @@
                            <origin xyz="${0.5*INCH_TO_M} 0 ${length/2}" rpy="${M_PI/2} 0 ${M_PI/2}" />
     </xacro:aluminium_sheet>
-    <xacro:standoff_632 name="${name}_standoff_1" parent="${name}_base_plate" length="${2.0*INCH_TO_M}">
+    <xacro:standoff radius="0.003175" name="${name}_standoff_1" parent="${name}_base_plate" length="${2.0*INCH_TO_M}">
       <origin xyz="${1.5*INCH_TO_M} ${-4*INCH_TO_M} ${0.0625*INCH_TO_M}"
               rpy="0 0 0" />
-    </xacro:standoff_632>
-    <xacro:standoff_632 name="${name}_standoff_2" parent="${name}_base_plate" length="${2.0*INCH_TO_M}">
+    </xacro:standoff>
+    <xacro:standoff radius="0.003175" name="${name}_standoff_2" parent="${name}_base_plate" length="${2.0*INCH_TO_M}">
       <origin xyz="${1.5*INCH_TO_M} ${4*INCH_TO_M} ${0.0625*INCH_TO_M}"
               rpy="0 0 0" />
-    </xacro:standoff_632>
-    <xacro:standoff_632 name="${name}_standoff_3" parent="${name}_base_plate" length="${2.0*INCH_TO_M}">
+    </xacro:standoff>
+    <xacro:standoff radius="0.003175" name="${name}_standoff_3" parent="${name}_base_plate" length="${2.0*INCH_TO_M}">
       <origin xyz="${-1.5*INCH_TO_M} ${4*INCH_TO_M} ${0.0625*INCH_TO_M}"
               rpy="0 0 0" />
-    </xacro:standoff_632>
-    <xacro:standoff_632 name="${name}_standoff_4" parent="${name}_base_plate" length="${2.0*INCH_TO_M}">
+    </xacro:standoff>
+    <xacro:standoff radius="0.003175" name="${name}_standoff_4" parent="${name}_base_plate" length="${2.0*INCH_TO_M}">
       <origin xyz="${-1.5*INCH_TO_M} ${-4*INCH_TO_M} ${0.0625*INCH_TO_M}"
               rpy="0 0 0" />
-    </xacro:standoff_632>
+    </xacro:standoff>
     <xacro:aluminium_sheet name="${name}_top_plate" parent="${name}_standoff_1"
                            thickness="${0.0625*INCH_TO_M}" length="${4*INCH_TO_M}" width="${9*INCH_TO_M}">

File: segbot_description/urdf/mounts/sensor_mount.urdf.xacro (robot description, xacro)
@@ -2,25 +2,25 @@
 <!-- mounting for Arduino and its attached sensors -->
 <root xmlns:xacro="http://ros.org/wiki/xacro">
-  <xacro:include filename="$(find segbot_description)/urdf/components/standoff_632.urdf.xacro" />
+  <xacro:include filename="$(find segbot_description)/urdf/components/standoff.urdf.xacro" />
   <xacro:include filename="$(find segbot_description)/urdf/components/aluminium_sheet.urdf.xacro" />
   <xacro:macro name="sensor_mount" params="name parent">
     <!-- add sensor mount plate and its standoffs -->
-    <xacro:standoff_632 name="${name}_front_left_standoff" parent="${parent}"
+    <xacro:standoff radius="0.003175" name="${name}_front_left_standoff" parent="${parent}"
                         length="${1.5*INCH_TO_M}">
       <origin xyz="${3.25*INCH_TO_M} ${4.5*INCH_TO_M} ${(1/32)*INCH_TO_M}"
               rpy="0 0 0" />
-    </xacro:standoff_632>
-    <xacro:standoff_632 name="${name}_front_right_standoff" parent="${parent}"
+    </xacro:standoff>
+    <xacro:standoff radius="0.003175" name="${name}_front_right_standoff" parent="${parent}"
                         length="${1.5*INCH_TO_M}">
       <origin xyz="${3.25*INCH_TO_M} ${-4.5*INCH_TO_M} ${(1/32)*INCH_TO_M}" rpy="0 0 0" />
-    </xacro:standoff_632>
-    <xacro:standoff_632 name="${name}_back_left_standoff" parent="${parent}"
+    </xacro:standoff>
+    <xacro:standoff radius="0.003175" name="${name}_back_left_standoff" parent="${parent}"
                         length="${1.5*INCH_TO_M}">
       <origin xyz="${1.25*INCH_TO_M} ${4.5*INCH_TO_M} ${(1/32)*INCH_TO_M}" rpy="0 0 0" />
-    </xacro:standoff_632>
-    <xacro:standoff_632 name="${name}_back_right_standoff" parent="${parent}"
+    </xacro:standoff>
+    <xacro:standoff radius="0.003175" name="${name}_back_right_standoff" parent="${parent}"
                         length="${1.5*INCH_TO_M}">
       <origin xyz="${1.25*INCH_TO_M} ${-4.5*INCH_TO_M} ${(1/32)*INCH_TO_M}" rpy="0 0 0" />
-    </xacro:standoff_632>
+    </xacro:standoff>
     <xacro:aluminium_sheet name="${name}_plate"
                            parent="${name}_front_left_standoff"
@@ -32,24 +32,24 @@
     </xacro:aluminium_sheet>
     <!-- add sensor mount top plate and its standoffs -->
-    <xacro:standoff_632 name="${name}_top_front_left_standoff"
+    <xacro:standoff radius="0.003175" name="${name}_top_front_left_standoff"
                         parent="${name}_front_left_standoff"
                         length="${2*INCH_TO_M}">
       <origin xyz="0 0 ${(1.5+1/16)*INCH_TO_M}" rpy="0 0 0" />
-    </xacro:standoff_632>
-    <xacro:standoff_632 name="${name}_top_front_right_standoff"
+    </xacro:standoff>
+    <xacro:standoff radius="0.003175" name="${name}_top_front_right_standoff"
                         parent="${name}_front_right_standoff"
                         length="${2*INCH_TO_M}">
       <origin xyz="0 0 ${(1.5+1/16)*INCH_TO_M}" rpy="0 0 0" />
-    </xacro:standoff_632>
-    <xacro:standoff_632 name="${name}_top_back_left_standoff"
+    </xacro:standoff>
+    <xacro:standoff radius="0.003175" name="${name}_top_back_left_standoff"
                         parent="${name}_back_left_standoff"
                         length="${2*INCH_TO_M}">
       <origin xyz="0 0 ${(1.5+1/16)*INCH_TO_M}" rpy="0 0 0" />
-    </xacro:standoff_632>
-    <xacro:standoff_632 name="${name}_top_back_right_standoff"
+    </xacro:standoff>
+    <xacro:standoff radius="0.003175" name="${name}_top_back_right_standoff"
                         parent="${name}_back_right_standoff"
                         length="${2*INCH_TO_M}">
       <origin xyz="0 0 ${(1.5+1/16)*INCH_TO_M}" rpy="0 0 0" />
-    </xacro:standoff_632>
+    </xacro:standoff>
     <xacro:aluminium_sheet name="${name}_top_plate"
                            parent="${name}_top_front_left_standoff"

File: segbot_description/urdf/v1/segbot_chassis.urdf.xacro (robot description, xacro)
@@ -6,5 +6,5 @@
   <xacro:include filename="$(find segbot_description)/urdf/components/beam_8020.urdf.xacro" />
   <xacro:include filename="$(find segbot_description)/urdf/components/laptop.urdf.xacro" />
-  <xacro:include filename="$(find segbot_description)/urdf/components/standoff_632.urdf.xacro" />
+  <xacro:include filename="$(find segbot_description)/urdf/components/standoff.urdf.xacro" />
   <xacro:macro name="segbot_chassis" params="parent *origin">
     <!-- base plate -->
@@ -14,20 +14,20 @@
     </xacro:aluminium_sheet>
     <!-- add chassis mount plate -->
-    <xacro:standoff_632 name="chassis_front_left_standoff" parent="chassis_base_plate"
+    <xacro:standoff radius="0.003175" name="chassis_front_left_standoff" parent="chassis_base_plate"
                         length="${0.5*INCH_TO_M}">
       <origin xyz="${8.25*INCH_TO_M} ${4.5*INCH_TO_M} ${0.125*INCH_TO_M}" rpy="0 0 0" />
-    </xacro:standoff_632>
-    <xacro:standoff_632 name="chassis_front_right_standoff" parent="chassis_base_plate"
+    </xacro:standoff>
+    <xacro:standoff radius="0.003175" name="chassis_front_right_standoff" parent="chassis_base_plate"
                         length="${0.5*INCH_TO_M}">
       <origin xyz="${8.25*INCH_TO_M} ${-4.5*INCH_TO_M} ${0.125*INCH_TO_M}" rpy="0 0 0" />
-    </xacro:standoff_632>
-    <xacro:standoff_632 name="chassis_back_left_standoff" parent="chassis_base_plate"
+    </xacro:standoff>
+    <xacro:standoff radius="0.003175" name="chassis_back_left_standoff" parent="chassis_base_plate"
                         length="${0.5*INCH_TO_M}">
       <origin xyz="${6.25*INCH_TO_M} ${4.5*INCH_TO_M} ${0.125*INCH_TO_M}" rpy="0 0 0" />
-    </xacro:standoff_632>
-    <xacro:standoff_632 name="chassis_back_right_standoff" parent="chassis_base_plate"
+    </xacro:standoff>
+    <xacro:standoff radius="0.003175" name="chassis_back_right_standoff" parent="chassis_base_plate"
                         length="${0.5*INCH_TO_M}">
       <origin xyz="${6.25*INCH_TO_M} ${-4.5*INCH_TO_M} ${0.125*INCH_TO_M}" rpy="0 0 0" />
-    </xacro:standoff_632>
+    </xacro:standoff>
     <xacro:aluminium_sheet name="chassis_mount_plate" parent="chassis_front_left_standoff"
                            thickness="${0.0625*INCH_TO_M}" length="${11*INCH_TO_M}"

File: segbot_description/urdf/v2/segbot_chassis.urdf.xacro (robot description, xacro)
@@ -6,5 +6,5 @@
   <xacro:include filename="$(find segbot_description)/urdf/components/beam_8020.urdf.xacro" />
   <xacro:include filename="$(find segbot_description)/urdf/components/laptop.urdf.xacro" />
-  <xacro:include filename="$(find segbot_description)/urdf/components/standoff_632.urdf.xacro" />
+  <xacro:include filename="$(find segbot_description)/urdf/components/standoff.urdf.xacro" />
   <xacro:macro name="segbot_chassis" params="parent *origin">
     <!-- base plate -->
