Commit message: still working through issues found on the real robot.

File: segbot_description/urdf/mounts/velodyne_mount.urdf.xacro (robot description, xacro)
@@ -39,6 +39,6 @@
       <origin xyz="0 0 ${3.125*INCH_TO_M}" rpy="0 0 0" />
     </xacro:aluminium_sheet>
-    <xacro:VLP-16 parent="${name}_top_plate_link" name="${name}" topic="${name}/points">
-      <origin xyz="0 0 ${0.125*INCH_TO_M}" rpy="0 0 ${M_PI/4}" />
+    <xacro:VLP-16 parent="${name}_top_plate_link" name="${name}" topic="${name}_points">
+      <origin xyz="0 0 ${0.125*INCH_TO_M}" rpy="0 0 -${M_PI/4}" />
     </xacro:VLP-16>
   </xacro:macro>
