Commit message: added a mount for the velodyne, along with necessary dependencies.

File: segbot_description/test/hokuyo_mount.test.xacro (robot description, xacro)
@@ -3,5 +3,5 @@
        xmlns:xacro="http://ros.org/wiki/xacro">
   <!-- Included URDF Files -->
-  <xacro:include filename="$(find segbot_description)/urdf/common.urdf.xacro" />
+  <xacro:include filename="$(find segbot_description)/urdf/v3/common.urdf.xacro" />
   <xacro:include filename="$(find segbot_description)/urdf/mounts/hokuyo_mount.urdf.xacro" />
   <!-- add the root link -->

File: segbot_description/test/velodyne_mount.test.xacro (robot description, xacro)
@@ -4,5 +4,5 @@
   <!-- Included URDF Files -->
   <xacro:include filename="$(find segbot_description)/urdf/v3/common.urdf.xacro" />
-  <xacro:include filename="$(find segbot_description)/urdf/mounts/kinect_mount.urdf.xacro" />
+  <xacro:include filename="$(find segbot_description)/urdf/mounts/velodyne_mount.urdf.xacro" />
   <!-- add the root link -->
   <link name="base_link">
@@ -15,6 +15,6 @@
   </link>
   <!-- Add the kinect camera -->
-  <xacro:kinect_mount name="test_kinect" parent="base" length="${10.75*INCH_TO_M}">
-    <origin xyz="0 0 0" rpy="-${M_PI/2} -${M_PI/2} 0" />
-  </xacro:kinect_mount>
+  <xacro:velodyne_mount name="test_kinect" parent="base">
+    <origin xyz="0 0 0" rpy="0 0 0" />
+  </xacro:velodyne_mount>
 </robot>
